File: AD4030/Hardware/AD4030-Voltage/DIFF.kicad_sch (KiCad schematic)
At the start: 66 parts, among them J203 1710072, U201 ADA4817-1ARD, U202 ADA4817-1ARD, U203 CPC1017N, U204 LMH6611

Commit message: Hardware design
Parts:
- removed U203: CPC1017N, Package_SO:SOP-4_3.8x4.1mm_P2.54mm, symbol Relay_SolidState:CPC1017N
- removed U204: LMH6611, Package_TO_SOT_SMD:TSOT-23-6, symbol Amplifier_Operational:LMH6611
- added C222: 50p, symbol Device:C
- added C223, C224, C225, C226, C227, C228, C229, C230, C231, C232: 0.1u, symbol Device:C
- added K202: UMS05-1A80-75D, Relay_THT:Relay_StandexMeder_UMS, symbol Relay:UMS05-1A80-75D
- added Q201: MMBT3904, Package_TO_SOT_SMD:SOT-23, symbol Transistor_BJT:MMBT3904
- added R237: R, symbol Device:R
- added R238: 51, symbol Device:R
- added RN201: VoltageDivider_CenterPin3, Package_TO_SOT_SMD:SOT-23, symbol Device:VoltageDivider_CenterPin3
- added RV203: 20k, symbol Device:R_Potentiometer_Trim
- added U203: ADG5236BCPZ, Package_DFN_QFN:QFN-16-1EP_4x4mm_P0.65mm_EP2.5x2.5mm_ThermalVias, symbol AD4030:ADG5236BCPZ
- added U205: AD797BRZ, symbol Amplifier_Operational:AD797
- added U206: ADA4895-1ARJZ, symbol Amplifier_Operational:ADA4807-1
- R233: value 560 -> 10k
Connections:
- net +5VA: now also C223.1, C224.1, C225.1, C226.1, C227.1, U203.11 (VDD), U205.7 (V+), U206.5 (~{DISABLE}), U206.6 (V+)
- net -5VA: now also C228.1, C229.1, C230.1, C231.1, C232.1, RV203.2, U203.17 (EP), U203.3 (VSS), U205.4 (V-), U206.2 (V-)
- net GND: now also Q201.2 (E)
- net GNDA: now also C223.2, C224.2, C225.2, C226.2, C227.2, C228.2, C229.2, C230.2, C231.2, C232.2, RN201.2, U203.4 (GND)
- net at C221.1, R231.1, R232.1: now also K202.4
- net at R227.2, R228.2, R234.1: now also U206.3 (+)
- net at C218.2, R222.2, R223.2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: now also K202.3
- net at R229.2, R230.2, R235.1: now also U206.4 (-)
- net at R235.2, R236.1: now also U206.1
- net at R233.1: now also Q201.1 (B)
- net GAIN_x10-100 renamed Gain_x10-x100
- net V_OUTPUT: no longer names the net of R236.2
- net V_OUTPUT: now also U203.1
- new net: K202.2, Q201.3 (C)
- new net: RV203.3, U205.1 (BAL)
- new net: RN201.3, U205.2 (-)
- new net: U203.2, U205.3 (+)
- new net: RV203.1, U205.5 (COMP)
- new net: C222.2, R237.1, U203.10, U205.6
- new net: C222.1, U205.8 (C/B)
- new net: R237.2, RN201.1
- new net: R238.1, U203.9
- new net: U203.16, U203.8
- new net +5V: K202.1, U203.12 (EN)
- new net GAIN_x3: U203.15, U203.6
- new net V_OUT: R238.2
Other:
- note added: "CMRR"
- note added: "Gain x3.125"
- note added: "OFFSET"
- moved on the sheet: C201, C202, C203, C204, C205, C206, C207, C208, C209, C210, C211, C212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

Commit message: Hardware
Changed lines of the file:
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@@
 		(dnp no)
 		(property "Reference" "RV203"
-			(at 344.17 142.24 90)
+			(at 344.17 141.986 90)
 			(effects
 				(font
@@
 		)
 		(property "Value" "20k"
-			(at 344.17 144.78 90)
+			(at 344.17 144.272 90)
 			(effects
 				(font

Commit message: Hardware
Other:
- moved on the sheet: C220, C221, R232
Changed lines of the file:
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@@
 	)
 	(junction
-		(at 191.77 115.57)
-		(diameter 0)
-		(color 0 0 0 0)
-	)
-	(junction
 		(at 30.48 99.06)
 		(diameter 0)
@@
 	)
 	(junction
+		(at 193.04 115.57)
+		(diameter 0)
+		(color 0 0 0 0)
+	)
+	(junction
 		(at 139.7 262.89)
 		(diameter 0)
@@
 	(wire
 		(pts
-			(xy 181.61 130.81) (xy 170.18 130.81)
+			(xy 181.61 130.81) (xy 166.37 130.81)
 		)
 		(stroke
@@
 	(wire
 		(pts
-			(xy 170.18 115.57) (xy 181.61 115.57)
+			(xy 166.37 115.57) (xy 181.61 115.57)
 		)
 		(stroke
@@
 	(wire
 		(pts
-			(xy 191.77 127) (xy 191.77 130.81)
+			(xy 193.04 127) (xy 193.04 130.81)
 		)
 		(stroke
@@
 	(wire
 		(pts
-			(xy 191.77 119.38) (xy 191.77 115.57)
+			(xy 193.04 119.38) (xy 193.04 115.57)
 		)
 		(stroke
@@
 	(wire
 		(pts
-			(xy 191.77 130.81) (xy 181.61 130.81)
+			(xy 193.04 130.81) (xy 181.61 130.81)
 		)
 		(stroke
@@
 	(wire
 		(pts
+			(xy 193.04 115.57) (xy 205.74 115.57)
+		)
+		(stroke
+			(width 0)
+			(type default)
+		)
+	)
+	(wire
+		(pts
 			(xy 379.73 119.38) (xy 382.27 119.38)
 		)
@@
 	(wire
 		(pts
-			(xy 181.61 115.57) (xy 191.77 115.57)
+			(xy 181.61 115.57) (xy 193.04 115.57)
 		)
 		(stroke
@@
 	(wire
 		(pts
-			(xy 191.77 115.57) (xy 205.74 115.57)
-		)
-		(stroke
-			(width 0)
-			(type default)
-		)
-	)
-	(wire
-		(pts
 			(xy 349.25 147.32) (xy 347.98 147.32)
 		)
@@
 	(symbol
 		(lib_id "Device:R")
-		(at 191.77 123.19 0)
+		(at 193.04 123.19 0)
 		(unit 1)
 		(exclude_from_sim no)
@@
 		(fields_autoplaced yes)
 		(property "Reference" "R232"
-			(at 194.31 121.9199 0)
+			(at 195.58 121.9199 0)
 			(effects
 				(font
@@
 		)
 		(property "Value" "120/0.1%"
-			(at 194.31 124.4599 0)
+			(at 195.58 124.4599 0)
 			(effects
 				(font
@@
 		)
 		(property "Footprint" ""
-			(at 189.992 123.19 90)
+			(at 191.262 123.19 90)
 			(effects
 				(font
@@
 		)
 		(property "Datasheet" "~"
-			(at 191.77 123.19 0)
+			(at 193.04 123.19 0)
 			(effects
 				(font
@@
 		)
 		(property "Description" "Resistor"
-			(at 191.77 123.19 0)
+			(at 193.04 123.19 0)
 			(effects
 				(font
@@
 	(symbol
 		(lib_id "Device:C")
-		(at 170.18 119.38 0)
+		(at 166.37 119.38 0)
 		(unit 1)
 		(exclude_from_sim no)
@@
 		(fields_autoplaced yes)
 		(property "Reference" "C221"
-			(at 173.99 118.1099 0)
+			(at 170.18 118.1099 0)
 			(effects
 				(font
@@
 		)
 		(property "Value" "470p"
-			(at 173.99 120.6499 0)
+			(at 170.18 120.6499 0)
 			(effects
 				(font
@@
 		)
 		(property "Footprint" ""
-			(at 171.1452 123.19 0)
+			(at 167.3352 123.19 0)
 			(effects
 				(font
@@
 		)
 		(property "Datasheet" "~"
-			(at 170.18 119.38 0)
+			(at 166.37 119.38 0)
 			(effects
 				(font
@@
 		)
 		(property "Description" "Unpolarized capacitor"
-			(at 170.18 119.38 0)
+			(at 166.37 119.38 0)
 			(effects
 				(font
@@
 	(symbol
 		(lib_id "Device:C")
-		(at 170.18 127 0)
+		(at 166.37 127 0)
 		(unit 1)
 		(exclude_from_sim no)
@@
 		(fields_autoplaced yes)
 		(property "Reference" "C220"
-			(at 173.99 125.7299 0)
+			(at 170.18 125.7299 0)
 			(effects
 				(font
@@
 		)
 		(property "Value" "470p"
-			(at 173.99 128.2699 0)
+			(at 170.18 128.2699 0)
 			(effects
 				(font
@@
 		)
 		(property "Footprint" ""
-			(at 171.1452 130.81 0)
+			(at 167.3352 130.81 0)
 			(effects
 				(font
@@
 		)
 		(property "Datasheet" "~"
-			(at 170.18 127 0)
+			(at 166.37 127 0)
 			(effects
 				(font
@@
 		)
 		(property "Description" "Unpolarized capacitor"
-			(at 170.18 127 0)
+			(at 166.37 127 0)
 			(effects
 				(font

Commit message: Hardware
Parts:
- C201: renamed from C205; footprint (none) -> Capacitor_SMD:C_1206_3216Metric_Pad1.33x1.80mm_HandSolder
- C202: renamed from C204; footprint (none) -> Capacitor_SMD:C_1206_3216Metric_Pad1.33x1.80mm_HandSolder
- C203: renamed from C206; footprint (none) -> Capacitor_SMD:C_1206_3216Metric_Pad1.33x1.80mm_HandSolder
- C204: renamed from C203; footprint (none) -> Capacitor_SMD:C_1206_3216Metric_Pad1.33x1.80mm_HandSolder
- C205: renamed from C223; footprint (none) -> Capacitor_SMD:C_0603_1608Metric_Pad1.08x0.95mm_HandSolder
- C206: renamed from C207; footprint (none) -> Capacitor_SMD:C_1206_3216Metric_Pad1.33x1.80mm_HandSolder
- C207: renamed from C202; footprint (none) -> Capacitor_SMD:C_1206_3216Metric_Pad1.33x1.80mm_HandSolder
- C208: renamed from C224; footprint (none) -> Capacitor_SMD:C_0603_1608Metric_Pad1.08x0.95mm_HandSolder
- C209: renamed from C208; footprint (none) -> Capacitor_SMD:C_1206_3216Metric_Pad1.33x1.80mm_HandSolder
- C210: renamed from C201; footprint (none) -> Capacitor_SMD:C_1206_3216Metric_Pad1.33x1.80mm_HandSolder
- C211: renamed from C225; footprint (none) -> Capacitor_SMD:C_0603_1608Metric_Pad1.08x0.95mm_HandSolder
- C212: renamed from C209; footprint (none) -> Capacitor_SMD:C_1206_3216Metric_Pad1.33x1.80mm_HandSolder
- C213: renamed from C210; footprint (none) -> Capacitor_SMD:C_1206_3216Metric_Pad1.33x1.80mm_HandSolder
- C214: renamed from C226; footprint (none) -> Capacitor_SMD:C_0603_1608Metric_Pad1.08x0.95mm_HandSolder
- C215: renamed from C211; footprint (none) -> Capacitor_SMD:C_0603_1608Metric_Pad1.08x0.95mm_HandSolder
- C216: renamed from C214; footprint (none) -> Capacitor_SMD:C_0603_1608Metric_Pad1.08x0.95mm_HandSolder
- C217: renamed from C227; footprint (none) -> Capacitor_SMD:C_0603_1608Metric_Pad1.08x0.95mm_HandSolder
- C218: renamed from C212; footprint (none) -> Capacitor_SMD:C_0603_1608Metric_Pad1.08x0.95mm_HandSolder
- C219: renamed from C215; footprint (none) -> Capacitor_SMD:C_0603_1608Metric_Pad1.08x0.95mm_HandSolder
- C220: renamed from C228; footprint (none) -> Capacitor_SMD:C_0603_1608Metric_Pad1.08x0.95mm_HandSolder
- C223: renamed from C229; footprint (none) -> Capacitor_SMD:C_0603_1608Metric_Pad1.08x0.95mm_HandSolder
- C224: renamed from C217; footprint (none) -> Capacitor_SMD:C_0603_1608Metric_Pad1.08x0.95mm_HandSolder
- C225: renamed from C230; footprint (none) -> Capacitor_SMD:C_0603_1608Metric_Pad1.08x0.95mm_HandSolder
- C226: renamed from C231; footprint (none) -> Capacitor_SMD:C_0603_1608Metric_Pad1.08x0.95mm_HandSolder
- C227: renamed from C221; footprint (none) -> Capacitor_SMD:C_0603_1608Metric_Pad1.08x0.95mm_HandSolder
- C228: renamed from C220; value 470p -> 10n; footprint (none) -> Capacitor_SMD:C_0603_1608Metric_Pad1.08x0.95mm_HandSolder
- C229: renamed from C232; footprint (none) -> Capacitor_SMD:C_0603_1608Metric_Pad1.08x0.95mm_HandSolder
- C230: renamed from C218; footprint (none) -> Capacitor_SMD:C_0603_1608Metric_Pad1.08x0.95mm_HandSolder
- C231: renamed from C219; footprint (none) -> Capacitor_SMD:C_0603_1608Metric_Pad1.08x0.95mm_HandSolder
- C232: renamed from C222; footprint (none) -> Capacitor_SMD:C_0603_1608Metric_Pad1.08x0.95mm_HandSolder
- R201: renamed from R205; footprint (none) -> Resistor_SMD:R_1206_3216Metric_Pad1.30x1.75mm_HandSolder
- R202: renamed from R204; footprint (none) -> Resistor_SMD:R_1206_3216Metric_Pad1.30x1.75mm_HandSolder
- R203: renamed from R206; footprint (none) -> Resistor_SMD:R_1206_3216Metric_Pad1.30x1.75mm_HandSolder
- R204: renamed from R203; footprint (none) -> Resistor_SMD:R_1206_3216Metric_Pad1.30x1.75mm_HandSolder
- R205: renamed from R207; footprint (none) -> Resistor_SMD:R_1206_3216Metric_Pad1.30x1.75mm_HandSolder
- R206: renamed from R202; footprint (none) -> Resistor_SMD:R_1206_3216Metric_Pad1.30x1.75mm_HandSolder
- R207: renamed from R208; footprint (none) -> Resistor_SMD:R_1206_3216Metric_Pad1.30x1.75mm_HandSolder
- R208: renamed from R201; footprint (none) -> Resistor_SMD:R_1206_3216Metric_Pad1.30x1.75mm_HandSolder
- R209, R210, R211, R212, R215, R216: footprint (none) -> Resistor_SMD:R_1206_3216Metric_Pad1.30x1.75mm_HandSolder
- R213, R214: value 910 -> 91; footprint (none) -> Resistor_SMD:R_1206_3216Metric_Pad1.30x1.75mm_HandSolder
- R217: renamed from R219; footprint (none) -> Resistor_SMD:R_0603_1608Metric_Pad0.98x0.95mm_HandSolder
- R218: renamed from R220; footprint (none) -> Resistor_SMD:R_0603_1608Metric_Pad0.98x0.95mm_HandSolder
- R219: renamed from R218; footprint (none) -> Resistor_SMD:R_0603_1608Metric_Pad0.98x0.95mm_HandSolder
- R220: renamed from R217; footprint (none) -> Resistor_SMD:R_0603_1608Metric_Pad0.98x0.95mm_HandSolder
- R221, R233, R234, R235, R236, R237, R238: footprint (none) -> Resistor_SMD:R_0603_1608Metric_Pad0.98x0.95mm_HandSolder
- R222: renamed from R224; footprint (none) -> Resistor_SMD:R_0603_1608Metric_Pad0.98x0.95mm_HandSolder
- R223: renamed from R231; footprint (none) -> Resistor_SMD:R_0603_1608Metric_Pad0.98x0.95mm_HandSolder
- R224: renamed from R222; footprint (none) -> Resistor_SMD:R_0603_1608Metric_Pad0.98x0.95mm_HandSolder
- R225: renamed from R232; footprint (none) -> Resistor_SMD:R_0603_1608Metric_Pad0.98x0.95mm_HandSolder
- R226: renamed from R225; footprint (none) -> Resistor_SMD:R_0603_1608Metric_Pad0.98x0.95mm_HandSolder
- R227: renamed from R223; footprint (none) -> Resistor_SMD:R_0603_1608Metric_Pad0.98x0.95mm_HandSolder
- R228: renamed from R226; footprint (none) -> Resistor_SMD:R_0603_1608Metric_Pad0.98x0.95mm_HandSolder
- R229: renamed from R227; footprint (none) -> Resistor_SMD:R_0603_1608Metric_Pad0.98x0.95mm_HandSolder
- R230: renamed from R228; footprint (none) -> Resistor_SMD:R_0603_1608Metric_Pad0.98x0.95mm_HandSolder
- R231: renamed from R229; footprint (none) -> Resistor_SMD:R_0603_1608Metric_Pad0.98x0.95mm_HandSolder
- R232: renamed from R230; footprint (none) -> Resistor_SMD:R_0603_1608Metric_Pad0.98x0.95mm_HandSolder
- RV201: value 100/10T -> 3266W-1-101; footprint (none) -> Potentiometer_THT:Potentiometer_Bourns_3266W_Vertical
- RV202: value 10k/10T -> 3266W-1-103; footprint (none) -> Potentiometer_THT:Potentiometer_Bourns_3266W_Vertical
- RV203: value 20k -> 3266W-1-203; footprint (none) -> Potentiometer_THT:Potentiometer_Bourns_3266W_Vertical
- U204: renamed from U206; footprint (none) -> Package_TO_SOT_SMD:SOT-23-6_Handsoldering
- U205: footprint (none) -> Package_SO:SOIC-8_3.9x4.9mm_P1.27mm
- renumbered C213 to C221, C216 to C222, J203 to J201, K202 to K201, U203 to U201, U201 to U203
Connections:
- net at C228.2, R223.2, R225.2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: now also C231.1, R226.1, R228.1; no longer C231.2, R226.2, R228.2
- new net: C231.2, R226.2, R228.2, U203.1 (FB)

Commit message: Hardware and started to create simulation.
Parts:
- removed R211, R212, R215, R216: 10k/0.1%, Resistor_SMD:R_1206_3216Metric_Pad1.30x1.75mm_HandSolder, symbol Device:R
- removed R224, R226, R227, R228, R229, R230, R231, R232, R234, R235: 1k/0.1%, Resistor_SMD:R_0603_1608Metric_Pad0.98x0.95mm_HandSolder, symbol Device:R
- added U206: LT5400-1, Package_SO:MSOP-8-1EP_3x3mm_P0.65mm_EP1.73x1.85mm_ThermalVias, symbol AD4030:LT5400
- added U207, U208, U209: LT5400-4, Package_SO:MSOP-8-1EP_3x3mm_P0.65mm_EP1.73x1.85mm_ThermalVias, symbol AD4030:LT5400
- C221, C222: value 9-70p -> JR500; footprint (none) -> Capacitor_SMD:C_Trimmer_Voltronics_JR
- R236, R238: footprint Resistor_SMD:R_0603_1608Metric_Pad0.98x0.95mm_HandSolder -> (none)
- R237: value R -> 2k5/0.1%
- RN201: value VoltageDivider_CenterPin3 -> MPMT50011002AT1
Connections:
- net GNDA: now also RN201.1, U206.9, U207.9, U208.9, U209.8, U209.9; no longer RN201.2
- net at C228.2, C231.1, R223.2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: now also U208.3, U208.4
- net at C212.2, C215.1, C218.1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: now also U206.1
- net at U202.6: now also U207.1, U207.2
- net at U204.3 (+): now also U207.7, U207.8, U209.1
- net at C213.2, C216.2, C219.2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: now also U206.5
- net at R214.2: now also U206.6
- net at C230.2, K201.3, U202.2 (-): now also U208.7, U208.8
- net at C230.1, U202.1 (FB): now also U208.1, U208.2
- net at C231.2, U203.1 (FB): now also U208.5, U208.6
- net at U203.6: now also U207.3, U207.4
- net at U204.4 (-): now also U207.5, U207.6, U209.4
- net at R236.1, U204.1: now also U209.5
- net at R237.2: now also RN201.2; no longer RN201.1
- net at R213.1: now also U206.2
- new net: U206.7, U206.8
- new net: U206.3, U206.4
- no-connect marks 0 -> 4
Other:
- note added: "1/250"
- note added: "Gain x2.5"
- note removed: "Gain x3.125"
- moved on the sheet: C201, C202, C203, C204, C206, C207, C209, C210, C212, C213, C215, C216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

Commit message: Hardware design and simulation
Parts:
- removed R237: 2k5/0.1%, Resistor_SMD:R_0603_1608Metric_Pad0.98x0.95mm_HandSolder, symbol Device:R
- removed RN201: MPMT50011002AT1, Package_TO_SOT_SMD:SOT-23, symbol Device:VoltageDivider_CenterPin3
- removed RV203: 3266W-1-203, Potentiometer_THT:Potentiometer_Bourns_3266W_Vertical, symbol Device:R_Potentiometer_Trim
- removed U204: ADA4895-1ARJZ, Package_TO_SOT_SMD:SOT-23-6_Handsoldering, symbol Amplifier_Operational:ADA4807-1
- removed U205: AD797BRZ, Package_SO:SOIC-8_3.9x4.9mm_P1.27mm, symbol Amplifier_Operational:AD797
- added U204, U210: LMH6611, Package_TO_SOT_SMD:TSOT-23-6_HandSoldering, symbol Amplifier_Operational:LMH6611
- added U205: LT5400-4, Package_SO:MSOP-8-1EP_3x3mm_P0.65mm_EP1.73x1.85mm_ThermalVias, symbol AD4030:LT5400
- added U211: LT5400-8, Package_SO:MSOP-8-1EP_3x3mm_P0.65mm_EP1.73x1.85mm_ThermalVias, symbol AD4030:LT5400
- added U212: NC7SZ125M5X, Package_TO_SOT_SMD:SOT-23-5_HandSoldering, symbol 74xGxx:NC7SZ125M5X
- C232: value 50p -> 0.1u
- R201, R202, R203, R204, R205, R206, R207, R208, R209, R210: value 1M/0.1% -> 2M/0.1%
Connections:
- net +5VA: now also U204.5 (~{DISABLE}), U204.6 (V+), U210.5 (~{DISABLE}), U210.6 (V+)
- net -5VA: now also U204.2 (V-), U210.2 (V-)
- net GND: now also C232.2, U212.1 (~{OE}), U212.3 (GND)
- net GNDA: now also U205.3, U205.4, U205.9, U211.2, U211.9
- net at U201.2: now also U205.1, U205.2
- net at U201.10: now also U204.1, U211.4; no longer C232.2
- net +3.3V: now reaches C232.1
- net +3.3V: now also U212.5 (VCC)
- net at U207.7, U207.8, U209.1: now also U210.3 (+)
- net at U207.5, U207.6, U209.4: now also U210.4 (-)
- net at R236.1, U209.5: now also U210.1
- net GAIN_x3 renamed GAIN_x20
- net Gain_x10-x100: no longer names the net of R233.2
- net Gain_x10-x100: now also U212.4 (Y)
- new net: U204.3 (+), U205.7, U205.8, U211.1
- new net: U211.7, U211.8
- new net: U211.5, U211.6
- new net: U204.4 (-), U205.5, U205.6, U211.3
- new net Gain_x10: U212.2 (A)
Other:
- note added: "Gain x20"
- note removed: "Gain x2.5"
- moved on the sheet: C201, C202, C203, C204, C205, C206, C207, C208, C209, C210, C211, C212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

Commit message: Hardware
Parts:
- removed U212: NC7SZ125M5X, Package_TO_SOT_SMD:SOT-23-5_HandSoldering, symbol 74xGxx:NC7SZ125M5X
- added C233: 0.1u, Capacitor_SMD:C_0603_1608Metric_Pad1.08x0.95mm_HandSolder, symbol Device:C
- added U209: TXB0101DBV, Package_TO_SOT_SMD:SOT-23-6, symbol Logic_LevelTranslator:TXB0101DBV
- J201: footprint (none) -> AD4030:1710072
- R222: renamed from R236; footprint (none) -> Resistor_SMD:R_0603_1608Metric_Pad0.98x0.95mm_HandSolder
- R223: renamed from R238; footprint (none) -> Resistor_SMD:R_0603_1608Metric_Pad0.98x0.95mm_HandSolder
- renumbered C217 to C215, C215 to C216, C216 to C217, C220 to C218, C218 to C219, C219 to C220, C223 to C221, C221 to C222, C222 to C223, C225 to C224, C224 to C225, R213 to R211, R214 to R212, R217 to R213, R218 to R214, R219 to R215, R220 to R216, R221 to R217, R222 to R218, R223 to R219, R225 to R220, R233 to R221, U206 to U202, U202 to U203, U203 to U204, U208 to U205, U207 to U206, U209 to U207, U205 to U208, U211 to U210, U210 to U211, U204 to U212
Connections:
- net +3.3V: now also U209.6 (V_{CCB})
- net GND: now also C233.2, U209.2 (GND)
- net Gain_x10: now also U209.3 (A)
- net at R221.2: now also U209.4 (B)
- new net VIO: C233.1, U209.1 (V_{CCA}), U209.5 (OE)
Other:
- moved on the sheet: C205, C208, C211, C214, C215, C218, C221, C224, C226, C229, C232, U202E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
