File: AD4030/Hardware/AD4030-Voltage/DIFF.kicad_sch (KiCad schematic)
At the start: 75 parts, among them J201 1710072, K201 UMS05-1A80-75D, Q201 MMBT3904, U201 ADG5236BCPZ, U202 LT5400-1, U203 ADA4817-1ARD, U204 ADA4817-1ARD, U205 LT5400-4, U206 LT5400-4, U207 LT5400-4, U208 LT5400-4, U209 TXB0101DBV, U210 LT5400-8, U211 LMH6611, U212 LMH6611

Commit message: Hardware and update to 2024.1
Parts:
- R211, R212: footprint Resistor_SMD:R_1206_3216Metric_Pad1.30x1.75mm_HandSolder -> Resistor_SMD:R_0603_1608Metric_Pad0.98x0.95mm_HandSolder
- U211, U212: footprint Package_TO_SOT_SMD:TSOT-23-6_HandSoldering -> Package_TO_SOT_SMD:TSOT-23-6
Connections:
- net GNDA: now also C223.2; no longer C223.1
- net at C213.2, C217.2, C220.2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: now also C223.1; no longer C223.2
Other:
- moved on the sheet: C223
Changed lines of the file:
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@@
 			)
 		)
-		(property "Footprint" "Resistor_SMD:R_1206_3216Metric_Pad1.30x1.75mm_HandSolder"
+		(property "Footprint" "Resistor_SMD:R_0603_1608Metric_Pad0.98x0.95mm_HandSolder"
 			(at 94.742 116.84 90)
 			(effects
@@
 			)
 		)
-		(property "Footprint" "Resistor_SMD:R_1206_3216Metric_Pad1.30x1.75mm_HandSolder"
+		(property "Footprint" "Resistor_SMD:R_0603_1608Metric_Pad0.98x0.95mm_HandSolder"
 			(at 94.742 101.6 90)
 			(effects
@@
 	(symbol
 		(lib_id "Device:C_Trim")
-		(at 137.16 135.89 0)
+		(at 137.16 135.89 180)
 		(unit 1)
 		(exclude_from_sim no)
@@
 		(fields_autoplaced yes)
 		(property "Reference" "C223"
-			(at 140.97 134.3659 0)
+			(at 140.97 134.8739 0)
 			(effects
 				(font
 					(size 1.27 1.27)
 				)
-				(justify left)
+				(justify right)
 			)
 		)
 		(property "Value" "JR500"
-			(at 140.97 136.9059 0)
+			(at 140.97 137.4139 0)
 			(effects
 				(font
 					(size 1.27 1.27)
 				)
-				(justify left)
+				(justify right)
 			)
 		)
@@
 			)
 		)
-		(property "Footprint" "Package_TO_SOT_SMD:TSOT-23-6_HandSoldering"
+		(property "Footprint" "Package_TO_SOT_SMD:TSOT-23-6"
 			(at 341.63 123.19 0)
 			(effects
@@
 			)
 		)
-		(property "Footprint" "Package_TO_SOT_SMD:TSOT-23-6_HandSoldering"
+		(property "Footprint" "Package_TO_SOT_SMD:TSOT-23-6"
 			(at 278.13 115.57 0)
 			(effects

Commit message: Hardware
Parts:
- renumbered U210 to U209, U209 to U210
Connections:
- net GNDA is gone; now on net GND: C205.2, C208.2, C211.2, C214.2, C215.2, C216.2, C217.1, C218.2, C219.2, C220.1, C221.2, C222.2, C223.2, C224.2, C225.2, C226.2, C229.2, R216.1, RV201.2, U201.4 (GND), U202.9, U203.9 (EP), U204.9 (EP), U205.9, U206.9, U207.8, U207.9, U208.3, U208.4, U208.9, U209.2, U209.9

Commit message: Hardware design
Parts:
- U203, U204: value ADA4817-1ARD -> ADA4817-1ACP; footprint Package_SO:SOIC-8-1EP_3.9x4.9mm_P1.27mm_EP2.29x3mm -> Package_CSP:LFCSP-8-1EP_3x3mm_P0.5mm_EP1.45x1.74mm; symbol Amplifier_Operational:ADA4817-1ARD -> Amplifier_Operational:ADA4817-1ACP
Connections:
- net +5VA: now also U203.1 (~{PD}), U204.1 (~{PD}); no longer U203.7 (+V_{S}), U204.7 (+V_{S})
- net -5VA: now also U203.5 (-V_{S}), U204.5 (-V_{S}); no longer U203.4 (-V_{S}), U204.4 (-V_{S})
- net at C228.2, C231.1, R219.2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: now also U204.3 (-), U205.5, U205.6; no longer U204.2 (-), U205.3, U205.4
- net at U203.2 (FB), U205.7, U205.8: now also C230.1; no longer C230.2, K201.3
- net at R218.1: now also U204.4 (+); no longer U204.3 (+)
- net at U206.3, U206.4: now also U204.7; no longer U204.6
- net at U205.1, U205.2: now also C230.2, K201.3, U203.3 (-); no longer C230.1, U203.1 (FB)
- net at R217.2: now also U203.4 (+); no longer U203.3 (+)
- net at U206.1, U206.2: now also U203.7; no longer U203.6
- new net: C231.2, U204.2 (FB), U205.3, U205.4
Other:
- moved on the sheet: U205A, U205B, U205C, U205D
Changed lines of the file:
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@@
 	(symbol
 		(lib_id "AD4030:LT5400")
-		(at 208.28 129.54 270)
+		(at 208.28 129.54 90)
 		(unit 4)
 		(exclude_from_sim no)
@@
 					(size 1.27 1.27)
 				)
-				(justify left)
+				(justify right)
 			)
 		)
@@
 					(size 1.27 1.27)
 				)
-				(justify left)
+				(justify right)
 			)
 		)
@@
 		)
 		(property "Datasheet" "https://www.analog.com/media/en/technical-documentation/data-sheets/5400fc.pdf"
-			(at 208.28 129.032 0)
+			(at 208.28 130.048 0)
 			(effects
 				(font
@@
 	)
 	(symbol
-		(lib_id "Amplifier_Operational:ADA4817-1ARD")
+		(lib_id "Amplifier_Operational:ADA4817-1ACP")
 		(at 173.99 138.43 0)
 		(unit 1)
@@
 			)
 		)
-		(property "Value" "ADA4817-1ARD"
+		(property "Value" "ADA4817-1ACP"
 			(at 182.626 141.732 0)
 			(effects
@@
 			)
 		)
-		(property "Footprint" "Package_SO:SOIC-8-1EP_3.9x4.9mm_P1.27mm_EP2.29x3mm"
+		(property "Footprint" "Package_CSP:LFCSP-8-1EP_3x3mm_P0.5mm_EP1.45x1.74mm"
 			(at 173.99 137.16 0)
 			(effects
@@
 			)
 		)
-		(property "Description" "Single Low Noise, 1 GHz, Unity-gain stable, FastFET Op Amp, with power down, SOIC-8-1EP"
+		(property "Description" "Single Low Noise, 1 GHz, Unity-gain stable, FastFET Op Amp, with power down, LFCSP-8-1EP"
 			(at 173.99 138.43 0)
 			(effects
@@
 	)
 	(symbol
-		(lib_id "Amplifier_Operational:ADA4817-1ARD")
+		(lib_id "Amplifier_Operational:ADA4817-1ACP")
 		(at 173.99 80.01 0)
 		(mirror x)
@@
 			)
 		)
-		(property "Value" "ADA4817-1ARD"
+		(property "Value" "ADA4817-1ACP"
 			(at 182.626 76.708 0)
 			(effects
@@
 			)
 		)
-		(property "Footprint" "Package_SO:SOIC-8-1EP_3.9x4.9mm_P1.27mm_EP2.29x3mm"
+		(property "Footprint" "Package_CSP:LFCSP-8-1EP_3x3mm_P0.5mm_EP1.45x1.74mm"
 			(at 173.99 81.28 0)
 			(effects
@@
 			)
 		)
-		(property "Description" "Single Low Noise, 1 GHz, Unity-gain stable, FastFET Op Amp, with power down, SOIC-8-1EP"
+		(property "Description" "Single Low Noise, 1 GHz, Unity-gain stable, FastFET Op Amp, with power down, LFCSP-8-1EP"
 			(at 173.99 80.01 0)
 			(effects
@@
 	(symbol
 		(lib_id "AD4030:LT5400")
-		(at 193.04 129.54 270)
+		(at 193.04 129.54 90)
 		(unit 3)
 		(exclude_from_sim no)
@@
 					(size 1.27 1.27)
 				)
-				(justify left)
+				(justify right)
 			)
 		)
@@
 					(size 1.27 1.27)
 				)
-				(justify left)
+				(justify right)
 			)
 		)
@@
 		)
 		(property "Datasheet" "https://www.analog.com/media/en/technical-documentation/data-sheets/5400fc.pdf"
-			(at 193.04 129.032 0)
+			(at 193.04 130.048 0)
 			(effects
 				(font
@@
 	(symbol
 		(lib_id "AD4030:LT5400")
-		(at 193.04 88.9 270)
+		(at 193.04 88.9 90)
 		(unit 1)
 		(exclude_from_sim no)
@@
 					(size 1.27 1.27)
 				)
-				(justify left)
+				(justify right)
 			)
 		)
@@
 					(size 1.27 1.27)
 				)
-				(justify left)
+				(justify right)
 			)
 		)
@@
 		)
 		(property "Datasheet" "https://www.analog.com/media/en/technical-documentation/data-sheets/5400fc.pdf"
-			(at 193.04 88.392 0)
+			(at 193.04 89.408 0)
 			(effects
 				(font
@@
 	(symbol
 		(lib_id "AD4030:LT5400")
-		(at 208.28 88.9 270)
+		(at 208.28 88.9 90)
 		(unit 2)
 		(exclude_from_sim no)
@@
 					(size 1.27 1.27)
 				)
-				(justify left)
+				(justify right)
 			)
 		)
@@
 					(size 1.27 1.27)
 				)
-				(justify left)
+				(justify right)
 			)
 		)
@@
 		)
 		(property "Datasheet" "https://www.analog.com/media/en/technical-documentation/data-sheets/5400fc.pdf"
-			(at 208.28 88.392 0)
+			(at 208.28 89.408 0)
 			(effects
 				(font

Commit message: PCB layout
Connections:
- net +3.3V is gone; now on net +5V: C232.1, U210.6 (V_{CCB})
Other:
- note added: "1/500"
- note removed: "1/250"
- moved on the sheet: J201
Changed lines of the file:
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@@
 	(wire
 		(pts
-			(xy 30.48 87.63) (xy 30.48 107.95)
-		)
-		(stroke
-			(width 0)
-			(type default)
-		)
-	)
-	(wire
-		(pts
 			(xy 171.45 129.54) (xy 171.45 130.81)
 		)
@@
 	(wire
 		(pts
-			(xy 30.48 110.49) (xy 30.48 130.81)
-		)
-		(stroke
-			(width 0)
-			(type default)
-		)
-	)
-	(wire
-		(pts
 			(xy 171.45 88.9) (xy 171.45 87.63)
 		)
@@
 	(wire
 		(pts
+			(xy 30.48 110.49) (xy 30.48 130.81)
+		)
+		(stroke
+			(width 0)
+			(type default)
+		)
+	)
+	(wire
+		(pts
 			(xy 311.15 106.68) (xy 311.15 90.17)
 		)
@@
 	(wire
 		(pts
-			(xy 26.67 110.49) (xy 30.48 110.49)
+			(xy 29.21 110.49) (xy 30.48 110.49)
 		)
 		(stroke
@@
 	(wire
 		(pts
-			(xy 26.67 107.95) (xy 30.48 107.95)
+			(xy 29.21 107.95) (xy 30.48 107.95)
 		)
 		(stroke
@@
 	(wire
 		(pts
+			(xy 30.48 87.63) (xy 30.48 107.95)
+		)
+		(stroke
+			(width 0)
+			(type default)
+		)
+	)
+	(wire
+		(pts
 			(xy 316.23 139.7) (xy 316.23 140.97)
 		)
@@
 		)
 	)
-	(text "1/250"
+	(text "1/500"
 		(exclude_from_sim no)
 		(at 62.992 62.23 0)
@@
 	)
 	(symbol
+		(lib_id "power:+5V")
+		(at 182.88 255.27 0)
+		(unit 1)
+		(exclude_from_sim no)
+		(in_bom yes)
+		(on_board yes)
+		(dnp no)
+		(fields_autoplaced yes)
+		(property "Reference" "#PWR0225"
+			(at 182.88 259.08 0)
+			(effects
+				(font
+					(size 1.27 1.27)
+				)
+				(hide yes)
+			)
+		)
+		(property "Value" "+5V"
+			(at 182.88 250.19 0)
+			(effects
+				(font
+					(size 1.27 1.27)
+				)
+			)
+		)
+		(property "Footprint" ""
+			(at 182.88 255.27 0)
+			(effects
+				(font
+					(size 1.27 1.27)
+				)
+				(hide yes)
+			)
+		)
+		(property "Datasheet" ""
+			(at 182.88 255.27 0)
+			(effects
+				(font
+					(size 1.27 1.27)
+				)
+				(hide yes)
+			)
+		)
+		(property "Description" "Power symbol creates a global label with name \"+5V\""
+			(at 182.88 255.27 0)
+			(effects
+				(font
+					(size 1.27 1.27)
+				)
+				(hide yes)
+			)
+		)
+		(pin "1"
+		)
+		(instances
+			(project "AD4030-Voltage"
+				(path "/af28bfe6-a5ae-47dd-9259-97a6edcec559/3bc08f1b-cd51-4945-94b2-c6f7f3a0b515"
+					(reference "#PWR0225")
+					(unit 1)
+				)
+			)
+		)
+	)
+	(symbol
 		(lib_id "power:+5VA")
 		(at 77.47 255.27 0)
@@
 	)
 	(symbol
-		(lib_id "power:+3.3V")
-		(at 270.51 143.51 0)
-		(unit 1)
-		(exclude_from_sim no)
-		(in_bom yes)
-		(on_board yes)
-		(dnp no)
-		(fields_autoplaced yes)
-		(property "Reference" "#PWR0237"
-			(at 270.51 147.32 0)
-			(effects
-				(font
-					(size 1.27 1.27)
-				)
-				(hide yes)
-			)
-		)
-		(property "Value" "+3.3V"
-			(at 270.51 138.43 0)
-			(effects
-				(font
-					(size 1.27 1.27)
-				)
-			)
-		)
-		(property "Footprint" ""
-			(at 270.51 143.51 0)
-			(effects
-				(font
-					(size 1.27 1.27)
-				)
-				(hide yes)
-			)
-		)
-		(property "Datasheet" ""
-			(at 270.51 143.51 0)
-			(effects
-				(font
-					(size 1.27 1.27)
-				)
-				(hide yes)
-			)
-		)
-		(property "Description" "Power symbol creates a global label with name \"+3.3V\""
-			(at 270.51 143.51 0)
-			(effects
-				(font
-					(size 1.27 1.27)
-				)
-				(hide yes)
-			)
-		)
-		(pin "1"
-		)
-		(instances
-			(project ""
-				(path "/af28bfe6-a5ae-47dd-9259-97a6edcec559/3bc08f1b-cd51-4945-94b2-c6f7f3a0b515"
-					(reference "#PWR0237")
-					(unit 1)
-				)
-			)
-		)
-	)
-	(symbol
 		(lib_id "power:-5VA")
 		(at 336.55 124.46 180)
@@
 	)
 	(symbol
-		(lib_id "power:+3.3V")
-		(at 182.88 255.27 0)
-		(unit 1)
-		(exclude_from_sim no)
-		(in_bom yes)
-		(on_board yes)
-		(dnp no)
-		(fields_autoplaced yes)
-		(property "Reference" "#PWR0225"
-			(at 182.88 259.08 0)
-			(effects
-				(font
-					(size 1.27 1.27)
-				)
-				(hide yes)
-			)
-		)
-		(property "Value" "+3.3V"
-			(at 182.88 250.19 0)
-			(effects
-				(font
-					(size 1.27 1.27)
-				)
-			)
-		)
-		(property "Footprint" ""
-			(at 182.88 255.27 0)
-			(effects
-				(font
-					(size 1.27 1.27)
-				)
-				(hide yes)
-			)
-		)
-		(property "Datasheet" ""
-			(at 182.88 255.27 0)
-			(effects
-				(font
-					(size 1.27 1.27)
-				)
-				(hide yes)
-			)
-		)
-		(property "Description" "Power symbol creates a global label with name \"+3.3V\""
-			(at 182.88 255.27 0)
-			(effects
-				(font
-					(size 1.27 1.27)
-				)
-				(hide yes)
-			)
-		)
-		(pin "1"
-		)
-		(instances
-			(project ""
-				(path "/af28bfe6-a5ae-47dd-9259-97a6edcec559/3bc08f1b-cd51-4945-94b2-c6f7f3a0b515"
-					(reference "#PWR0225")
-					(unit 1)
-				)
-			)
-		)
-	)
-	(symbol
 		(lib_id "power:GND")
 		(at 177.8 72.39 180)
@@
 	)
 	(symbol
+		(lib_id "power:+5V")
+		(at 270.51 143.51 0)
+		(unit 1)
+		(exclude_from_sim no)
+		(in_bom yes)
+		(on_board yes)
+		(dnp no)
+		(fields_autoplaced yes)
+		(property "Reference" "#PWR0237"
+			(at 270.51 147.32 0)
+			(effects
+				(font
+					(size 1.27 1.27)
+				)
+				(hide yes)
+			)
+		)
+		(property "Value" "+5V"
+			(at 270.51 138.43 0)
+			(effects
+				(font
+					(size 1.27 1.27)
+				)
+			)
+		)
+		(property "Footprint" ""
+			(at 270.51 143.51 0)
+			(effects
+				(font
+					(size 1.27 1.27)
+				)
+				(hide yes)
+			)
+		)
+		(property "Datasheet" ""
+			(at 270.51 143.51 0)
+			(effects
+				(font
+					(size 1.27 1.27)
+				)
+				(hide yes)
+			)
+		)
+		(property "Description" "Power symbol creates a global label with name \"+5V\""
+			(at 270.51 143.51 0)
+			(effects
+				(font
+					(size 1.27 1.27)
+				)
+				(hide yes)
+			)
+		)
+		(pin "1"
+		)
+		(instances
+			(project "AD4030-Voltage"
+				(path "/af28bfe6-a5ae-47dd-9259-97a6edcec559/3bc08f1b-cd51-4945-94b2-c6f7f3a0b515"
+					(reference "#PWR0237")
+					(unit 1)
+				)
+			)
+		)
+	)
+	(symbol
 		(lib_id "Device:C")
 		(at 87.63 130.81 90)
@@
 	(symbol
 		(lib_id "Connector_Generic:Conn_01x02")
-		(at 21.59 107.95 0)
+		(at 24.13 107.95 0)
 		(mirror y)
 		(unit 1)
@@
 		(dnp no)
 		(property "Reference" "J201"
-			(at 21.59 102.362 0)
+			(at 24.13 102.362 0)
 			(effects
 				(font
@@
 		)
 		(property "Value" "1710072"
-			(at 21.59 104.902 0)
+			(at 24.13 104.902 0)
 			(effects
 				(font
@@
 		)
 		(property "Footprint" "AD4030:1710072"
-			(at 21.59 107.95 0)
+			(at 24.13 107.95 0)
 			(effects
 				(font
@@
 		)
 		(property "Datasheet" "~"
-			(at 21.59 107.95 0)
+			(at 24.13 107.95 0)
 			(effects
 				(font
@@
 		)
 		(property "Description" ""
-			(at 21.59 107.95 0)
+			(at 24.13 107.95 0)
 			(effects
 				(font

Commit message: PCB layout
Parts:
- R211, R212: value 91 -> 91/.1%
- U211, U212: value LMH6611 -> LMH6611MK
- renumbered U202 to RN202, U205 to RN205, U206 to RN206, U207 to RN207, U208 to RN208, U209 to RN209

Commit message: PCB layout
Parts:
- removed U201: ADG5236BCPZ, Package_DFN_QFN:QFN-16-1EP_4x4mm_P0.65mm_EP2.5x2.5mm_ThermalVias, symbol AD4030:ADG5236BCPZ
- added C233, C235: 0.1u, Capacitor_SMD:C_0603_1608Metric_Pad1.08x0.95mm_HandSolder, symbol Device:C
- added U201: ADG1436YCPZ, Package_DFN_QFN:QFN-16-1EP_4x4mm_P0.65mm_EP2.5x2.5mm_ThermalVias, symbol AD4030:ADG1436YCPZ
- added U207: TXB0101DBV, Package_TO_SOT_SMD:SOT-23-6, symbol Logic_LevelTranslator:TXB0101DBV
- renumbered C233 to C234, RN202 to RN201, RN205 to RN202, RN206 to RN203, RN207 to RN204, RN208 to RN205, RN209 to RN206, U203 to U202, U204 to U203, U210 to U204, U211 to U205, U212 to U206
Connections:
- net +5V: now also C233.1, U201.12 (EN), U207.6 (V_{CCB})
- net +5VA: now also U201.11 (VDD)
- net -5VA: now also U201.17 (EP), U201.3 (VSS)
- net GAIN_x20: now also U207.3 (A)
- net GND: now also C233.2, C235.2, U201.4 (GND), U207.2 (GND)
- net VIO: now also C235.1, U207.1 (V_{CCA}), U207.5 (OE)
- net at RN205.1, RN205.2: now also U201.2
- net at RN206.4, U206.1: now also U201.10
- net at R223.1: now also U201.9
- net at R222.2: now also U201.1
- new net: U201.16, U201.8
- new net SW_GAIN_x20: U201.15, U201.6, U207.4 (B)
Other:
- moved on the sheet: C205, C208, C211, C214, C215, C218, C221, C224, C226, C229, C232, C234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
