File: AD4030/Hardware/AD4030-Voltage/Isolation.kicad_sch (KiCad schematic)
At the start: 3 parts, among them U401 ADuM260N, U402 ADuM260N, U403 TSR1-2450E

Commit message: Hardware
Parts:
- removed U403: TSR1-2450E, Converter_DCDC:Converter_DCDC_TRACO_TSR1-xxxxE_THT, symbol Regulator_Switching:TSR1-2450E
- added C401, C403, C405, C406: 0.1u, symbol Device:C
- added C402, C404, C407, C408: 1u, symbol Device:C
- added J401: Conn_01x08, symbol Connector_Generic:Conn_01x08
- added J402: Conn_01x10, symbol Connector_Generic:Conn_01x10
- added R401, R402, R403, R404, R405, R406, R407, R408, R409, R410, R411: 50, symbol Device:R
Connections:
- net GND: now also C405.2, C406.2, C407.2, C408.2
- net GNDS: now also C401.2, C402.2, C403.2, C404.2, J402.7 (Pin_7)
- net VCCQ: now also C401.1, C402.1, C403.1, C404.1
- net VIO: now also C405.1, C406.1, C407.1, C408.1
- net at U401.11 (VOE): now also R405.1
- net at U401.12 (VOD): now also R404.1
- net at U401.13 (VOC): now also R403.1
- net at U401.14 (VOB): now also R402.1
- net at U401.15 (VOA): now also R401.1
- net Gain_x10-x100: now reaches U402.10 (VOF)
- net GAIN_x3: now reaches U402.11 (VOE)
- net at U402.2 (VIA): now also R406.1
- net at U402.3 (VIB): now also R407.1
- net at U402.4 (VIC): now also R408.1
- net at U402.5 (VID): now also R409.1
- net at U402.6 (VIE): now also R410.1
- net at U402.7 (VIF): now also R411.1
- new net IO0: J401.1 (Pin_1), R401.2
- new net IO1: J401.2 (Pin_2), R402.2
- new net IO10: J402.3 (Pin_3), R411.2
- new net IO2: J401.3 (Pin_3), R403.2
- new net IO3: J401.4 (Pin_4), R404.2
- new net IO4: J401.5 (Pin_5), R405.2
- new net IO5: J401.6 (Pin_6), R406.2
- new net IO6: J401.7 (Pin_7), R407.2
- new net IO7: J401.8 (Pin_8), R408.2
- new net IO8: J402.1 (Pin_1), R409.2
- new net IO9: J402.2 (Pin_2), R410.2
- no-connect marks 6 -> 8
Other:
- note removed: "LT1763"
- moved on the sheet: U401, U402

Commit message: Hardware
Parts:
- C401: renamed from C405; footprint (none) -> Capacitor_SMD:C_0603_1608Metric_Pad1.08x0.95mm_HandSolder
- C402: renamed from C406; footprint (none) -> Capacitor_SMD:C_0603_1608Metric_Pad1.08x0.95mm_HandSolder
- C403: renamed from C407; footprint (none) -> Capacitor_SMD:C_0603_1608Metric_Pad1.08x0.95mm_HandSolder
- C404: renamed from C408; footprint (none) -> Capacitor_SMD:C_0603_1608Metric_Pad1.08x0.95mm_HandSolder
- C405: renamed from C403; footprint (none) -> Capacitor_SMD:C_0603_1608Metric_Pad1.08x0.95mm_HandSolder
- C406: renamed from C401; footprint (none) -> Capacitor_SMD:C_0603_1608Metric_Pad1.08x0.95mm_HandSolder
- C407: renamed from C404; footprint (none) -> Capacitor_SMD:C_0603_1608Metric_Pad1.08x0.95mm_HandSolder
- C408: renamed from C402; footprint (none) -> Capacitor_SMD:C_0603_1608Metric_Pad1.08x0.95mm_HandSolder
- J401: footprint (none) -> Connector_PinHeader_2.54mm:PinHeader_1x08_P2.54mm_Vertical
- J402: footprint (none) -> Connector_PinHeader_2.54mm:PinHeader_1x10_P2.54mm_Vertical
- R401, R402, R403, R404, R405, R406, R407, R408, R409, R410, R411: footprint (none) -> Resistor_SMD:R_0603_1608Metric_Pad0.98x0.95mm_HandSolder

Commit message: Hardware and started to create simulation.
Parts:
- added J403, J404: PMOD, Connector_PinHeader_2.54mm:PinHeader_2x06_P2.54mm_Horizontal, symbol Connector_Generic:Conn_02x06_Top_Bottom
- added R412: 50, Resistor_SMD:R_0603_1608Metric_Pad0.98x0.95mm_HandSolder, symbol Device:R
Connections:
- net IO5 is gone; now on net CONN_100MHz: J401.6 (Pin_6), R406.2
- net IO7 is gone; now on net CONN_SDI: J401.8 (Pin_8), R408.2
- net GNDS: now also J403.2 (Pin_2), J403.8 (Pin_8), J404.2 (Pin_2), J404.8 (Pin_8)
- net at R408.1: now also J403.9 (Pin_9); no longer U402.4 (VIC)
- net CONN_CNV: now reaches R411.1
- net CONN_CNV: now also J402.2 (Pin_2), U402.5 (VID); no longer U402.7 (VIF)
- net CONN_SDO0: now reaches R401.1, U401.15 (VOA)
- net CONN_SDO0: now also J401.1 (Pin_1)
- net at R410.1: now also J404.12 (Pin_12); no longer U402.6 (VIE)
- net CONN_SCK: now reaches R409.1
- net CONN_SCK: now also J402.1 (Pin_1), U402.4 (VIC); no longer U402.5 (VID)
- net CONN_SDO2: now reaches R403.1, U401.13 (VOC)
- net CONN_SDO2: now also J401.3 (Pin_3)
- net CONN_100MHz: now reaches U401.10 (VOF)
- net CONN_BUSY: now reaches R405.1, U401.11 (VOE)
- net CONN_BUSY: now also J401.5 (Pin_5)
- net at R404.1: now also J403.11 (Pin_11); no longer U401.12 (VOD)
- net at R402.1: now also J403.12 (Pin_12); no longer U401.14 (VOB)
- net CLK_100MHz: now reaches U401.7 (VIF)
- net CONN_SDI: now reaches U402.3 (VIB)
- net CONN_SDI: no longer R407.1
- net at R406.1: now also J403.10 (Pin_10); no longer U402.2 (VIA)
- net CONN_GAIN_x10-100: now reaches J402.4 (Pin_4)
- net CONN_GAIN_x10-100: now also U402.7 (VIF), R412.2
- net IO0: no longer names the net of R401.2
- net IO0: now also J403.6 (Pin_6); no longer J401.1 (Pin_1)
- net IO1 renamed CONN_SDO1
- net CONN_SDO1: now also U401.14 (VOB)
- net IO10: no longer names the net of R411.2
- net IO10: now also J404.5 (Pin_5); no longer J402.3 (Pin_3)
- net IO2: no longer names the net of R403.2
- net IO2: now also J403.5 (Pin_5); no longer J401.3 (Pin_3)
- net IO3 renamed CONN_SDO3
- net CONN_SDO3: now also U401.12 (VOD)
- net IO4: no longer names the net of R405.2
- net IO4: now also J403.4 (Pin_4); no longer J401.5 (Pin_5)
- net IO6: no longer names the net of R407.2
- net IO6: now also J403.3 (Pin_3); no longer J401.7 (Pin_7)
- net IO8: no longer names the net of R409.2
- net IO8: now also J404.6 (Pin_6); no longer J402.1 (Pin_1)
- net IO9 renamed CONN_GAIN_x3
- net CONN_GAIN_x3: now also J402.3 (Pin_3), U402.6 (VIE); no longer J402.2 (Pin_2)
- new net: J404.11 (Pin_11), R412.1
- new net CONN_~{CS}: J401.7 (Pin_7), R407.1, U402.2 (VIA)
- no-connect marks 8 -> 13
Other:
- moved on the sheet: C401, C402, C403, C404, C405, C406, C407, C408, J401, J402, R401, R402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

Commit message: Hardware design and simulation
Connections:
- net CONN_GAIN_x10-100 renamed CONN_GAIN_x10
- net CONN_GAIN_x3 renamed CONN_GAIN_x20
- net GAIN_x3 renamed GAIN_x20
- net Gain_x10-x100 renamed Gain_x10
Changed lines of the file:
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@@
 		)
 	)
-	(label "CONN_GAIN_x3"
+	(label "CONN_GAIN_x20"
 		(at 133.35 113.03 0)
 		(fields_autoplaced yes)
@@
 		)
 	)
-	(label "CONN_GAIN_x10-100"
+	(label "CONN_GAIN_x10"
 		(at 133.35 115.57 0)
 		(fields_autoplaced yes)
@@
 		)
 	)
-	(label "CONN_GAIN_x10-100"
+	(label "CONN_GAIN_x10"
 		(at 266.7 88.9 180)
 		(fields_autoplaced yes)
@@
 		)
 	)
-	(label "CONN_GAIN_x3"
+	(label "CONN_GAIN_x20"
 		(at 266.7 86.36 180)
 		(fields_autoplaced yes)
@@
 		)
 	)
-	(hierarchical_label "GAIN_x3"
+	(hierarchical_label "GAIN_x20"
 		(shape output)
 		(at 71.12 113.03 180)
@@
 		)
 	)
-	(hierarchical_label "Gain_x10-x100"
+	(hierarchical_label "Gain_x10"
 		(shape output)
 		(at 71.12 115.57 180)

Commit message: Hardware
Parts:
- R401, R412: footprint Resistor_SMD:R_0603_1608Metric_Pad0.98x0.95mm_HandSolder -> Resistor_SMD:R_0402_1005Metric_Pad0.72x0.64mm_HandSolder
- R402: renamed from R403; footprint Resistor_SMD:R_0603_1608Metric_Pad0.98x0.95mm_HandSolder -> Resistor_SMD:R_0402_1005Metric_Pad0.72x0.64mm_HandSolder
- R403: renamed from R405; footprint Resistor_SMD:R_0603_1608Metric_Pad0.98x0.95mm_HandSolder -> Resistor_SMD:R_0402_1005Metric_Pad0.72x0.64mm_HandSolder
- R404: renamed from R407; footprint Resistor_SMD:R_0603_1608Metric_Pad0.98x0.95mm_HandSolder -> Resistor_SMD:R_0402_1005Metric_Pad0.72x0.64mm_HandSolder
- R405: renamed from R409; footprint Resistor_SMD:R_0603_1608Metric_Pad0.98x0.95mm_HandSolder -> Resistor_SMD:R_0402_1005Metric_Pad0.72x0.64mm_HandSolder
- R406: renamed from R411; footprint Resistor_SMD:R_0603_1608Metric_Pad0.98x0.95mm_HandSolder -> Resistor_SMD:R_0402_1005Metric_Pad0.72x0.64mm_HandSolder
- R407: renamed from R402; footprint Resistor_SMD:R_0603_1608Metric_Pad0.98x0.95mm_HandSolder -> Resistor_SMD:R_0402_1005Metric_Pad0.72x0.64mm_HandSolder
- R408: renamed from R404; footprint Resistor_SMD:R_0603_1608Metric_Pad0.98x0.95mm_HandSolder -> Resistor_SMD:R_0402_1005Metric_Pad0.72x0.64mm_HandSolder
- R409: renamed from R406; footprint Resistor_SMD:R_0603_1608Metric_Pad0.98x0.95mm_HandSolder -> Resistor_SMD:R_0402_1005Metric_Pad0.72x0.64mm_HandSolder
- R410: renamed from R408; footprint Resistor_SMD:R_0603_1608Metric_Pad0.98x0.95mm_HandSolder -> Resistor_SMD:R_0402_1005Metric_Pad0.72x0.64mm_HandSolder
- R411: renamed from R410; footprint Resistor_SMD:R_0603_1608Metric_Pad0.98x0.95mm_HandSolder -> Resistor_SMD:R_0402_1005Metric_Pad0.72x0.64mm_HandSolder
- renumbered C402 to C401, C404 to C402, C401 to C403, C403 to C404, C406 to C405, C408 to C406, C405 to C407, C407 to C408

Commit message: Hardware and update to 2024.1
Parts:
- removed J402: Conn_01x10, Connector_PinHeader_2.54mm:PinHeader_1x10_P2.54mm_Vertical, symbol Connector_Generic:Conn_01x10
- added J405: Conn_01x07, Connector_PinHeader_2.54mm:PinHeader_1x07_P2.54mm_Vertical_SMD_Pin1Right, symbol Connector_Generic:Conn_01x07
- J401: footprint Connector_PinHeader_2.54mm:PinHeader_1x08_P2.54mm_Vertical -> Connector_PinHeader_2.54mm:PinHeader_1x08_P2.54mm_Vertical_SMD_Pin1Right
Connections:
- net CONN_CNV: now also J405.2 (Pin_2)
- net CONN_GAIN_x10: now also J405.4 (Pin_4)
- net CONN_GAIN_x20: now also J405.3 (Pin_3)
- net CONN_SCK: now also J405.1 (Pin_1)
- net GNDS: now also J405.7 (Pin_7)
- no-connect marks 13 -> 10
Changed lines of the file:
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@@
 	)
 	(no_connect
-		(at 153.67 125.73)
-	)
-	(no_connect
 		(at 219.71 91.44)
 	)
@@
 	)
 	(no_connect
-		(at 153.67 128.27)
-	)
-	(no_connect
 		(at 219.71 99.06)
 	)
@@
 	)
 	(no_connect
-		(at 153.67 130.81)
-	)
-	(no_connect
 		(at 232.41 93.98)
 	)
@@
 	)
 	(symbol
+		(lib_id "Connector_Generic:Conn_01x07")
+		(at 158.75 115.57 0)
+		(unit 1)
+		(exclude_from_sim no)
+		(in_bom yes)
+		(on_board yes)
+		(dnp no)
+		(fields_autoplaced yes)
+		(property "Reference" "J405"
+			(at 161.29 114.2999 0)
+			(effects
+				(font
+					(size 1.27 1.27)
+				)
+				(justify left)
+			)
+		)
+		(property "Value" "Conn_01x07"
+			(at 161.29 116.8399 0)
+			(effects
+				(font
+					(size 1.27 1.27)
+				)
+				(justify left)
+			)
+		)
+		(property "Footprint" "Connector_PinHeader_2.54mm:PinHeader_1x07_P2.54mm_Vertical_SMD_Pin1Right"
+			(at 158.75 115.57 0)
+			(effects
+				(font
+					(size 1.27 1.27)
+				)
+				(hide yes)
+			)
+		)
+		(property "Datasheet" "~"
+			(at 158.75 115.57 0)
+			(effects
+				(font
+					(size 1.27 1.27)
+				)
+				(hide yes)
+			)
+		)
+		(property "Description" "Generic connector, single row, 01x07, script generated (kicad-library-utils/schlib/autogen/connector/)"
+			(at 158.75 115.57 0)
+			(effects
+				(font
+					(size 1.27 1.27)
+				)
+				(hide yes)
+			)
+		)
+		(pin "6"
+		)
+		(pin "2"
+		)
+		(pin "4"
+		)
+		(pin "5"
+		)
+		(pin "7"
+		)
+		(pin "1"
+		)
+		(pin "3"
+		)
+		(instances
+			(project ""
+				(path "/af28bfe6-a5ae-47dd-9259-97a6edcec559/c043c7b2-3c43-41f1-9746-1c7b8c419471"
+					(reference "J405")
+					(unit 1)
+				)
+			)
+		)
+	)
+	(symbol
 		(lib_id "Device:R")
 		(at 210.82 88.9 90)
@@
 	)
 	(symbol
-		(lib_id "Connector_Generic:Conn_01x10")
-		(at 158.75 118.11 0)
-		(unit 1)
-		(exclude_from_sim no)
-		(in_bom yes)
-		(on_board yes)
-		(dnp no)
-		(fields_autoplaced yes)
-		(property "Reference" "J402"
-			(at 161.29 118.1099 0)
-			(effects
-				(font
-					(size 1.27 1.27)
-				)
-				(justify left)
-			)
-		)
-		(property "Value" "Conn_01x10"
-			(at 161.29 120.6499 0)
-			(effects
-				(font
-					(size 1.27 1.27)
-				)
-				(justify left)
-			)
-		)
-		(property "Footprint" "Connector_PinHeader_2.54mm:PinHeader_1x10_P2.54mm_Vertical"
-			(at 158.75 118.11 0)
-			(effects
-				(font
-					(size 1.27 1.27)
-				)
-				(hide yes)
-			)
-		)
-		(property "Datasheet" "~"
-			(at 158.75 118.11 0)
-			(effects
-				(font
-					(size 1.27 1.27)
-				)
-				(hide yes)
-			)
-		)
-		(property "Description" "Generic connector, single row, 01x10, script generated (kicad-library-utils/schlib/autogen/connector/)"
-			(at 158.75 118.11 0)
-			(effects
-				(font
-					(size 1.27 1.27)
-				)
-				(hide yes)
-			)
-		)
-		(pin "3"
-		)
-		(pin "2"
-		)
-		(pin "1"
-		)
-		(pin "7"
-		)
-		(pin "10"
-		)
-		(pin "8"
-		)
-		(pin "5"
-		)
-		(pin "4"
-		)
-		(pin "9"
-		)
-		(pin "6"
-		)
-		(instances
-			(project ""
-				(path "/af28bfe6-a5ae-47dd-9259-97a6edcec559/c043c7b2-3c43-41f1-9746-1c7b8c419471"
-					(reference "J402")
-					(unit 1)
-				)
-			)
-		)
-	)
-	(symbol
 		(lib_id "Connector_Generic:Conn_01x08")
 		(at 158.75 68.58 0)
@@
 			)
 		)
-		(property "Footprint" "Connector_PinHeader_2.54mm:PinHeader_1x08_P2.54mm_Vertical"
+		(property "Footprint" "Connector_PinHeader_2.54mm:PinHeader_1x08_P2.54mm_Vertical_SMD_Pin1Right"
 			(at 158.75 68.58 0)
 			(effects

Commit message: Hardware
Parts:
- renumbered J405 to J402
Changed lines of the file:
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@@
 		(dnp no)
 		(fields_autoplaced yes)
-		(property "Reference" "J405"
+		(property "Reference" "J402"
 			(at 161.29 114.2999 0)
 			(effects
@@
 			(project ""
 				(path "/af28bfe6-a5ae-47dd-9259-97a6edcec559/c043c7b2-3c43-41f1-9746-1c7b8c419471"
-					(reference "J405")
+					(reference "J402")
 					(unit 1)
 				)
