File: AD4030/Hardware/AD4030-Voltage/Power.kicad_sch (KiCad schematic)
At the start: 1 part, among them U501 TEC3-2419WI

Commit message: Hardware
Parts:
- added C501, C502, C504, C505: 10u/50V, symbol Device:C
- added C503, C521, C523, C524, C525: 10u, symbol Device:C
- added C506, C511, C513, C520, C522: 0.01u, symbol Device:C
- added C507, C509, C514, C517: 47u/25V, symbol Device:C
- added C508, C510, C512, C515, C516, C519: 1u, symbol Device:C
- added C518: 10u/25V, symbol Device:C
- added D501: BZX84C10LT1G, Package_TO_SOT_SMD:SOT-23, symbol Diode:BZX84Cxx
- added D502: 1N4148W, Diode_SMD:D_SOD-123, symbol Diode:1N4148W
- added F501: 1812L075/33DR, Fuse:Fuse_1812_4532Metric_Pad1.30x3.40mm_HandSolder, symbol Device:Fuse
- added FB501, FB502, FB503: FerriteBead_Small, symbol Device:FerriteBead_Small
- added J501: 1715721, TerminalBlock_Phoenix:TerminalBlock_Phoenix_MKDS-1,5-2_1x02_P5.00mm_Horizontal, symbol Connector_Generic:Conn_01x02
- added L501: TCK-141, symbol Device:L
- added L502: TCK-133, symbol Device:L
- added Q501: SI5618A, Package_TO_SOT_SMD:SOT-23, symbol Device:Q_PMOS_GSD
- added Q502: MMBT3904, Package_TO_SOT_SMD:SOT-23, symbol Transistor_BJT:MMBT3904
- added R501, R502: 100k, Resistor_SMD:R_0603_1608Metric_Pad0.98x0.95mm_HandSolder, symbol Device:R
- added R503, R504: R, symbol Device:R
- added R505: 5k11, symbol Device:R
- added R506: 10k, symbol Device:R
- added U502: TSR1-2450E, Converter_DCDC:Converter_DCDC_TRACO_TSR1-xxxxE_THT, symbol Regulator_Switching:TSR1-2450E
- added U503: LT1763CS8-1.8, Package_SO:SOIC-8_3.9x4.9mm_P1.27mm, symbol AD4030:LT1763CS8
- added U504, U505: LT1763CS8-ADJ, Package_SO:SOIC-8_3.9x4.9mm_P1.27mm, symbol AD4030:LT1763CS8
- added U506: LT1461DxS8-5, Package_SO:SOIC-8_3.9x4.9mm_P1.27mm, symbol Reference_Voltage:LT1461DxS8-5
- added U507: LT3032-5, Package_DFN_QFN:Linear_DE14MA, symbol Regulator_Linear:LT3032-5
- U501: value TEC3-2419WI -> TEC2-2419WI
Connections:
- net +9V: now also U501.6 (+VOUT), FB501.1, FB502.1, FB503.1
- net GND: now also U501.7 (-VOUT), C509.2, C510.2, C512.2, C514.2, C515.2, C516.2, C517.2, C518.2, C519.2, C521.2, C523.1, C524.2, C525.1, R506.2, U503.3 (GND), U503.6 (GND), U503.7 (GND), U505.3 (GND), U505.6 (GND), U505.7 (GND), U506.4 (GND), U507.4 (GND), U507.5 (GND)
- net GNDS: now reaches U501.1 (-VIN)
- net GNDS: now also C501.2, C502.2, C503.2, C504.2, C505.2, C507.2, C508.2, R504.2, U502.2 (GND), U504.3 (GND), U504.6 (GND), U504.7 (GND)
- net at U501.2 (+VIN): now also C505.1, L502.2
- new net: C516.1, FB502.2, U505.5 (~{SHDN}), U505.8 (IN)
- new net: R505.2, R506.1, U505.2 (SENSE/ADJ)
- new net: C513.2, U505.4 (BYP)
- new net: D502.1 (K), Q502.1 (B), R502.1
- new net: C501.1, C504.1, D501.3 (K), D502.2 (A), L501.1, L502.1, Q501.2 (S), Q502.2 (E)
- new net: C502.1, L501.2, U502.1 (Vin)
- new net: C511.2, U503.4 (BYP)
- new net: C512.1, FB501.2, U503.5 (~{SHDN}), U503.8 (IN)
- new net: R503.2, R504.1, U504.2 (SENSE/ADJ)
- new net: C522.1, U507.11 (BYPN)
- new net: C519.1, FB503.2, U506.2 (VIN)
- new net: D501.1 (A), Q501.1 (G), Q502.3 (C), R501.1
- new net: C506.2, U504.4 (BYP)
- new net: C503.1, U502.3 (Vout), U504.5 (~{SHDN}), U504.8 (IN)
- new net: F501.1, J501.1 (Pin_1)
- new net: F501.2, Q501.3 (D)
- new net: C524.1, U507.10 (~{SHDNN}), U507.12 (~{SHDNP}), U507.14 (INP)
- new net: J501.2 (Pin_2), R501.2, R502.2
- new net: C525.2, U507.6 (INN), U507.9 (INN)
- new net: C520.2, U507.3 (BYPP)
- new net +1V8: C509.1, C510.1, C511.1, U503.1 (OUT), U503.2 (SENSE/ADJ)
- new net +5VA: C520.1, C521.1, U507.1 (OUTP)
- new net +5VREF: C517.1, C518.1, U506.6 (VOUT)
- new net -5VA: C522.2, C523.2, U507.7 (OUTN)
- new net VCCQ: C506.1, C507.1, C508.1, R503.1, U504.1 (OUT)
- new net VIO: C513.1, C514.1, C515.1, R505.1, U505.1 (OUT)
- no-connect marks 1 -> 2
Other:
- note added: "Reverse voltage protection"
- note added: "https://www.analog.com/en/resources/technical-articles/bipolar-power-solutions-for-precision-test-and-measurement-systems.html"
- moved on the sheet: U501

Commit message: Hardware
Parts:
- removed C514: 47u/25V, symbol Device:C
- removed C516: 1u, symbol Device:C
- removed C524, C525: 10u, symbol Device:C
- removed L502: TCK-133, symbol Device:L
- removed R506: 10k, symbol Device:R
- removed U501: TEC2-2419WI, Converter_DCDC:Converter_DCDC_TRACO_TMR-xxxx_THT, symbol Converter_DCDC:TEC2-2419WI
- removed U505: LT1763CS8-ADJ, Package_SO:SOIC-8_3.9x4.9mm_P1.27mm, symbol AD4030:LT1763CS8
- added C501, C506, C507, C509, C510, C533: 10u/25V, Capacitor_SMD:C_1206_3216Metric_Pad1.33x1.80mm_HandSolder, symbol Device:C
- added C502, C503: 47n, Capacitor_SMD:C_0603_1608Metric_Pad1.08x0.95mm_HandSolder, symbol Device:C
- added C508: 1u, Capacitor_SMD:C_0603_1608Metric_Pad1.08x0.95mm_HandSolder, symbol Device:C
- added C512: 10u/50V, Capacitor_SMD:C_1210_3225Metric_Pad1.33x2.70mm_HandSolder, symbol Device:C
- added C522: 1u, Capacitor_SMD:C_0805_2012Metric_Pad1.18x1.45mm_HandSolder, symbol Device:C
- added C528: 0.01u, Capacitor_SMD:C_0603_1608Metric_Pad1.08x0.95mm_HandSolder, symbol Device:C
- added C530: 47u/25V, Capacitor_SMD:C_1210_3225Metric_Pad1.33x2.70mm_HandSolder, symbol Device:C
- added D503, D504: DFLS240, symbol Device:D_Schottky
- added L501: XAL4030-332ME, symbol Device:L_Small
- added L502: XAL4030-682ME, symbol Device:L_Small
- added L504: TCK-133, symbol Device:L
- added R501: 3k9, Resistor_SMD:R_0603_1608Metric_Pad0.98x0.95mm_HandSolder, symbol Device:R
- added R502: 8k2, Resistor_SMD:R_0603_1608Metric_Pad0.98x0.95mm_HandSolder, symbol Device:R
- added R504: 121k, Resistor_SMD:R_0603_1608Metric_Pad0.98x0.95mm_HandSolder, symbol Device:R
- added R507: 787k, Resistor_SMD:R_0603_1608Metric_Pad0.98x0.95mm_HandSolder, symbol Device:R
- added R508: R, Resistor_SMD:R_0603_1608Metric_Pad0.98x0.95mm_HandSolder, symbol Device:R
- added U501: TSR1-2450E, Converter_DCDC:Converter_DCDC_TRACO_TSR1-xxxxE_THT, symbol Regulator_Switching:TSR1-2450E
- added U502: ADP5070AREZ, Package_SO:ETSSOP-20-1EP_4.4x6.5mm_P0.65mm_EP3x4.2mm, symbol AD4030:ADP5070AREZ
- added U503: TSR1-2433E, Converter_DCDC:Converter_DCDC_TRACO_TSR1-xxxxE_THT, symbol Regulator_Switching:TSR1-2433E
- added U506: TEC2-2419WI, Converter_DCDC:Converter_DCDC_TRACO_TMR-xxxx_THT, symbol Converter_DCDC:TEC2-2419WI
- added U509: LT1763CS8-1.8, Package_SO:SOIC-8_3.9x4.9mm_P1.27mm, symbol AD4030:LT1763CS8
- C504: value 10u/50V -> 1u; footprint (none) -> Capacitor_SMD:C_0603_1608Metric_Pad1.08x0.95mm_HandSolder
- C505: value 10u/50V -> 10u/25V; footprint (none) -> Capacitor_SMD:C_1206_3216Metric_Pad1.33x1.80mm_HandSolder
- C511: renamed from C501; footprint (none) -> Capacitor_SMD:C_1210_3225Metric_Pad1.33x2.70mm_HandSolder
- C513: value 0.01u -> 10u/25V; footprint (none) -> Capacitor_SMD:C_1206_3216Metric_Pad1.33x1.80mm_HandSolder
- C514: renamed from C502; footprint (none) -> Capacitor_SMD:C_1210_3225Metric_Pad1.33x2.70mm_HandSolder
- C515: value 1u -> 10u/50V; footprint (none) -> Capacitor_SMD:C_1210_3225Metric_Pad1.33x2.70mm_HandSolder
- C516: renamed from C520; footprint (none) -> Capacitor_SMD:C_0603_1608Metric_Pad1.08x0.95mm_HandSolder
- C517: renamed from C522; footprint (none) -> Capacitor_SMD:C_0603_1608Metric_Pad1.08x0.95mm_HandSolder
- C518: renamed from C503; footprint (none) -> Capacitor_SMD:C_1206_3216Metric_Pad1.33x1.80mm_HandSolder
- C519: renamed from C521; footprint (none) -> Capacitor_SMD:C_1206_3216Metric_Pad1.33x1.80mm_HandSolder
- C520: renamed from C523; footprint (none) -> Capacitor_SMD:C_1206_3216Metric_Pad1.33x1.80mm_HandSolder
- C521: renamed from C512; footprint (none) -> Capacitor_SMD:C_0805_2012Metric_Pad1.18x1.45mm_HandSolder
- C523: renamed from C506; footprint (none) -> Capacitor_SMD:C_0603_1608Metric_Pad1.08x0.95mm_HandSolder
- C524: renamed from C507; footprint (none) -> Capacitor_SMD:C_1210_3225Metric_Pad1.33x2.70mm_HandSolder
- C525: renamed from C519; footprint (none) -> Capacitor_SMD:C_0805_2012Metric_Pad1.18x1.45mm_HandSolder
- C526: renamed from C508; footprint (none) -> Capacitor_SMD:C_0805_2012Metric_Pad1.18x1.45mm_HandSolder
- C527: renamed from C511; footprint (none) -> Capacitor_SMD:C_0603_1608Metric_Pad1.08x0.95mm_HandSolder
- C529: renamed from C509; footprint (none) -> Capacitor_SMD:C_1210_3225Metric_Pad1.33x2.70mm_HandSolder
- C531: renamed from C517; footprint (none) -> Capacitor_SMD:C_1210_3225Metric_Pad1.33x2.70mm_HandSolder
- C532: renamed from C510; value 1u -> 10u/25V; footprint (none) -> Capacitor_SMD:C_1206_3216Metric_Pad1.33x1.80mm_HandSolder
- C534: renamed from C518; footprint (none) -> Capacitor_SMD:C_1206_3216Metric_Pad1.33x1.80mm_HandSolder
- R505: value 5k11 -> 133k; footprint (none) -> Resistor_SMD:R_0603_1608Metric_Pad0.98x0.95mm_HandSolder
- R509: renamed from R503; footprint (none) -> Resistor_SMD:R_0603_1608Metric_Pad0.98x0.95mm_HandSolder
- R510: renamed from R504; footprint (none) -> Resistor_SMD:R_0603_1608Metric_Pad0.98x0.95mm_HandSolder
- renumbered L501 to L503, R501 to R503, R502 to R506, U507 to U504, U502 to U505, U504 to U507, U503 to U508, U506 to U510
Connections:
- net +9V: now also C505.1, C501.1, C507.1, U501.1 (Vin), U502.17 (PVIN1), U502.18 (PVINSYS), U502.19 (PVIN2), U503.1 (Vin), U506.6 (+VOUT); no longer FB501.1, FB502.1
- net GND: now also C504.1, C505.2, C513.2, C501.2, C506.2, C507.2, C508.2, C509.2, C510.1, C522.2, C530.2, C533.2, L502.2, R501.1, R502.1, R504.2, U501.2 (GND), U502.1 (PGND), U502.15 (AGND), U502.21 (EP), U502.4 (SYNQ/FREQ), U503.2 (GND), U506.7 (-VOUT), U509.3 (GND), U509.6 (GND), U509.7 (GND); no longer C515.2
- net GNDS: now also C515.2, C512.2, U506.1 (-VIN); no longer C504.2, C505.2
- net VIO: now also C528.1, C530.1, C533.1, U509.1 (OUT), U509.2 (SENSE/ADJ); no longer C513.1, C515.1, R505.1
- net at FB502.2: now also C522.1, U509.5 (~{SHDN}), U509.8 (IN)
- net at R505.2: now also R508.1, U502.13 (FB2)
- net at C511.1, D501.3 (K), D502.2 (A)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: now also C512.1, L504.1; no longer C504.1
- net at U504.10 (~{SHDNN}), U504.12 (~{SHDNP}), U504.14 (INP): now also C509.1, D503.1 (K), R507.2
- net at U504.6 (INN), U504.9 (INN): now also C510.2, D504.2 (A), R508.2
- new net: C503.1, R502.2
- new net: C503.2, U502.12 (COMP2)
- new net: C502.1, R501.2
- new net: D504.1 (K), L502.1, U502.20 (SW2)
- new net: C515.1, L504.2, U506.2 (+VIN)
- new net: D503.2 (A), L501.2, U502.2 (SW1)
- new net: C508.1, R505.1, U502.14 (VREF)
- new net: C504.2, U502.16 (VREG)
- new net: C528.2, U509.4 (BYP)
- new net: L501.1, U502.3 (INBK)
- new net: R504.1, R507.1, U502.7 (FB1)
- new net: C502.2, U502.8 (COMP1)
- new net +3.3V: C513.1, FB501.1, FB502.1, U503.3 (Vout)
- new net +5V: C506.1, U501.3 (Vout), U502.11 (EN2), U502.9 (EN1)
- no-connect marks 2 -> 5
Other:
- note removed: "https://www.analog.com/en/resources/technical-articles/bipolar-power-solutions-for-precision-test-and-measurement-systems.html"
- moved on the sheet: C511, C514, C516, C517, C518, C519, C520, C521, C523, C524, C525, C526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

Commit message: Hardware and started to create simulation.
Parts:
- removed C525: 1u, Capacitor_SMD:C_0805_2012Metric_Pad1.18x1.45mm_HandSolder, symbol Device:C
- removed C531: 47u/25V, Capacitor_SMD:C_1210_3225Metric_Pad1.33x2.70mm_HandSolder, symbol Device:C
- removed C534: 10u/25V, Capacitor_SMD:C_1206_3216Metric_Pad1.33x1.80mm_HandSolder, symbol Device:C
- removed FB503: FerriteBead_Small, symbol Device:FerriteBead_Small
- removed U501, U505: TSR1-2450E, Converter_DCDC:Converter_DCDC_TRACO_TSR1-xxxxE_THT, symbol Regulator_Switching:TSR1-2450E
- removed U503: TSR1-2433E, Converter_DCDC:Converter_DCDC_TRACO_TSR1-xxxxE_THT, symbol Regulator_Switching:TSR1-2433E
- removed U510: LT1461DxS8-5, Package_SO:SOIC-8_3.9x4.9mm_P1.27mm, symbol Reference_Voltage:LT1461DxS8-5
- added U501: LM1117MP-3.3, Package_TO_SOT_SMD:SOT-223-3_TabPin2, symbol Regulator_Linear:LM1117MP-3.3
- added U510: TSR1-2433E, Converter_DCDC:Converter_DCDC_TRACO_TSR1-xxxxE_THT, symbol Regulator_Switching:TSR1-2433E
- added U511: LM1117MP-5.0, Package_TO_SOT_SMD:SOT-223-3_TabPin2, symbol Regulator_Linear:LM1117MP-5.0
- FB501, FB502: value FerriteBead_Small -> BLM31PG330SN1L; footprint (none) -> Inductor_SMD:L_1206_3216Metric_Pad1.22x1.90mm_HandSolder
- U506: value TEC2-2419WI -> TEC3-2419WI
Connections:
- net +3.3V: now also U501.2 (VO)
- net +5V: now also C507.1, U501.3 (VI), U511.2 (VO)
- net +9V: now also U511.3 (VI); no longer C507.1
- net GND: now also U501.1 (GND), U511.1 (GND)
- net GNDS: now also U510.2 (GND)
- net at C514.1, L503.2: now also U510.1 (Vin)
- net at C518.1, U507.5 (~{SHDN}), U507.8 (IN): now also U510.3 (Vout)
- no-connect marks 5 -> 4
Other:
- moved on the sheet: C505, C507

Commit message: Hardware
Parts:
- removed U501: LM1117MP-3.3, Package_TO_SOT_SMD:SOT-223-3_TabPin2, symbol Regulator_Linear:LM1117MP-3.3
- removed U510: TSR1-2433E, Converter_DCDC:Converter_DCDC_TRACO_TSR1-xxxxE_THT, symbol Regulator_Switching:TSR1-2433E
- removed U511: LM1117MP-5.0, Package_TO_SOT_SMD:SOT-223-3_TabPin2, symbol Regulator_Linear:LM1117MP-5.0
- added U501: TSR_1-2450, Converter_DCDC:Converter_DCDC_TRACO_TSR-1_THT, symbol Regulator_Switching:TSR_1-2450
- added U503, U505: TSR_1-2433, Converter_DCDC:Converter_DCDC_TRACO_TSR-1_THT, symbol Regulator_Switching:TSR_1-2433
- D503, D504: footprint (none) -> AD4030:POWERDI123_DIO
- L501, L502: footprint (none) -> AD4030:XAL4030
- L503: footprint (none) -> Inductor_SMD:L_TracoPower_TCK-141
- L504: footprint (none) -> AD4030:TCK-133
- renumbered C526 to C525, C527 to C526, C528 to C527, C529 to C528, C530 to C529, C532 to C530, C533 to C531
Connections:
- net +3.3V: now also U503.3 (Vout)
- net +5V: now also U501.3 (Vout); no longer C507.1
- net +9V: now also C507.1, U501.1 (Vin), U503.1 (Vin)
- net GND: now also U501.2 (GND), U503.2 (GND)
- net GNDS: now also U505.2 (GND)
- net at C514.1, L503.2: now also U505.1 (Vin)
- net at C518.1, U507.5 (~{SHDN}), U507.8 (IN): now also U505.3 (Vout)
Other:
- note added: "https://www.analog.com/en/resources/technical-articles/bipolar-power-solutions-for-precision-test-and-measurement-systems.html https://xdevs.com/article/x732/"

Commit message: Hardware
Parts:
- removed D503, D504: DFLS240, AD4030:POWERDI123_DIO, symbol Device:D_Schottky
- removed L501: XAL4030-332ME, AD4030:XAL4030, symbol Device:L_Small
- removed L502: XAL4030-682ME, AD4030:XAL4030, symbol Device:L_Small
- removed U502: ADP5070AREZ, Package_SO:ETSSOP-20-1EP_4.4x6.5mm_P0.65mm_EP3x4.2mm, symbol AD4030:ADP5070AREZ
- added C532: 22u, symbol Device:C
- added R511: DNP, symbol Device:R
- added R512, R513: 100k, symbol Device:R
- added TP501: TestPoint, symbol Connector:TestPoint
- added U502: LTM8049, Package_BGA:Analog_BGA-77_9.0x15.0mm_Layout7x11_P1.27mm_Ball0.63mm, symbol Regulator_Switching:LTM8049
- C501: value 10u/25V -> 0.1u; footprint Capacitor_SMD:C_1206_3216Metric_Pad1.33x1.80mm_HandSolder -> (none)
- C502: value 47n -> 0.1u; footprint Capacitor_SMD:C_0603_1608Metric_Pad1.08x0.95mm_HandSolder -> (none)
- C503: value 47n -> 10u; footprint Capacitor_SMD:C_0603_1608Metric_Pad1.08x0.95mm_HandSolder -> Capacitor_SMD:C_1206_3216Metric_Pad1.33x1.80mm_HandSolder
- C504: value 1u -> 10u; footprint Capacitor_SMD:C_0603_1608Metric_Pad1.08x0.95mm_HandSolder -> Capacitor_SMD:C_1206_3216Metric_Pad1.33x1.80mm_HandSolder
- C508: footprint Capacitor_SMD:C_0603_1608Metric_Pad1.08x0.95mm_HandSolder -> (none)
- C509: value 10u/25V -> 1u; footprint Capacitor_SMD:C_1206_3216Metric_Pad1.33x1.80mm_HandSolder -> (none)
- C510: value 10u/25V -> 22u; footprint Capacitor_SMD:C_1206_3216Metric_Pad1.33x1.80mm_HandSolder -> (none)
- R501: value 3k9 -> R; footprint Resistor_SMD:R_0603_1608Metric_Pad0.98x0.95mm_HandSolder -> (none)
- R502: value 8k2 -> R; footprint Resistor_SMD:R_0603_1608Metric_Pad0.98x0.95mm_HandSolder -> (none)
- R504: value 121k -> 200k; footprint Resistor_SMD:R_0603_1608Metric_Pad0.98x0.95mm_HandSolder -> (none)
- R505: value 133k -> 153k; footprint Resistor_SMD:R_0603_1608Metric_Pad0.98x0.95mm_HandSolder -> (none)
- R507: value 787k -> 153k; footprint Resistor_SMD:R_0603_1608Metric_Pad0.98x0.95mm_HandSolder -> (none)
- R508: value R -> 200k; footprint Resistor_SMD:R_0603_1608Metric_Pad0.98x0.95mm_HandSolder -> (none)
Connections:
- net +9V: no longer C501.1
- net GND: now also C501.1, C502.2, C503.2, C509.1, C510.2, R505.1, R507.1, C532.1, U502.A3 (GND), U502.A4 (GND), U502.B3 (GND), U502.B4 (GND), U502.B5 (GND), U502.B6 (GND), U502.C2 (V_{OUT1N}), U502.C3 (GND), U502.C4 (GND), U502.C5 (GND), U502.C6 (GND), U502.D1 (V_{OUT1N}), U502.D2 (V_{OUT1N}), U502.D3 (GND), U502.D4 (GND), U502.D5 (GND), U502.E1 (V_{OUT1N}), U502.E2 (V_{OUT1N}), U502.E3 (GND), U502.E4 (GND), U502.E5 (GND), U502.F1 (GND), U502.F2 (GND), U502.F5 (GND), U502.F6 (GND), U502.F7 (GND), U502.G3 (GND), U502.G4 (GND), U502.G5 (GND), U502.H3 (GND), U502.H4 (GND), U502.H5 (GND), U502.J3 (GND), U502.J4 (GND), U502.J5 (GND), U502.J6 (GND), U502.K1 (V_{OUT2P}), U502.K2 (V_{OUT2P}), U502.K3 (GND), U502.K4 (GND), U502.K5 (GND), U502.K6 (GND), U502.L1 (V_{OUT2P}), U502.L2 (V_{OUT2P}), U502.L3 (GND), U502.L4 (GND); no longer C501.2, C509.2, C510.1, R501.1, R502.1, R504.2
- net at C503.1, R502.2: now also C508.1, C510.1, U504.10 (~{SHDNN}), U504.12 (~{SHDNP}), U504.14 (INP), U502.A1 (V_{OUT1P}), U502.A2 (V_{OUT1P}), U502.B1 (V_{OUT1P}), U502.B2 (V_{OUT1P})
- net at R501.2: now also C504.2, C509.2, U504.6 (INN), U504.9 (INN), C532.2, U502.G1 (V_{OUT2N}), U502.G2 (V_{OUT2N}), U502.H1 (V_{OUT2N}), U502.H2 (V_{OUT2N}), U502.J2 (V_{OUT2N}); no longer C502.1
- net at R505.2: now also U502.E7 (RT1); no longer R508.1
- net at R504.1: now also U502.H6 (PG2); no longer R507.1
- new net: R507.2, U502.G7 (RT2)
- new net: R502.1, U502.C1 (FBX1)
- new net: TP501.1, U502.G6 (CLKOUT2)
- new net: R512.2, U502.K7 (RUN2)
- new net: R511.1, U502.F3 (SHARE1)
- new net: R511.2, U502.F4 (SHARE2)
- new net: R501.1, U502.J1 (FBX2)
- new net: R513.2, U502.B7 (RUN1)
- new net: R508.1, U502.D6 (PG1)
- new net: C502.1, U502.J7 (SS2)
- new net: C501.2, U502.C7 (SS1)
- new net: U502.E6 (CLKOUT1), U502.H7 (SYNC2)
- new net VIN_9V: R504.2, R508.2, R512.1, R513.1, U502.A5 (V_{IN1}), U502.A6 (V_{IN1}), U502.A7 (V_{IN1}), U502.L5 (V_{IN2}), U502.L6 (V_{IN2}), U502.L7 (V_{IN2})
- no-connect marks 4 -> 1
Other:
- moved on the sheet: C516, C517, C519, C520, U504A, U504B

Commit message: Hardware and update to 2024.1
Parts:
- removed C501, C502: 0.1u, symbol Device:C
- removed C503, C504: 10u, Capacitor_SMD:C_1206_3216Metric_Pad1.33x1.80mm_HandSolder, symbol Device:C
- removed C508, C509: 1u, symbol Device:C
- removed C510, C532: 22u, symbol Device:C
- removed C516, C517: 0.01u, Capacitor_SMD:C_0603_1608Metric_Pad1.08x0.95mm_HandSolder, symbol Device:C
- removed R501, R502: R, symbol Device:R
- removed R504, R508: 200k, symbol Device:R
- removed R505, R507: 153k, symbol Device:R
- removed R511: DNP, symbol Device:R
- removed R512, R513: 100k, symbol Device:R
- removed TP501: TestPoint, symbol Connector:TestPoint
- removed U501: TSR_1-2450, Converter_DCDC:Converter_DCDC_TRACO_TSR-1_THT, symbol Regulator_Switching:TSR_1-2450
- removed U502: LTM8049, Package_BGA:Analog_BGA-77_9.0x15.0mm_Layout7x11_P1.27mm_Ball0.63mm, symbol Regulator_Switching:LTM8049
- removed U503: TSR_1-2433, Converter_DCDC:Converter_DCDC_TRACO_TSR-1_THT, symbol Regulator_Switching:TSR_1-2433
- removed U504: LT3032-5, Package_DFN_QFN:Linear_DE14MA, symbol Regulator_Linear:LT3032-5
- added U501: LM1117DT-3.3, Package_TO_SOT_SMD:TO-252-3_TabPin2, symbol Regulator_Linear:LM1117DT-3.3
- added U503: TSR_1-2450, Converter_DCDC:Converter_DCDC_TRACO_TSR-1_THT, symbol Regulator_Switching:TSR_1-2450
Connections:
- net +3.3V: now also U501.2 (VO)
- net +5V: now also C507.1, U501.3 (VI), U503.3 (Vout)
- net +9V: now also U503.1 (Vin); no longer C507.1
- net GND: now also U501.1 (GND), U503.2 (GND)
Other:
- moved on the sheet: C505, C506, C507, C513, C519, C520, C521, C522, C526, C527, C528, C529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

Commit message: Hardware
Parts:
- removed C507, C513, C531: 10u/25V, Capacitor_SMD:C_1206_3216Metric_Pad1.33x1.80mm_HandSolder, symbol Device:C
- removed C527: 0.01u, Capacitor_SMD:C_0603_1608Metric_Pad1.08x0.95mm_HandSolder, symbol Device:C
- removed C529: 47u/25V, Capacitor_SMD:C_1210_3225Metric_Pad1.33x2.70mm_HandSolder, symbol Device:C
- removed U501: LM1117DT-3.3, Package_TO_SOT_SMD:TO-252-3_TabPin2, symbol Regulator_Linear:LM1117DT-3.3
- removed U503: TSR_1-2450, Converter_DCDC:Converter_DCDC_TRACO_TSR-1_THT, symbol Regulator_Switching:TSR_1-2450
- removed U507: LT1763CS8-ADJ, Package_SO:SOIC-8_3.9x4.9mm_P1.27mm, symbol AD4030:LT1763CS8
- removed U508, U509: LT1763CS8-1.8, Package_SO:SOIC-8_3.9x4.9mm_P1.27mm, symbol AD4030:LT1763CS8
- added C501, C504, C505: 10u/25V, Capacitor_SMD:C_1206_3216Metric_Pad1.33x1.80mm_HandSolder, symbol Device:C
- added C508, C509: 470u/10V, Capacitor_Tantalum_SMD:CP_EIA-7343-43_Kemet-X_Pad2.25x2.55mm_HandSolder, symbol Device:C_Polarized
- added C512: 1u, Capacitor_SMD:C_0805_2012Metric_Pad1.18x1.45mm_HandSolder, symbol Device:C
- added L501, L502, L505, L506: XFL4020-472MEC, Inductor_SMD:L_Coilcraft_XxL4020, symbol Device:L
- added U501: TPS65133DPDR, Package_SON:WSON-12-1EP_3x3mm_P0.5mm_EP1.5x2.5mm_ThermalVias, symbol AD4030:TPS65133DPDR
- added U504: LT1763CDE-ADJ, Package_DFN_QFN:DFN-12-1EP_3x4mm_P0.5mm_EP1.7x3.3mm, symbol AD4030:LT1763xDE
- added U505: LT1763CDE-1.8, Package_DFN_QFN:DFN-12-1EP_3x4mm_P0.5mm_EP1.7x3.3mm, symbol AD4030:LT1763xDE
- added U506: LT1763IDE-3.3, Package_DFN_QFN:DFN-12-1EP_3x4mm_P0.5mm_EP1.7x3.3mm, symbol AD4030:LT1763xDE
- added U508: TSR_1-2450, Converter_DCDC:Converter_DCDC_TRACO_TSR-1_THT, symbol Regulator_Switching:TSR_1-2433
- C519: value 10u -> 0.01u; footprint Capacitor_SMD:C_1206_3216Metric_Pad1.33x1.80mm_HandSolder -> Capacitor_SMD:C_0603_1608Metric_Pad1.08x0.95mm_HandSolder
- C520: value 10u -> 47u/25V; footprint Capacitor_SMD:C_1206_3216Metric_Pad1.33x1.80mm_HandSolder -> Capacitor_SMD:C_1210_3225Metric_Pad1.33x2.70mm_HandSolder
- C522: value 1u -> 10u/25V; footprint Capacitor_SMD:C_0805_2012Metric_Pad1.18x1.45mm_HandSolder -> Capacitor_SMD:C_1206_3216Metric_Pad1.33x1.80mm_HandSolder
- renumbered C511 to C502, C512 to C503, C514 to C506, C515 to C507, C518 to C510, C521 to C511, C523 to C513, C505 to C514, C524 to C515, C525 to C516, C506 to C517, C526 to C518, C528 to C521, C530 to C523, R503 to R501, R506 to R502, R509 to R503, R510 to R504, U505 to U502, U506 to U503
Connections:
- net +1V8: now also U505.2 (OUT), U505.3 (OUT), U505.5 (SENSE/ADJ)
- net +3.3V: now also C519.1, C520.1, C522.1, U506.2 (OUT), U506.3 (OUT), U506.5 (SENSE/ADJ); no longer FB502.1
- net +5V: now also FB502.1, C501.1, L501.1, U501.11 (AVIN), U501.12 (PVIN), U501.7 (EN), U508.3 (Vout)
- net +5VA: now also C508.1, L506.2; no longer C519.1
- net +9V: now also U508.1 (Vin)
- net -5VA: now also C509.2, L505.2; no longer C520.2
- net GND: now also C520.2, C501.2, C504.2, C505.1, C508.2, C509.1, C512.2, L502.2, U501.13 (EP), U501.2 (PGND), U501.4 (GND), U501.5 (AGND), U501.6 (GND), U501.8 (GND), U505.13 (GND), U505.7 (GND), U506.13 (GND), U506.7 (GND), U508.2 (GND); no longer C519.2, C520.1
- net GNDS: now also U504.13 (GND), U504.7 (GND)
- net VCCQ: now also U504.2 (OUT), U504.3 (OUT)
- net at C510.1, U502.3 (Vout): now also U504.10 (IN), U504.11 (IN), U504.8 (~{SHDN})
- net at C518.2: now also U505.6 (BYP)
- net at C511.1, FB501.2: now also U505.10 (IN), U505.11 (IN), U505.8 (~{SHDN})
- net at R503.2, R504.1: now also U504.5 (SENSE/ADJ)
- net at FB502.2: now also C512.1, U506.10 (IN), U506.11 (IN), U506.8 (~{SHDN}); no longer C522.1
- net at C513.2: now also U504.6 (BYP)
- new net: L501.2, U501.1 (SWP)
- new net: C504.1, L506.1, U501.3 (VPOS)
- new net: C519.2, U506.6 (BYP)
- new net: L502.1, U501.10 (SWN)
- new net: C505.2, L505.1, U501.9 (VNEG)
Other:
- moved on the sheet: C503, C507, C511, C514, C517, C518, C521, C523, FB501, L504, U503
