File: AD4030/Hardware/AD4030-Voltage/AD4030-Voltage.kicad_pcb (KiCad board)
At the start: 2 copper layers, 187 parts, among them J401 Conn_01x08, J402 Conn_01x10, J501 1715721, K201 UMS05-1A80-75D, Q201 MMBT3904, Q501 SI5618A, Q502 MMBT3904, U201 ADG5236BCPZ, U202 ADA4817-1ARD, U203 ADA4817-1ARD, U204 ADA4895-1ARJZ, U205 AD797BRZ, U301 AD8475ACPZ, U302 AD4030-24, U401 ADuM260N, U402 ADuM260N, U501 TSR1-2450E, U502 ADP5070AREZ, U503 TSR1-2433E, U504 LT3032-5, U505 TSR1-2450E, U506 TEC2-2419WI, U507 LT1763CS8-ADJ, U508 LT1763CS8-1.8, U509 LT1763CS8-1.8, U510 LT1461DxS8-5, X301 ECS-2520MV-1000-BN-TR

Commit message: Hardware and started to create simulation.
Parts:
- removed U503: TSR1-2433E, Converter_DCDC:Converter_DCDC_TRACO_TSR1-xxxxE_THT
- added R306: 10k, Resistor_SMD:R_0603_1608Metric_Pad0.98x0.95mm_HandSolder, F.Cu at (116.7, 108.9)
- added U511: LM1117MP-5.0, Package_TO_SOT_SMD:SOT-223-3_TabPin2, F.Cu at (122.4, 113.4)
- C312: value 10u -> 1u
- R237: value R -> 2k5/0.1%
- RN201: value VoltageDivider_CenterPin3 -> MPMT50011002AT1
- U501: value TSR1-2450E -> LM1117MP-3.3; footprint Converter_DCDC:Converter_DCDC_TRACO_TSR1-xxxxE_THT -> Package_TO_SOT_SMD:SOT-223-3_TabPin2
- moved U501 19.5 mm to (103.5, 112.8), turned to 90 degrees
Connections:
- C312 pad 1: VIO -> Net-(U302-~{RST})
- C507 pad 1: +9V -> +5V
- RN201 pad 1: Net-(R237-Pad2) -> GND
- RN201 pad 2: GND -> Net-(R237-Pad2)
- U302 pad A7: VIO -> Net-(U302-~{RST})
- U501 pad 1: +9V -> GND
- U501 pad 2: GND -> +3.3V

Commit message: Hardware and update to 2024.1
Parts:
- removed C501, C509, C510, C532, C533, C534: 10u/25V, Capacitor_SMD:C_1206_3216Metric_Pad1.33x1.80mm_HandSolder
- removed C502, C503: 47n, Capacitor_SMD:C_0603_1608Metric_Pad1.08x0.95mm_HandSolder
- removed C504, C508: 1u, Capacitor_SMD:C_0603_1608Metric_Pad1.08x0.95mm_HandSolder
- removed C516, C517: 0.01u, Capacitor_SMD:C_0603_1608Metric_Pad1.08x0.95mm_HandSolder
- removed J402: Conn_01x10, Connector_PinHeader_2.54mm:PinHeader_1x10_P2.54mm_Vertical
- removed R224, R226, R227, R228, R229, R230, R231, R232, R234, R235: 1k/0.1%, Resistor_SMD:R_0603_1608Metric_Pad0.98x0.95mm_HandSolder
- removed R225: 120/0.1%, Resistor_SMD:R_0603_1608Metric_Pad0.98x0.95mm_HandSolder
- removed R233: 10k, Resistor_SMD:R_0603_1608Metric_Pad0.98x0.95mm_HandSolder
- removed R236, R238: 51, Resistor_SMD:R_0603_1608Metric_Pad0.98x0.95mm_HandSolder
- removed R237: 2k5/0.1%, Resistor_SMD:R_0603_1608Metric_Pad0.98x0.95mm_HandSolder
- removed R501: 3k9, Resistor_SMD:R_0603_1608Metric_Pad0.98x0.95mm_HandSolder
- removed R502: 8k2, Resistor_SMD:R_0603_1608Metric_Pad0.98x0.95mm_HandSolder
- removed R504: 121k, Resistor_SMD:R_0603_1608Metric_Pad0.98x0.95mm_HandSolder
- removed R505: 133k, Resistor_SMD:R_0603_1608Metric_Pad0.98x0.95mm_HandSolder
- removed R507: 787k, Resistor_SMD:R_0603_1608Metric_Pad0.98x0.95mm_HandSolder
- removed R508: R, Resistor_SMD:R_0603_1608Metric_Pad0.98x0.95mm_HandSolder
- removed RN201: MPMT50011002AT1, Package_TO_SOT_SMD:SOT-23
- removed RV203: 3266W-1-203, Potentiometer_THT:Potentiometer_Bourns_3266W_Vertical
- removed U502: ADP5070AREZ, Package_SO:ETSSOP-20-1EP_4.4x6.5mm_P0.65mm_EP3x4.2mm
- removed U504: LT3032-5, Package_DFN_QFN:Linear_DE14MA
- removed U510: LT1461DxS8-5, Package_SO:SOIC-8_3.9x4.9mm_P1.27mm
- removed U511: LM1117MP-5.0, Package_TO_SOT_SMD:SOT-223-3_TabPin2
- added C221: 0.1u, Capacitor_SMD:C_0603_1608Metric_Pad1.08x0.95mm_HandSolder, F.Cu at (313.8, 51.6)
- added C222: JR500, Capacitor_SMD:C_Trimmer_Voltronics_JR, F.Cu at (78.4, 58.6)
- added C233: 0.1u, Capacitor_SMD:C_0603_1608Metric_Pad1.08x0.95mm_HandSolder, F.Cu at (313.8, 54.1)
- added C313: 0.1u, Capacitor_SMD:C_0402_1005Metric_Pad0.74x0.62mm_HandSolder, F.Cu at (341.9, 21.6)
- added C314: 2u2, Capacitor_SMD:C_0805_2012Metric_Pad1.18x1.45mm_HandSolder, F.Cu at (345.8, 24.6)
- added C315: 1u, Capacitor_SMD:C_0805_2012Metric_Pad1.18x1.45mm_HandSolder, F.Cu at (345.8, 27.6)
- added C316: 1u, Capacitor_SMD:C_0805_2012Metric_Pad1.18x1.45mm_HandSolder, F.Cu at (345.8, 30.6)
- added C317: 2n7, Capacitor_SMD:C_0603_1608Metric_Pad1.08x0.95mm_HandSolder, F.Cu at (333.4, 27.8)
- added C318: 2u2, Capacitor_SMD:C_1210_3225Metric_Pad1.33x2.70mm_HandSolder, F.Cu at (340.4, 25.2)
- added C319: 2u2, Capacitor_SMD:C_1210_3225Metric_Pad1.33x2.70mm_HandSolder, F.Cu at (340.4, 29.5)
- added FB301: BLM31PG330SN1L, Inductor_SMD:L_1206_3216Metric_Pad1.22x1.90mm_HandSolder, F.Cu at (334.3, 24.8)
- added FB501: BLM31PG330SN1L, Inductor_SMD:L_1206_3216Metric_Pad1.22x1.90mm_HandSolder, F.Cu at (344.5, 37.1)
- added FB502: BLM31PG330SN1L, Inductor_SMD:L_1206_3216Metric_Pad1.22x1.90mm_HandSolder, F.Cu at (344.5, 40.5)
- added J201: 1710072, AD4030:1710072, F.Cu at (67.5, 65.0)
- added J403: PMOD, Connector_PinHeader_2.54mm:PinHeader_2x06_P2.54mm_Horizontal, F.Cu at (163.0, 55.0)
- added J404: PMOD, Connector_PinHeader_2.54mm:PinHeader_2x06_P2.54mm_Horizontal, F.Cu at (163.1, 73.4)
- added J405: Conn_01x07, Connector_PinHeader_2.54mm:PinHeader_1x07_P2.54mm_Vertical_SMD_Pin1Right, B.Cu at (147.6, 54.7)
- added L503: TCK-141, Inductor_SMD:L_TracoPower_TCK-141, F.Cu at (331.8, 47.5)
- added L504: TCK-133, AD4030:TCK-133, F.Cu at (147.4, 43.3)
- added R307: 10k, Resistor_SMD:R_0603_1608Metric_Pad0.98x0.95mm_HandSolder, F.Cu at (333.4, 30.3)
- added R412: 50, Resistor_SMD:R_0402_1005Metric_Pad0.72x0.64mm_HandSolder, F.Cu at (299.0, 32.4)
- added U206: LT5400-4, Package_SO:MSOP-8-1EP_3x3mm_P0.65mm_EP1.73x1.85mm_ThermalVias, F.Cu at (301.0, 37.7)
- added U207: LT5400-4, Package_SO:MSOP-8-1EP_3x3mm_P0.65mm_EP1.73x1.85mm_ThermalVias, F.Cu at (301.0, 42.3)
- added U208: LT5400-4, Package_SO:MSOP-8-1EP_3x3mm_P0.65mm_EP1.73x1.85mm_ThermalVias, F.Cu at (103.1, 58.0)
- added U209: TXB0101DBV, Package_TO_SOT_SMD:SOT-23-6, F.Cu at (299.9, 56.2)
- added U210: LT5400-8, Package_SO:MSOP-8-1EP_3x3mm_P0.65mm_EP1.73x1.85mm_ThermalVias, F.Cu at (103.5, 68.9)
- added U211: LMH6611, Package_TO_SOT_SMD:TSOT-23-6, F.Cu at (98.2, 63.9)
- added U212: LMH6611, Package_TO_SOT_SMD:TSOT-23-6, F.Cu at (103.5, 63.9)
- added U303: AD4030-24, AD4030:05-08-1797_ADI, F.Cu at (125.3, 65.1)
- added U304: MAX6350ESA, Package_SO:SOIC-8_3.9x4.9mm_P1.27mm, F.Cu at (344.6, 17.4)
- added U503: TSR_1-2450, Converter_DCDC:Converter_DCDC_TRACO_TSR-1_THT, F.Cu at (118.0, 42.5)
- C215: value 330p -> 0.1u
- C216, C219, U401, U507, U508, U509: moved to B.Cu
- C217: value 0.1u -> 330p
- C218: value 120p -> 0.1u
- C220: value 0.1u -> 120p
- C223: value 0.1u -> JR500; footprint Capacitor_SMD:C_0603_1608Metric_Pad1.08x0.95mm_HandSolder -> Capacitor_SMD:C_Trimmer_Voltronics_JR
- C224: value 100n -> 0.1u
- C225: value 0.1u -> 100n; moved to B.Cu
- C232: value 50p -> 0.1u
- C307: value 0.1u -> 560p
- C308: footprint Capacitor_SMD:C_0603_1608Metric_Pad1.08x0.95mm_HandSolder -> Capacitor_SMD:C_0402_1005Metric_Pad0.74x0.62mm_HandSolder
- C309: value 560p -> 0.1u; footprint Capacitor_SMD:C_0603_1608Metric_Pad1.08x0.95mm_HandSolder -> Capacitor_SMD:C_0402_1005Metric_Pad0.74x0.62mm_HandSolder
- C312: value 1u -> 0.1u; footprint Capacitor_SMD:C_0805_2012Metric_Pad1.18x1.45mm_HandSolder -> Capacitor_SMD:C_0402_1005Metric_Pad0.74x0.62mm_HandSolder
- C402, C406: value 0.1u -> 1u
- C403, C407: value 1u -> 0.1u
- C526: value 1u -> 0.01u; footprint Capacitor_SMD:C_0805_2012Metric_Pad1.18x1.45mm_HandSolder -> Capacitor_SMD:C_0603_1608Metric_Pad1.08x0.95mm_HandSolder
- C528: value 0.01u -> 47u/25V; footprint Capacitor_SMD:C_0603_1608Metric_Pad1.08x0.95mm_HandSolder -> Capacitor_SMD:C_1210_3225Metric_Pad1.33x2.70mm_HandSolder
- C530, C531: value 47u/25V -> 10u/25V; footprint Capacitor_SMD:C_1210_3225Metric_Pad1.33x2.70mm_HandSolder -> Capacitor_SMD:C_1206_3216Metric_Pad1.33x1.80mm_HandSolder
- J401: footprint Connector_PinHeader_2.54mm:PinHeader_1x08_P2.54mm_Vertical -> Connector_PinHeader_2.54mm:PinHeader_1x08_P2.54mm_Vertical_SMD_Pin1Right; moved to B.Cu
- R201, R202, R203, R204, R205, R206, R207, R208, R209, R210: value 1M/0.1% -> 2M/0.1%
- R211, R212: value 10k/0.1% -> 91; footprint Resistor_SMD:R_1206_3216Metric_Pad1.30x1.75mm_HandSolder -> Resistor_SMD:R_0603_1608Metric_Pad0.98x0.95mm_HandSolder
- R213, R214: value 91 -> 7k5; footprint Resistor_SMD:R_1206_3216Metric_Pad1.30x1.75mm_HandSolder -> Resistor_SMD:R_0603_1608Metric_Pad0.98x0.95mm_HandSolder; moved to B.Cu
- R215, R216: value 10k/0.1% -> 10M; footprint Resistor_SMD:R_1206_3216Metric_Pad1.30x1.75mm_HandSolder -> Resistor_SMD:R_0603_1608Metric_Pad0.98x0.95mm_HandSolder
- R217, R218: value 7k5 -> 510
- R219: value 10M -> 1k5
- R220: value 10M -> 120/0.1%
- R221: value 510 -> 10k
- R222: value 510 -> 51
- R223: value 1k5 -> 51
- R302, R303, R401, R402, R403, R404, R405, R406, R407, R408, R409, R410, R411: footprint Resistor_SMD:R_0603_1608Metric_Pad0.98x0.95mm_HandSolder -> Resistor_SMD:R_0402_1005Metric_Pad0.72x0.64mm_HandSolder
- R304: value 100 -> 33; footprint Resistor_SMD:R_0603_1608Metric_Pad0.98x0.95mm_HandSolder -> Resistor_SMD:R_0402_1005Metric_Pad0.72x0.64mm_HandSolder
- R305: value OPT -> 100
- R306: value 10k -> OPT
- U202: value ADA4817-1ARD -> LT5400-1; footprint Package_SO:SOIC-8-1EP_3.9x4.9mm_P1.27mm_EP2.29x3mm -> Package_SO:MSOP-8-1EP_3x3mm_P0.65mm_EP1.73x1.85mm_ThermalVias
- U204: value ADA4895-1ARJZ -> ADA4817-1ARD; footprint Package_TO_SOT_SMD:SOT-23-6_Handsoldering -> Package_SO:SOIC-8-1EP_3.9x4.9mm_P1.27mm_EP2.29x3mm
- U205: value AD797BRZ -> LT5400-4; footprint Package_SO:SOIC-8_3.9x4.9mm_P1.27mm -> Package_SO:MSOP-8-1EP_3x3mm_P0.65mm_EP1.73x1.85mm_ThermalVias
- U302: value AD4030-24 -> SN74AUC1G79DBVR; footprint AD4030:05-08-1797_ADI -> Package_TO_SOT_SMD:SOT-23-5_HandSoldering
- U501: value LM1117MP-3.3 -> LM1117DT-3.3; footprint Package_TO_SOT_SMD:SOT-223-3_TabPin2 -> Package_TO_SOT_SMD:TO-252-3_TabPin2
- U505: value TSR1-2450E -> TSR_1-2433; footprint Converter_DCDC:Converter_DCDC_TRACO_TSR1-xxxxE_THT -> Converter_DCDC:Converter_DCDC_TRACO_TSR-1_THT
- U506: value TEC2-2419WI -> TEC3-2419WI
- moved U302 250.2 mm to (348.2, -26.2)
- moved C202 246.5 mm to (264.0, -30.5)
- moved C204 246.5 mm to (264.0, -23.8)
- moved C207 246.5 mm to (264.0, -17.1)
- moved C210 246.5 mm to (264.0, -10.4)
- moved C213 246.5 mm to (264.0, -3.73)
- moved C220 246.5 mm to (273.5, -34.3)
- moved C224 246.5 mm to (273.5, -29.3)
- moved C226 246.5 mm to (273.5, -24.3)
- moved C227 246.5 mm to (273.5, -21.7)
- moved C228 246.5 mm to (273.5, -19.2)
- moved C229 246.5 mm to (273.5, -16.7)
- moved C230 246.5 mm to (273.5, -14.2)
- moved C231 246.5 mm to (277.9, -34.3)
- moved C232 246.5 mm to (277.9, -31.8)
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Connections:
- net /DIFF/GAIN_x3 renamed /DIFF/GAIN_x20
- C215 pad 1: Net-(C212-Pad2) -> +5VA
- C216 pad 1: GND -> Net-(C212-Pad2)
- C216 pad 2: Net-(C213-Pad2) -> GND
- C217 pad 1: +5VA -> GND
- C217 pad 2: GND -> Net-(C213-Pad2)
- C218 pad 1: Net-(C212-Pad2) -> -5VA
- C219 pad 1: GND -> Net-(C212-Pad2)
- C219 pad 2: Net-(C213-Pad2) -> GND
- C220 pad 1: -5VA -> GND
- C220 pad 2: GND -> Net-(C213-Pad2)
- C223 pad 1: -5VA -> Net-(C213-Pad2)
- C224 pad 1: Net-(C224-Pad1) -> -5VA
- C225 pad 1: -5VA -> Net-(C225-Pad1)
- C228 pad 2: Net-(U203--) -> Net-(U204--)
- C230 pad 1: Net-(U202-FB) -> Net-(U203-FB)
- C230 pad 2: Net-(U202--) -> Net-(U203--)
- C231 pad 1: Net-(U203--) -> Net-(U204--)
- C231 pad 2: Net-(U203-FB) -> Net-(U204-FB)
- C232 pad 1: Net-(U205-C/B) -> +3.3V
- C232 pad 2: Net-(C232-Pad2) -> GND
- C307 pad 1: +5VA -> Net-(U303-IN+)
- C308 pad 1: Net-(U302-IN+) -> GND
- C308 pad 2: GND -> Net-(U303-IN-)
- C309 pad 1: GND -> +5VA
- C309 pad 2: Net-(U302-IN-) -> GND
- C310 pad 1: Net-(U302-IN+) -> Net-(U303-IN+)
- C310 pad 2: Net-(U302-IN-) -> Net-(U303-IN-)
- C311 pad 2: Net-(U302-REFIN) -> Net-(U303-REFIN)
- C312 pad 1: Net-(U302-~{RST}) -> VIO
- C525 pad 1: Net-(U510-VIN) -> VCCQ
- C525 pad 2: GND -> GNDS
- C526 pad 1: VCCQ -> +1V8
- C526 pad 2: GNDS -> Net-(U508-BYP)
- C527 pad 1: +1V8 -> VIO
- C527 pad 2: Net-(U508-BYP) -> Net-(U509-BYP)
- C528 pad 1: VIO -> +1V8
- C528 pad 2: Net-(U509-BYP) -> GND
- C529 pad 1: +1V8 -> VIO
- C530 pad 1: VIO -> +1V8
- C531 pad 1: +5VREF -> VIO
- J401 pad 1: /Isolation/IO0 -> /Isolation/CONN_SDO0
- J401 pad 2: /Isolation/IO1 -> /Isolation/CONN_SDO1
- J401 pad 3: /Isolation/IO2 -> /Isolation/CONN_SDO2
- J401 pad 4: /Isolation/IO3 -> /Isolation/CONN_SDO3
- J401 pad 5: /Isolation/IO4 -> /Isolation/CONN_BUSY
- J401 pad 6: /Isolation/IO5 -> /Isolation/CONN_100MHz
- J401 pad 7: /Isolation/IO6 -> /Isolation/CONN_~{CS}
- J401 pad 8: /Isolation/IO7 -> /Isolation/CONN_SDI
- K201 pad 3: Net-(U202--) -> Net-(U203--)
- R211 pad 1: Net-(C212-Pad2) -> Net-(R211-Pad1)
- R212 pad 1: Net-(R211-Pad2) -> Net-(R212-Pad1)
- R213 pad 1: Net-(R212-Pad2) -> +5VA
- R214 pad 2: Net-(R214-Pad2) -> -5VA
- R215 pad 1: Net-(R214-Pad2) -> Net-(C212-Pad2)
- R215 pad 2: Net-(R215-Pad2) -> Net-(C225-Pad1)
- R216 pad 1: Net-(R215-Pad2) -> GND
- R217 pad 1: +5VA -> Net-(C212-Pad2)
- R217 pad 2: Net-(R217-Pad2) -> Net-(U203-+)
- R218 pad 1: Net-(R218-Pad1) -> Net-(U204-+)
- R218 pad 2: -5VA -> Net-(C213-Pad2)
- R219 pad 1: Net-(C212-Pad2) -> Net-(C227-Pad1)
- R219 pad 2: Net-(C224-Pad1) -> Net-(U204--)
- R220 pad 1: GND -> Net-(C227-Pad1)
- R220 pad 2: Net-(C213-Pad2) -> Net-(U204--)
- R221 pad 1: Net-(C212-Pad2) -> Net-(Q201-B)
- R221 pad 2: Net-(U202-+) -> Net-(U209-B)
- R222 pad 1: Net-(U203-+) -> Net-(R222-Pad1)
- R222 pad 2: Net-(C213-Pad2) -> Net-(R222-Pad2)
- R223 pad 1: Net-(C227-Pad1) -> Net-(R223-Pad1)
- R223 pad 2: Net-(U203--) -> /ADC/V_OUT
- R301 pad 1: Net-(X301-Tri-State) -> VIO
- R301 pad 2: GND -> Net-(X301-Tri-State)
- R302 pad 1: Net-(U301-+) -> Net-(X301-OUT)
- R302 pad 2: Net-(U302-IN+) -> /ADC/CLK_100MHz
- R303 pad 1: Net-(U301--) -> Net-(U301-+)
- R303 pad 2: Net-(U302-IN-) -> Net-(U303-IN+)
- R304 pad 1: +5VREF -> Net-(U301--)
- R304 pad 2: Net-(U302-REFIN) -> Net-(U303-IN-)
- R305 pad 2: Net-(R305-Pad2) -> Net-(U303-REFIN)
- R306 pad 1: VIO -> +5VREF
- R306 pad 2: Net-(U302-~{RST}) -> Net-(R306-Pad2)
- R401 pad 1: Net-(U401-VOA) -> /Isolation/CONN_SDO0
- R401 pad 2: /Isolation/IO0 -> Net-(J403-Pin_6)
- R402 pad 1: Net-(U401-VOB) -> /Isolation/CONN_SDO2
- R402 pad 2: /Isolation/IO1 -> Net-(J403-Pin_5)
- R403 pad 1: Net-(U401-VOC) -> /Isolation/CONN_BUSY
- R403 pad 2: /Isolation/IO2 -> Net-(J403-Pin_4)
- R404 pad 1: Net-(U401-VOD) -> /Isolation/CONN_~{CS}
- R404 pad 2: /Isolation/IO3 -> Net-(J403-Pin_3)
- R405 pad 1: Net-(U401-VOE) -> /Isolation/CONN_SCK
- R405 pad 2: /Isolation/IO4 -> Net-(J404-Pin_6)
- R406 pad 1: Net-(U402-VIA) -> /Isolation/CONN_CNV
- R406 pad 2: /Isolation/IO5 -> Net-(J404-Pin_5)
- R407 pad 1: Net-(U402-VIB) -> Net-(J403-Pin_12)
- R407 pad 2: /Isolation/IO6 -> /Isolation/CONN_SDO1
- R408 pad 1: Net-(U402-VIC) -> Net-(J403-Pin_11)
- R408 pad 2: /Isolation/IO7 -> /Isolation/CONN_SDO3
- R409 pad 1: Net-(U402-VID) -> Net-(J403-Pin_10)
- R409 pad 2: /Isolation/IO8 -> /Isolation/CONN_100MHz
- R410 pad 1: Net-(U402-VIE) -> Net-(J403-Pin_9)
- R410 pad 2: /Isolation/IO9 -> /Isolation/CONN_SDI
- R411 pad 1: Net-(U402-VIF) -> Net-(J404-Pin_12)
- R411 pad 2: /Isolation/IO10 -> /Isolation/CONN_GAIN_x20
- RV201 pad 1: Net-(R213-Pad2) -> Net-(R211-Pad2)
- RV201 pad 3: Net-(R214-Pad1) -> Net-(R212-Pad1)
- RV202 pad 1: Net-(R217-Pad2) -> Net-(R213-Pad2)
- RV202 pad 2: Net-(C224-Pad1) -> Net-(C225-Pad1)
- RV202 pad 3: Net-(R218-Pad1) -> Net-(R214-Pad1)
- U201 pad 1: Net-(R236-Pad2) -> Net-(R222-Pad2)
- U201 pad 10: Net-(C232-Pad2) -> Net-(U201-Pad10)
- U201 pad 2: Net-(U205-+) -> Net-(U201-Pad2)
- U201 pad 9: Net-(R238-Pad1) -> Net-(R223-Pad1)
- U202 pad 1: Net-(U202-FB) -> Net-(C212-Pad2)
- U202 pad 2: Net-(U202--) -> Net-(R211-Pad1)
- U202 pad 3: Net-(U202-+) -> Net-(U202-Pad3)
- U202 pad 4: -5VA -> Net-(U202-Pad3)
- U202 pad 5: unconnected-(U202-Pad5) -> Net-(C213-Pad2)
- U202 pad 6: Net-(R229-Pad1) -> Net-(R212-Pad2)
- U202 pad 7: +5VA -> Net-(U202-Pad7)
- U202 pad 8: +5VA -> Net-(U202-Pad7)
- U204 pad 1: Net-(R235-Pad2) -> Net-(U204-FB)
- U204 pad 2: -5VA -> Net-(U204--)
- U204 pad 4: Net-(U204--) -> -5VA
- U204 pad 5: +5VA -> unconnected-(U204-Pad5)
- U204 pad 6: +5VA -> Net-(U204-Pad6)
- U205 pad 1: Net-(U205-BAL) -> Net-(U203-FB)
- U205 pad 2: Net-(U205--) -> Net-(U203-FB)
- U205 pad 3: Net-(U205-+) -> Net-(U204--)
- U205 pad 4: -5VA -> Net-(U204--)
- U205 pad 5: Net-(U205-COMP) -> Net-(U204-FB)
- U205 pad 6: Net-(C232-Pad2) -> Net-(U204-FB)
- U205 pad 7: +5VA -> Net-(U203--)
- U205 pad 8: Net-(U205-C/B) -> Net-(U203--)
- U401 pad 10: unconnected-(U401-VOF-Pad10) -> /Isolation/CONN_100MHz
- U401 pad 11: Net-(U401-VOE) -> /Isolation/CONN_BUSY
- U401 pad 12: Net-(U401-VOD) -> /Isolation/CONN_SDO3
- U401 pad 13: Net-(U401-VOC) -> /Isolation/CONN_SDO2
- U401 pad 14: Net-(U401-VOB) -> /Isolation/CONN_SDO1
- U401 pad 15: Net-(U401-VOA) -> /Isolation/CONN_SDO0
- U401 pad 7: unconnected-(U401-VIF-Pad7) -> /ADC/CLK_100MHz
- U402 pad 10: /DIFF/Gain_x10-x100 -> /DIFF/Gain_x10
- U402 pad 2: Net-(U402-VIA) -> /Isolation/CONN_~{CS}
- U402 pad 3: Net-(U402-VIB) -> /Isolation/CONN_SDI
- U402 pad 4: Net-(U402-VIC) -> /Isolation/CONN_SCK
- U402 pad 5: Net-(U402-VID) -> /Isolation/CONN_CNV
- U402 pad 6: Net-(U402-VIE) -> /Isolation/CONN_GAIN_x20
- U402 pad 7: Net-(U402-VIF) -> /Isolation/CONN_GAIN_x10
- X301 pad 3: unconnected-(X301-OUT-Pad3) -> Net-(X301-OUT)

Commit message: Hardware
Parts:
- removed C524, C528, C529: 47u/25V, Capacitor_SMD:C_1210_3225Metric_Pad1.33x2.70mm_HandSolder
- removed C525: 1u, Capacitor_SMD:C_0805_2012Metric_Pad1.18x1.45mm_HandSolder
- removed C526, C527: 0.01u, Capacitor_SMD:C_0603_1608Metric_Pad1.08x0.95mm_HandSolder
- removed C530, C531: 10u/25V, Capacitor_SMD:C_1206_3216Metric_Pad1.33x1.80mm_HandSolder
- removed J405: Conn_01x07, Connector_PinHeader_2.54mm:PinHeader_1x07_P2.54mm_Vertical_SMD_Pin1Right
- removed R506: 100k, Resistor_SMD:R_0603_1608Metric_Pad0.98x0.95mm_HandSolder
- removed R509, R510: R, Resistor_SMD:R_0603_1608Metric_Pad0.98x0.95mm_HandSolder
- removed U507: LT1763CS8-ADJ, Package_SO:SOIC-8_3.9x4.9mm_P1.27mm
- removed U509: LT1763CS8-1.8, Package_SO:SOIC-8_3.9x4.9mm_P1.27mm
- added C501: 10u/25V, Capacitor_SMD:C_1206_3216Metric_Pad1.33x1.80mm_HandSolder, F.Cu at (97.4, 159.8)
- added C502: 10u/50V, Capacitor_SMD:C_1210_3225Metric_Pad1.33x2.70mm_HandSolder, B.Cu at (175.1, 70.2)
- added C503: 10u/50V, Capacitor_SMD:C_1210_3225Metric_Pad1.33x2.70mm_HandSolder, B.Cu at (102.4, 159.6)
- added C504: 10u/25V, Capacitor_SMD:C_1206_3216Metric_Pad1.33x1.80mm_HandSolder, F.Cu at (139.6, 79.2)
- added C508: 470u/10V, Capacitor_Tantalum_SMD:CP_EIA-7343-43_Kemet-X_Pad2.25x2.55mm_HandSolder, F.Cu at (150.6, 75.7)
- added C509: 470u/10V, Capacitor_Tantalum_SMD:CP_EIA-7343-43_Kemet-X_Pad2.25x2.55mm_HandSolder, F.Cu at (129.0, 75.6)
- added C510: 10u, Capacitor_SMD:C_1206_3216Metric_Pad1.33x1.80mm_HandSolder, F.Cu at (151.3, 92.9)
- added C516: 1u, Capacitor_SMD:C_0805_2012Metric_Pad1.18x1.45mm_HandSolder, F.Cu at (168.3, 158.5)
- added C517: 10u/25V, Capacitor_SMD:C_1206_3216Metric_Pad1.33x1.80mm_HandSolder, F.Cu at (126.7, 64.8)
- added J402: Conn_01x07, Connector_PinHeader_2.54mm:PinHeader_1x07_P2.54mm_Vertical_SMD_Pin1Right, B.Cu at (167.3, 97.2)
- added L501: XFL4020-472MEC, Inductor_SMD:L_Coilcraft_XxL4020, F.Cu at (145.5, 78.1)
- added L502: XFL4020-472MEC, Inductor_SMD:L_Coilcraft_XxL4020, F.Cu at (134.0, 78.1)
- added L505: XFL4020-472MEC, Inductor_SMD:L_Coilcraft_XxL4020, F.Cu at (134.0, 73.2)
- added L506: XFL4020-472MEC, Inductor_SMD:L_Coilcraft_XxL4020, F.Cu at (145.5, 73.3)
- added R308: OPT, Resistor_SMD:R_0603_1608Metric_Pad0.98x0.95mm_HandSolder, F.Cu at (131.8, 149.1)
- added R309: 10k, Resistor_SMD:R_0603_1608Metric_Pad0.98x0.95mm_HandSolder, F.Cu at (131.8, 151.1)
- added R501: 100k, Resistor_SMD:R_0603_1608Metric_Pad0.98x0.95mm_HandSolder, F.Cu at (157.7, 160.8)
- added R502: 100k, Resistor_SMD:R_0603_1608Metric_Pad0.98x0.95mm_HandSolder, F.Cu at (157.7, 163.3)
- added R504: R, Resistor_SMD:R_0603_1608Metric_Pad0.98x0.95mm_HandSolder, F.Cu at (157.7, 165.8)
- added U502: TSR_1-2433, Converter_DCDC:Converter_DCDC_TRACO_TSR-1_THT, F.Cu at (174.7, 62.7)
- added U504: LT1763CDE-ADJ, Package_DFN_QFN:DFN-12-1EP_3x4mm_P0.5mm_EP1.7x3.3mm, F.Cu at (129.3, 86.5)
- C314: value 2u2 -> 2u2/25V
- C506: value 10u/25V -> 10u/50V; footprint Capacitor_SMD:C_1206_3216Metric_Pad1.33x1.80mm_HandSolder -> Capacitor_SMD:C_1210_3225Metric_Pad1.33x2.70mm_HandSolder; moved to B.Cu
- C507: value 10u/25V -> 10u/50V; footprint Capacitor_SMD:C_1206_3216Metric_Pad1.33x1.80mm_HandSolder -> Capacitor_SMD:C_1210_3225Metric_Pad1.33x2.70mm_HandSolder
- C511, C512: value 10u/50V -> 1u; footprint Capacitor_SMD:C_1210_3225Metric_Pad1.33x2.70mm_HandSolder -> Capacitor_SMD:C_0805_2012Metric_Pad1.18x1.45mm_HandSolder
- C513: value 10u/25V -> 0.01u; footprint Capacitor_SMD:C_1206_3216Metric_Pad1.33x1.80mm_HandSolder -> Capacitor_SMD:C_0603_1608Metric_Pad1.08x0.95mm_HandSolder; moved to B.Cu
- C514: value 10u/50V -> 10u/25V; footprint Capacitor_SMD:C_1210_3225Metric_Pad1.33x2.70mm_HandSolder -> Capacitor_SMD:C_1206_3216Metric_Pad1.33x1.80mm_HandSolder
- C515: value 10u/50V -> 47u/25V
- C518, C519: value 10u -> 0.01u; footprint Capacitor_SMD:C_1206_3216Metric_Pad1.33x1.80mm_HandSolder -> Capacitor_SMD:C_0603_1608Metric_Pad1.08x0.95mm_HandSolder
- C520: value 10u -> 47u/25V; footprint Capacitor_SMD:C_1206_3216Metric_Pad1.33x1.80mm_HandSolder -> Capacitor_SMD:C_1210_3225Metric_Pad1.33x2.70mm_HandSolder
- C521: value 1u -> 47u/25V; footprint Capacitor_SMD:C_0805_2012Metric_Pad1.18x1.45mm_HandSolder -> Capacitor_SMD:C_1210_3225Metric_Pad1.33x2.70mm_HandSolder
- C522: value 1u -> 10u/25V; footprint Capacitor_SMD:C_0805_2012Metric_Pad1.18x1.45mm_HandSolder -> Capacitor_SMD:C_1206_3216Metric_Pad1.33x1.80mm_HandSolder
- C523: value 0.01u -> 10u/25V; footprint Capacitor_SMD:C_0603_1608Metric_Pad1.08x0.95mm_HandSolder -> Capacitor_SMD:C_1206_3216Metric_Pad1.33x1.80mm_HandSolder
- F501: moved to B.Cu
- R303, R304: value 33 -> DNP
- R305: value 100 -> 33; footprint Resistor_SMD:R_0603_1608Metric_Pad0.98x0.95mm_HandSolder -> Resistor_SMD:R_0402_1005Metric_Pad0.72x0.64mm_HandSolder
- R306: value OPT -> 33; footprint Resistor_SMD:R_0603_1608Metric_Pad0.98x0.95mm_HandSolder -> Resistor_SMD:R_0402_1005Metric_Pad0.72x0.64mm_HandSolder
- R307: value 10k -> 100
- R503: value 100k -> R
- U209: value TXB0101DBV -> LT5400-8; footprint Package_TO_SOT_SMD:SOT-23-6 -> Package_SO:MSOP-8-1EP_3x3mm_P0.65mm_EP1.73x1.85mm_ThermalVias
- U210: value LT5400-8 -> TXB0101DBV; footprint Package_SO:MSOP-8-1EP_3x3mm_P0.65mm_EP1.73x1.85mm_ThermalVias -> Package_TO_SOT_SMD:SOT-23-6
- U501: value LM1117DT-3.3 -> TPS65133DPDR; footprint Package_TO_SOT_SMD:TO-252-3_TabPin2 -> Package_SON:WSON-12-1EP_3x3mm_P0.5mm_EP1.5x2.5mm_ThermalVias
- U503: value TSR_1-2450 -> TEC3-2419WI; footprint Converter_DCDC:Converter_DCDC_TRACO_TSR-1_THT -> Converter_DCDC:Converter_DCDC_TRACO_TMR-xxxx_THT
- U505: value TSR_1-2433 -> LT1763CDE-1.8; footprint Converter_DCDC:Converter_DCDC_TRACO_TSR-1_THT -> Package_DFN_QFN:DFN-12-1EP_3x4mm_P0.5mm_EP1.7x3.3mm
- U506: value TEC3-2419WI -> LT1763IDE-3.3; footprint Converter_DCDC:Converter_DCDC_TRACO_TMR-xxxx_THT -> Package_DFN_QFN:DFN-12-1EP_3x4mm_P0.5mm_EP1.7x3.3mm
- U508: value LT1763CS8-1.8 -> TSR_1-2450; footprint Package_SO:SOIC-8_3.9x4.9mm_P1.27mm -> Converter_DCDC:Converter_DCDC_TRACO_TSR-1_THT; moved to F.Cu
- moved C519 254.4 mm to (157.7, 158.3)
- moved C513 240.2 mm to (123.3, 77.9), turned to 180 degrees
- moved F501 214.5 mm to (186.8, 70.3), turned to -90 degrees
- moved C514 213.0 mm to (120.8, 69.8), turned to -90 degrees
- moved C520 205.2 mm to (143.5, 86.5), turned to -90 degrees
- moved C505 200.2 mm to (139.8, 72.0), turned to 180 degrees
- moved C506 170.0 mm to (170.9, 70.2), turned to 90 degrees
- moved L503 160.6 mm to (173.0, 71.9), turned to 180 degrees
- moved Q501 146.9 mm to (186.7, 74.6), turned to 90 degrees
- moved U208 66.1 mm to (125.0, 120.4)
- moved U201 56.2 mm to (129.6, 110.4)
- moved C307 51.6 mm to (135.3, 108.1)
- moved U503 51.1 mm to (163.1, 66.4)
- moved C203 48.3 mm to (95.4, 87.8)
- moved C209 48.3 mm to (107.2, 87.8)
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Connections:
- C233 pad 1: VIO -> +1V8
- C304 pad 1: VIO -> +1V8
- C305 pad 1: VIO -> +1V8
- C312 pad 1: VIO -> +1V8
- C313 pad 1: VIO -> +1V8
- C317 pad 1: VIO -> +1V8
- C401 pad 1: VIO -> +1V8
- C402 pad 1: VIO -> +1V8
- C403 pad 1: VIO -> +1V8
- C404 pad 1: VIO -> +1V8
- C505 pad 1: +9V -> GND
- C505 pad 2: GND -> Net-(U501-VNEG)
- C506 pad 1: +5V -> Net-(U502-Vin)
- C506 pad 2: GND -> GNDS
- C507 pad 1: +5V -> Net-(U503-+VIN)
- C507 pad 2: GND -> GNDS
- C511 pad 1: Net-(D501-K) -> Net-(U505-~{SHDN})
- C511 pad 2: GNDS -> GND
- C512 pad 1: Net-(D501-K) -> Net-(U506-~{SHDN})
- C512 pad 2: GNDS -> GND
- C513 pad 1: +3.3V -> VCCQ
- C513 pad 2: GND -> Net-(U504-BYP)
- C514 pad 1: Net-(U505-Vin) -> +9V
- C514 pad 2: GNDS -> GND
- C515 pad 1: Net-(U506-+VIN) -> VCCQ
- C518 pad 1: Net-(U505-Vout) -> +1V8
- C518 pad 2: GNDS -> Net-(U505-BYP)
- C519 pad 1: +5VA -> +3.3V
- C519 pad 2: GND -> Net-(U506-BYP)
- C520 pad 1: GND -> +3.3V
- C520 pad 2: -5VA -> GND
- C521 pad 1: Net-(U508-IN) -> +1V8
- C522 pad 1: Net-(U509-IN) -> +3.3V
- C523 pad 1: VCCQ -> +1V8
- C523 pad 2: Net-(U507-BYP) -> GND
- FB501 pad 2: Net-(U508-IN) -> Net-(U505-~{SHDN})
- FB502 pad 1: +3.3V -> +5V
- FB502 pad 2: Net-(U509-IN) -> Net-(U506-~{SHDN})
- L503 pad 2: Net-(U505-Vin) -> Net-(U502-Vin)
- L504 pad 2: Net-(U506-+VIN) -> Net-(U503-+VIN)
- R221 pad 2: Net-(U209-B) -> Net-(U210-B)
- R301 pad 1: VIO -> +1V8
- R303 pad 1: Net-(U301-+) -> /ADC/V_OUT
- R303 pad 2: Net-(U303-IN+) -> Net-(U301-+)
- R304 pad 2: Net-(U303-IN-) -> GND
- R305 pad 1: +5VREF -> Net-(U301-+)
- R305 pad 2: Net-(U303-REFIN) -> Net-(U303-IN+)
- R306 pad 1: +5VREF -> Net-(U301--)
- R306 pad 2: Net-(R306-Pad2) -> Net-(U303-IN-)
- R307 pad 1: VIO -> +5VREF
- R307 pad 2: Net-(U303-~{RST}) -> Net-(U303-REFIN)
- R503 pad 1: Net-(D501-A) -> VCCQ
- R503 pad 2: Net-(J501-Pin_2) -> Net-(U504-SENSE/ADJ)
- U209 pad 1: VIO -> Net-(U212-+)
- U209 pad 3: /DIFF/Gain_x10 -> Net-(U212--)
- U209 pad 4: Net-(U209-B) -> Net-(U201-Pad10)
- U209 pad 5: VIO -> Net-(U209-Pad5)
- U209 pad 6: +3.3V -> Net-(U209-Pad5)
- U210 pad 1: Net-(U212-+) -> +1V8
- U210 pad 3: Net-(U212--) -> /DIFF/Gain_x10
- U210 pad 4: Net-(U201-Pad10) -> Net-(U210-B)
- U210 pad 5: Net-(U210-Pad5) -> +1V8
- U210 pad 6: Net-(U210-Pad5) -> +3.3V
- U302 pad 5: VIO -> +1V8
- U303 pad A8: VIO -> +1V8
- U303 pad B8: VIO -> +1V8
- U303 pad D2: Net-(R306-Pad2) -> Net-(R308-Pad2)
- U303 pad D3: Net-(R306-Pad2) -> Net-(R308-Pad2)
- U303 pad E2: Net-(R306-Pad2) -> Net-(R308-Pad2)
- U303 pad E3: Net-(R306-Pad2) -> Net-(R308-Pad2)
- U401 pad 1: VIO -> +1V8
- U402 pad 16: VIO -> +1V8
- U501 pad 1: GND -> Net-(U501-SWP)
- U501 pad 2: +3.3V -> GND
- U501 pad 3: +5V -> Net-(U501-VPOS)
- U503 pad 1: +9V -> GNDS
- U503 pad 2: GND -> Net-(U503-+VIN)
- U503 pad 3: +5V -> unconnected-(U503-ON/~{OFF}-Pad3)
- U505 pad 1: Net-(U505-Vin) -> unconnected-(U505-NC-Pad1)
- U505 pad 2: GNDS -> +1V8
- U505 pad 3: Net-(U505-Vout) -> +1V8
- U506 pad 1: GNDS -> unconnected-(U506-NC-Pad1)
- U506 pad 2: Net-(U506-+VIN) -> +3.3V
- U506 pad 3: unconnected-(U506-ON/~{OFF}-Pad3) -> +3.3V
- U506 pad 5: unconnected-(U506-NC-Pad5) -> +3.3V
- U506 pad 6: +9V -> Net-(U506-BYP)
- U506 pad 8: unconnected-(U506-NC-Pad8) -> Net-(U506-~{SHDN})
- U508 pad 1: +1V8 -> +9V
- U508 pad 2: +1V8 -> GND
- U508 pad 3: GND -> +5V
- X301 pad 4: VIO -> +1V8
Other:
- board outline added: 110 x 70 mm

Commit message: Created readme.md
Parts:
- moved R404 180.5 mm to (179.6, 99.6)
- moved C514 5.19 mm to (118.9, 65.0)
- moved C504 0.51 mm to (139.1, 79.2)
- moved C508 0.51 mm to (150.1, 75.7)
- moved C509 0.51 mm to (128.5, 75.6)
- moved L501 0.51 mm to (145.0, 78.1)
- moved L502 0.51 mm to (133.5, 78.1)
- moved L505 0.51 mm to (133.5, 73.2)
- moved L506 0.51 mm to (145.0, 73.3)
- moved U501 0.51 mm to (139.1, 75.8)
- moved C513 0.51 mm to (122.8, 77.9)
- moved C505 0.51 mm to (139.3, 72.0)
Changed lines of the file:
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@@
 	(footprint "Resistor_SMD:R_0402_1005Metric_Pad0.72x0.64mm_HandSolder"
 		(layer "F.Cu")
-		(at 316.1085 -18.485)
+		(at 179.578 99.568)
 		(descr "Resistor SMD 0402 (1005 Metric), square (rectangular) end terminal, IPC_7351 nominal with elongated pad for handsoldering. (Body size source: IPC-SM-782 page 72, https://www.pcb-3d.com/wordpress/wp-content/uploads/ipc-sm-782a_amendment_1_and_2.pdf), generated with kicad-footprint-generator")
 		(tags "resistor handsolder")
@@
 	(footprint "Capacitor_SMD:C_1206_3216Metric_Pad1.33x1.80mm_HandSolder"
 		(layer "F.Cu")
-		(at 139.565 79.248 180)
+		(at 139.057 79.248 180)
 		(descr "Capacitor SMD 1206 (3216 Metric), square (rectangular) end terminal, IPC_7351 nominal with elongated pad for handsoldering. (Body size source: IPC-SM-782 page 76, https://www.pcb-3d.com/wordpress/wp-content/uploads/ipc-sm-782a_amendment_1_and_2.pdf), generated with kicad-footprint-generator")
 		(tags "capacitor handsolder")
 		(property "Reference" "C504"
-			(at 0 -1.85 360)
+			(at 0 -1.85 0)
 			(layer "F.SilkS")
 			(effects
@@
 		)
 		(property "Value" "10u/25V"
-			(at 0 1.85 360)
+			(at 0 1.85 0)
 			(layer "F.Fab")
 			(effects
@@
 		)
 		(fp_text user "${REFERENCE}"
-			(at 0 0 360)
+			(at 0 0 0)
 			(layer "F.Fab")
 			(effects
@@
 	(footprint "Capacitor_SMD:C_1206_3216Metric_Pad1.33x1.80mm_HandSolder"
 		(layer "F.Cu")
-		(at 139.819 72.009 180)
+		(at 139.311 72.009 180)
 		(descr "Capacitor SMD 1206 (3216 Metric), square (rectangular) end terminal, IPC_7351 nominal with elongated pad for handsoldering. (Body size source: IPC-SM-782 page 76, https://www.pcb-3d.com/wordpress/wp-content/uploads/ipc-sm-782a_amendment_1_and_2.pdf), generated with kicad-footprint-generator")
 		(tags "capacitor handsolder")
 		(property "Reference" "C505"
-			(at 0 -1.85 360)
+			(at 0 -1.85 0)
 			(layer "F.SilkS")
 			(effects
@@
 		)
 		(property "Value" "10u/25V"
-			(at 0 1.85 360)
+			(at 0 1.85 0)
 			(layer "F.Fab")
 			(effects
@@
 		)
 		(fp_text user "${REFERENCE}"
-			(at 0 0 360)
+			(at 0 0 0)
 			(layer "F.Fab")
 			(effects
@@
 		(tags "DFN 0.5")
 		(property "Reference" "U504"
-			(at 0 -3.05 360)
+			(at 0 -3.05 0)
 			(layer "F.SilkS")
 			(effects
@@
 		)
 		(property "Value" "LT1763CDE-ADJ"
-			(at 0 3.05 360)
+			(at 0 3.05 0)
 			(layer "F.Fab")
 			(effects
@@
 	(footprint "Capacitor_SMD:C_1206_3216Metric_Pad1.33x1.80mm_HandSolder"
 		(layer "F.Cu")
-		(at 120.777 69.85 -90)
+		(at 118.872 65.024 -90)
 		(descr "Capacitor SMD 1206 (3216 Metric), square (rectangular) end terminal, IPC_7351 nominal with elongated pad for handsoldering. (Body size source: IPC-SM-782 page 76, https://www.pcb-3d.com/wordpress/wp-content/uploads/ipc-sm-782a_amendment_1_and_2.pdf), generated with kicad-footprint-generator")
 		(tags "capacitor handsolder")
@@
 	(footprint "Capacitor_Tantalum_SMD:CP_EIA-7343-43_Kemet-X_Pad2.25x2.55mm_HandSolder"
 		(layer "F.Cu")
-		(at 150.622 75.692 -90)
+		(at 150.114 75.692 -90)
 		(descr "Tantalum Capacitor SMD Kemet-X (7343-43 Metric), IPC_7351 nominal, (Body size from: http://www.kemet.com/Lists/ProductCatalog/Attachments/253/KEM_TC101_STD.pdf), generated with kicad-footprint-generator")
 		(tags "capacitor tantalum")
@@
 	(footprint "Capacitor_Tantalum_SMD:CP_EIA-7343-43_Kemet-X_Pad2.25x2.55mm_HandSolder"
 		(layer "F.Cu")
-		(at 129.032 75.565 90)
+		(at 128.524 75.565 90)
 		(descr "Tantalum Capacitor SMD Kemet-X (7343-43 Metric), IPC_7351 nominal, (Body size from: http://www.kemet.com/Lists/ProductCatalog/Attachments/253/KEM_TC101_STD.pdf), generated with kicad-footprint-generator")
 		(tags "capacitor tantalum")
@@
 	(footprint "Package_SON:WSON-12-1EP_3x3mm_P0.5mm_EP1.5x2.5mm_ThermalVias"
 		(layer "F.Cu")
-		(at 139.573 75.819 180)
+		(at 139.065 75.819 180)
 		(descr "WSON, 12 Pin (https://www.ti.com/lit/ds/symlink/tps63710.pdf#page=33), generated with kicad-footprint-generator ipc_noLead_generator.py")
 		(tags "WSON NoLead")
 		(property "Reference" "U501"
-			(at 0 -2.45 360)
+			(at 0 -2.45 0)
 			(layer "F.SilkS")
 			(effects
@@
 		)
 		(property "Value" "TPS65133DPDR"
-			(at 0 2.45 360)
+			(at 0 2.45 0)
 			(layer "F.Fab")
 			(effects
@@
 		)
 		(property "Footprint" "Package_SON:WSON-12-1EP_3x3mm_P0.5mm_EP1.5x2.5mm_ThermalVias"
-			(at 0 0 360)
+			(at 0 0 0)
 			(layer "F.Fab")
 			(hide yes)
@@
 		)
 		(property "Datasheet" "https://www.ti.com/lit/ds/symlink/tps65133.pdf?ts=1724434561817&ref_url=https%253A%252F%252Fwww.google.com%252F"
-			(at 0 0 360)
+			(at 0 0 0)
 			(layer "F.Fab")
 			(hide yes)
@@
 		)
 		(property "Description" "TPS65133 ±5-V, 250-mA Dual-Output Power Supply"
-			(at 0 0 360)
+			(at 0 0 0)
 			(layer "F.Fab")
 			(hide yes)
@@
 		)
 		(fp_text user "${REFERENCE}"
-			(at 0 0 360)
+			(at 0 0 0)
 			(layer "F.Fab")
 			(effects
@@
 		(tags "DCDC-Converter TRACO TSR-1")
 		(property "Reference" "U508"
-			(at -1.5 -6.71 360)
+			(at -1.5 -6.71 0)
 			(layer "F.SilkS")
 			(effects
@@
 		)
 		(property "Value" "TSR_1-2450"
-			(at 2.5 3.25 360)
+			(at 2.5 3.25 0)
 			(layer "F.Fab")
 			(effects
@@
 		)
 		(fp_text user "${REFERENCE}"
-			(at 3 -3 360)
+			(at 3 -3 0)
 			(layer "F.Fab")
 			(effects
@@
 		(tags "DFN 0.5")
 		(property "Reference" "U506"
-			(at 0 -3.05 360)
+			(at 0 -3.05 0)
 			(layer "F.SilkS")
 			(effects
@@
 		)
 		(property "Value" "LT1763IDE-3.3"
-			(at 0 3.05 360)
+			(at 0 3.05 0)
 			(layer "F.Fab")
 			(effects
@@
 	(footprint "Inductor_SMD:L_Coilcraft_XxL4020"
 		(layer "F.Cu")
-		(at 133.985 78.105 -90)
+		(at 133.477 78.105 -90)
 		(descr "L_Coilcraft_XxL4020 https://www.coilcraft.com/pdfs/xfl4020.pdf")
 		(tags "L Coilcraft XxL4020")
@@
 	(footprint "Inductor_SMD:L_Coilcraft_XxL4020"
 		(layer "F.Cu")
-		(at 133.985 73.152 90)
+		(at 133.477 73.152 90)
 		(descr "L_Coilcraft_XxL4020 https://www.coilcraft.com/pdfs/xfl4020.pdf")
 		(tags "L Coilcraft XxL4020")
@@
 	(footprint "Inductor_SMD:L_Coilcraft_XxL4020"
 		(layer "F.Cu")
-		(at 145.542 73.279 90)
+		(at 145.034 73.279 90)
 		(descr "L_Coilcraft_XxL4020 https://www.coilcraft.com/pdfs/xfl4020.pdf")
 		(tags "L Coilcraft XxL4020")
@@
 	(footprint "Inductor_SMD:L_Coilcraft_XxL4020"
 		(layer "F.Cu")
-		(at 145.542 78.105 90)
+		(at 145.034 78.105 90)
 		(descr "L_Coilcraft_XxL4020 https://www.coilcraft.com/pdfs/xfl4020.pdf")
 		(tags "L Coilcraft XxL4020")
@@
 	(footprint "Capacitor_SMD:C_0603_1608Metric_Pad1.08x0.95mm_HandSolder"
 		(layer "B.Cu")
-		(at 123.317 77.851 180)
+		(at 122.809 77.851 180)
 		(descr "Capacitor SMD 0603 (1608 Metric), square (rectangular) end terminal, IPC_7351 nominal with elongated pad for handsoldering. (Body size source: IPC-SM-782 page 76, https://www.pcb-3d.com/wordpress/wp-content/uploads/ipc-sm-782a_amendment_1_and_2.pdf), generated with kicad-footprint-generator")
 		(tags "capacitor handsolder")
