File: AD4030/Hardware/AD4030-Voltage/AD4030-Voltage.kicad_pcb (KiCad board)
At the start: 2 copper layers, 110 x 70 mm, 186 parts, among them J201 1710072, J401 Conn_01x08, J402 Conn_01x07, J403 PMOD, J404 PMOD, J501 1715721, K201 UMS05-1A80-75D, Q201 MMBT3904, Q501 SI5618A, Q502 MMBT3904, U201 ADG5236BCPZ, U202 LT5400-1, U203 ADA4817-1ARD, U204 ADA4817-1ARD, U205 LT5400-4, U206 LT5400-4, U207 LT5400-4, U208 LT5400-4, U209 LT5400-8, U210 TXB0101DBV, U211 LMH6611, U212 LMH6611, U301 AD8475ACPZ, U302 SN74AUC1G79DBVR, U303 AD4030-24, U304 MAX6350ESA, U401 ADuM260N, U402 ADuM260N, U501 TPS65133DPDR, U502 TSR_1-2433, U503 TEC3-2419WI, U504 LT1763CDE-ADJ, U505 LT1763CDE-1.8, U506 LT1763IDE-3.3, U508 TSR_1-2450, X301 ECS-2520MV-1000-BN-TR

Commit message: Hardware design
Parts:
- C215, C217, C220, C229, C302, C303, C304, C305, C306, C309, C315, C317, C401, C402, C403, C404, C405, C406, C407, C408, C501, C514, C522, C523, R211, R212, R303, R304: moved to B.Cu
- C310: footprint Capacitor_SMD:C_0603_1608Metric_Pad1.08x0.95mm_HandSolder -> Capacitor_SMD:C_0402_1005Metric_Pad0.74x0.62mm_HandSolder
- C311, C312, C313: footprint Capacitor_SMD:C_0402_1005Metric_Pad0.74x0.62mm_HandSolder -> Capacitor_SMD:C_0603_1608Metric_Pad1.08x0.95mm_HandSolder; moved to B.Cu
- C316: footprint Capacitor_SMD:C_0805_2012Metric_Pad1.18x1.45mm_HandSolder -> Resistor_SMD:R_0603_1608Metric_Pad0.98x0.95mm_HandSolder
- C318: footprint Capacitor_SMD:C_1210_3225Metric_Pad1.33x2.70mm_HandSolder -> Capacitor_SMD:C_0805_2012Metric_Pad1.18x1.45mm_HandSolder; moved to B.Cu
- C319: footprint Capacitor_SMD:C_1210_3225Metric_Pad1.33x2.70mm_HandSolder -> Capacitor_SMD:C_0805_2012Metric_Pad1.18x1.45mm_HandSolder
- C503, C513, F501, U401: moved to F.Cu
- C515: value 47u/25V -> 2u2; footprint Capacitor_SMD:C_1210_3225Metric_Pad1.33x2.70mm_HandSolder -> Capacitor_SMD:C_0805_2012Metric_Pad1.18x1.45mm_HandSolder; moved to B.Cu
- C516: renamed from C517; moved to B.Cu
- FB301, FB501, FB502: value BLM31PG330SN1L -> FBMJ2125HM330-T; footprint Inductor_SMD:L_1206_3216Metric_Pad1.22x1.90mm_HandSolder -> Inductor_SMD:L_0805_2012Metric_Pad1.15x1.40mm_HandSolder
- L501, L502, L505, L506: value XFL4020-472MEC -> 1239AS-H-4R7M; footprint Inductor_SMD:L_Coilcraft_XxL4020 -> Inductor_SMD:L_1008_2520Metric_Pad1.43x2.20mm_HandSolder
- R302: footprint Resistor_SMD:R_0402_1005Metric_Pad0.72x0.64mm_HandSolder -> Resistor_SMD:R_0603_1608Metric_Pad0.98x0.95mm_HandSolder
- U203, U204: value ADA4817-1ARD -> ADA4817-1ACP; footprint Package_SO:SOIC-8-1EP_3.9x4.9mm_P1.27mm_EP2.29x3mm -> Package_CSP:LFCSP-8-1EP_3x3mm_P0.5mm_EP1.45x1.74mm
- moved H101 262.0 mm to (83.5, 63.5)
- moved C301 257.3 mm to (143.5, 108.2)
- moved H102 253.6 mm to (133.5, 126.5)
- moved C308 251.4 mm to (148.5, 107.3), turned to 90 degrees
- moved C302 247.5 mm to (151.9, 108.0), turned to 180 degrees
- moved RN301 245.5 mm to (143.0, 99.1), turned to -90 degrees
- moved C304 243.8 mm to (151.9, 106.9), turned to 180 degrees
- moved C309 243.4 mm to (151.9, 102.1), turned to 180 degrees
- moved C303 239.1 mm to (155.7, 102.1), turned to 180 degrees
- moved C306 238.2 mm to (151.9, 103.1), turned to 180 degrees
- moved R305 237.5 mm to (146.4, 103.8), turned to 90 degrees
- moved C521 237.1 mm to (131.2, 75.3), turned to -90 degrees
- moved C305 237.0 mm to (155.7, 103.1), turned to 180 degrees
- moved X301 237.0 mm to (149.5, 88.5), turned to -90 degrees
- moved C202 235.1 mm to (85.0, 121.8)
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- renumbered C516 to C517, U508 to U507
Connections:
- C228 pad 2: Net-(U204--) -> Net-(U204-+)
- C231 pad 1: Net-(U204--) -> Net-(U204-+)
- C231 pad 2: Net-(U204-FB) -> Net-(U204--)
- J403 pad 2: GNDS -> unconnected-(J403-Pin_2-Pad2)
- J403 pad 3: Net-(J403-Pin_3) -> GNDS
- J403 pad 4: Net-(J403-Pin_4) -> GNDS
- J403 pad 7: unconnected-(J403-Pin_7-Pad7) -> Net-(J403-Pin_7)
- J403 pad 8: GNDS -> Net-(J403-Pin_8)
- J404 pad 10: unconnected-(J404-Pin_10-Pad10) -> Net-(J404-Pin_10)
- J404 pad 2: GNDS -> unconnected-(J404-Pin_2-Pad2)
- J404 pad 3: unconnected-(J404-Pin_3-Pad3) -> GNDS
- J404 pad 4: unconnected-(J404-Pin_4-Pad4) -> GNDS
- J404 pad 5: Net-(J404-Pin_5) -> unconnected-(J404-Pin_5-Pad5)
- J404 pad 6: Net-(J404-Pin_6) -> unconnected-(J404-Pin_6-Pad6)
- J404 pad 8: GNDS -> unconnected-(J404-Pin_8-Pad8)
- J404 pad 9: unconnected-(J404-Pin_9-Pad9) -> Net-(J404-Pin_9)
- J501 pad 2: Net-(J501-Pin_2) -> GNDS
- R218 pad 1: Net-(U204-+) -> Net-(U204--V_{S})
- R219 pad 2: Net-(U204--) -> Net-(U204-+)
- R220 pad 2: Net-(U204--) -> Net-(U204-+)
- R401 pad 2: Net-(J403-Pin_6) -> Net-(J403-Pin_12)
- R402 pad 2: Net-(J403-Pin_5) -> Net-(J403-Pin_10)
- R403 pad 2: Net-(J403-Pin_4) -> Net-(J403-Pin_8)
- R404 pad 2: Net-(J403-Pin_3) -> Net-(J403-Pin_6)
- R405 pad 2: Net-(J404-Pin_6) -> Net-(J404-Pin_12)
- R406 pad 2: Net-(J404-Pin_5) -> Net-(J404-Pin_10)
- R407 pad 1: Net-(J403-Pin_12) -> Net-(J403-Pin_11)
- R408 pad 1: Net-(J403-Pin_11) -> Net-(J403-Pin_9)
- R409 pad 1: Net-(J403-Pin_10) -> Net-(J403-Pin_7)
- R410 pad 1: Net-(J403-Pin_9) -> Net-(J403-Pin_5)
- R411 pad 1: Net-(J404-Pin_12) -> Net-(J404-Pin_11)
- R412 pad 1: Net-(J404-Pin_11) -> Net-(J404-Pin_9)
- R501 pad 2: Net-(J501-Pin_2) -> GNDS
- R502 pad 2: Net-(J501-Pin_2) -> GNDS
- U203 pad 1: Net-(U203-FB) -> +5VA
- U203 pad 2: Net-(U203--) -> Net-(U203-FB)
- U203 pad 3: Net-(U203-+) -> Net-(U203--)
- U203 pad 4: -5VA -> Net-(U203-+)
- U203 pad 5: unconnected-(U203-Pad5) -> -5VA
- U203 pad 6: Net-(U203-Pad6) -> unconnected-(U203-Pad6)
- U203 pad 7: +5VA -> Net-(U203-Pad7)
- U204 pad 1: Net-(U204-FB) -> +5VA
- U204 pad 4: -5VA -> Net-(U204--V_{S})
- U204 pad 5: unconnected-(U204-Pad5) -> -5VA
- U204 pad 6: Net-(U204-Pad6) -> unconnected-(U204-Pad6)
- U204 pad 7: +5VA -> Net-(U204-+V_{S})
- U205 pad 1: Net-(U203-FB) -> Net-(U203--)
- U205 pad 2: Net-(U203-FB) -> Net-(U203--)
- U205 pad 5: Net-(U204-FB) -> Net-(U204-+)
- U205 pad 6: Net-(U204-FB) -> Net-(U204-+)
- U205 pad 7: Net-(U203--) -> Net-(U203-FB)
- U205 pad 8: Net-(U203--) -> Net-(U203-FB)
- U206 pad 1: Net-(U203-Pad6) -> Net-(U203-Pad7)
- U206 pad 2: Net-(U203-Pad6) -> Net-(U203-Pad7)
- U206 pad 3: Net-(U204-Pad6) -> Net-(U204-+V_{S})
- U206 pad 4: Net-(U204-Pad6) -> Net-(U204-+V_{S})
Other:
- copper layers 2 -> 4

Commit message: Hardware design
Parts:
- C208, C211, C221, C224: moved to B.Cu
- R303: moved to F.Cu
- moved H102 16.5 mm to (117.0, 126.5)
- moved C401 13.7 mm to (158.5, 115.3)
- moved C402 13.7 mm to (160.0, 115.3)
- moved C405 13.6 mm to (173.7, 115.4)
- moved C406 13.6 mm to (172.2, 115.4)
- moved C403 13.6 mm to (160.0, 94.9)
- moved C404 13.6 mm to (158.5, 94.9)
- moved C407 13.5 mm to (171.8, 94.7)
- moved C408 13.5 mm to (173.4, 94.7)
- moved U401 13.5 mm to (166.5, 98.3)
- moved U402 13.5 mm to (166.5, 111.8)
- moved C509 10.6 mm to (116.5, 74.4), turned to -90 degrees
- moved C233 5.26 mm to (131.3, 114.8), turned to 90 degrees
- moved R303 3.24 mm to (143.5, 102.4), turned to 0 degrees
- moved C317 2.41 mm to (156.3, 98.2)
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Connections:
- J401 pad 1: /Isolation/CONN_SDO0 -> /Isolation/CONN_100MHz
- J401 pad 2: /Isolation/CONN_SDO1 -> /Isolation/CONN_SDO0
- J401 pad 3: /Isolation/CONN_SDO2 -> /Isolation/CONN_SDO1
- J401 pad 4: /Isolation/CONN_SDO3 -> /Isolation/CONN_SDO2
- J401 pad 5: /Isolation/CONN_BUSY -> /Isolation/CONN_SDO3
- J401 pad 6: /Isolation/CONN_100MHz -> /Isolation/CONN_BUSY
- U401 pad 10: /Isolation/CONN_100MHz -> /Isolation/CONN_BUSY
- U401 pad 11: /Isolation/CONN_BUSY -> /Isolation/CONN_SDO3
- U401 pad 12: /Isolation/CONN_SDO3 -> /Isolation/CONN_SDO2
- U401 pad 13: /Isolation/CONN_SDO2 -> /Isolation/CONN_SDO1
- U401 pad 14: /Isolation/CONN_SDO1 -> /Isolation/CONN_SDO0
- U401 pad 15: /Isolation/CONN_SDO0 -> /Isolation/CONN_100MHz
- U401 pad 2: /ADC/ADC_SDO0 -> /ADC/CLK_100MHz
- U401 pad 3: /ADC/ADC_SDO1 -> /ADC/ADC_SDO0
- U401 pad 4: /ADC/ADC_SDO2 -> /ADC/ADC_SDO1
- U401 pad 5: /ADC/ADC_SDO3 -> /ADC/ADC_SDO2
- U401 pad 6: /ADC/ADC_BUSY -> /ADC/ADC_SDO3
- U401 pad 7: /ADC/CLK_100MHz -> /ADC/ADC_BUSY
Routing:
- net Net-(C212-Pad2): track 0.00 -> 37.4 mm, vias 0 -> 1
- net Net-(C213-Pad2): track 0.00 -> 35.3 mm, vias 0 -> 1
- net Net-(U204--): track 0.00 -> 33.0 mm
- net Net-(U203--): track 0.00 -> 32.3 mm, vias 0 -> 2
- net GND: track 0.00 -> 28.6 mm, vias 0 -> 26
- net +5VREF: track 0.00 -> 26.1 mm, vias 0 -> 1
- net Net-(R222-Pad1): track 0.00 -> 21.3 mm
- net Net-(U201-Pad10): track 0.00 -> 17.6 mm
- net Net-(U204-Pad7): track 0.00 -> 17.3 mm
- net +5VA: track 0.00 -> 15.4 mm, vias 0 -> 6
- net Net-(C225-Pad1): track 0.00 -> 14.3 mm
- net Net-(J201-Pin_1): track 0.00 -> 14.2 mm
- net Net-(J201-Pin_2): track 0.00 -> 14.2 mm
- net Net-(U212--): track 0.00 -> 13.9 mm
- net Net-(C227-Pad1): track 0.00 -> 13.3 mm, vias 0 -> 1
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- added copper zone on In1.Cu, net GND
- added copper zone on B.Cu, net GNDS
- added copper zone on F.Cu, net GNDS
- added copper zone on In1.Cu, net GNDS
- added copper zone on F.Cu, net Net-(D501-A)
- added copper zone on F.Cu, net Net-(D501-K)
- added copper zone on F.Cu, net Net-(D502-K)
- added copper zone on F.Cu, net Net-(J501-Pin_1)
- added copper zone on F.Cu, net Net-(Q501-D)
- added copper zone on F.Cu, net Net-(U502-Vin)
Other:
- outline, holes or cut-outs redrawn
- board text added: "AD4030-24 TEST BOARD MODULE FOR ARTY Z7"
- board text added: "CMRR"
- board text added: "OFFSET"

Commit message: PCB layout
Parts:
- C504: moved to B.Cu
- moved C513 5.36 mm to (174.6, 83.8), turned to 180 degrees
- moved C504 5.06 mm to (122.9, 70.5), turned to 180 degrees
- moved C501 4.77 mm to (126.2, 67.7), turned to 180 degrees
- moved R504 4.32 mm to (170.9, 83.8)
- moved R503 3.18 mm to (170.1, 81.0), turned to -90 degrees
- moved C515 2.03 mm to (170.1, 79.4), turned to -90 degrees
- moved C511 1.06 mm to (138.7, 76.2)
- moved FB501 1.06 mm to (138.7, 72.4)
- moved FB502 1.06 mm to (150.1, 72.4)
- moved C518 1.06 mm to (135.4, 77.6)
- moved C519 1.06 mm to (146.8, 77.6)
- moved U505 1.06 mm to (135.4, 74.3)
- moved U506 1.06 mm to (146.8, 74.3)
- moved C512 1.06 mm to (150.1, 76.2)
- moved C502 0.51 mm to (177.0, 67.2)
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Routing:
- net +5V: track 2.37 -> 74.3 mm, vias 0 -> 7
- net +5VA: track 15.4 -> 57.2 mm, vias 6 -> 13
- net +9V: track 10.2 -> 39.5 mm, vias 0 -> 1
- net -5VA: track 8.85 -> 33.4 mm, vias 5 -> 10
- net +1V8: track 7.13 -> 22.7 mm, vias 1 -> 8
- net /DIFF/GAIN_x20: track 0.86 -> 15.6 mm, vias 1 -> 2
- net GND: track 28.6 -> 43.3 mm, vias 26 -> 33
- net Net-(U201-Pad16): track 1.67 -> 13.2 mm
- net VCCQ: track 0.00 -> 9.78 mm, vias 0 -> 4
- net +2V5: track 4.95 -> 12.9 mm, vias 1 -> 2
- net +3.3V: track 2.88 -> 9.11 mm, vias 1 -> 5
- net Net-(U303-~{RST}): track 0.00 -> 4.67 mm
- net Net-(U504-SENSE/ADJ): track 0.00 -> 4.66 mm
- net Net-(U503-+VIN): track 3.89 -> 0.00 mm
- net Net-(D501-K): track 3.89 -> 0.00 mm, vias 0 -> 6
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- added copper zone on B.Cu, net +1V8
- added copper zone on F.Cu, net +1V8
- added copper zone on In2.Cu, net +1V8
- added copper zone on B.Cu, net +3.3V
- added copper zone on F.Cu, net +3.3V
- added copper zone on In2.Cu, net +3.3V
- added copper zone on B.Cu, net +5V
- added copper zone on F.Cu, net +5V
- added copper zone on F.Cu, net +5VA
- added copper zone on In2.Cu, net +5VA
- added copper zone on In2.Cu, net +9V
- added copper zone on F.Cu, net -5VA
- added copper zone on In2.Cu, net -5VA
- added copper zone on B.Cu, net GND
- added copper zone on F.Cu, net GND
- added copper zone on B.Cu, net Net-(D501-K)
- added copper zone on F.Cu, net Net-(U501-SWN)
- added copper zone on F.Cu, net Net-(U501-SWP)
- added copper zone on F.Cu, net Net-(U501-VNEG)
- added copper zone on F.Cu, net Net-(U501-VPOS)
- added copper zone on B.Cu, net Net-(U502-Vin)
- added copper zone on F.Cu, net Net-(U502-Vout)
- added copper zone on In2.Cu, net Net-(U502-Vout)
- added copper zone on F.Cu, net Net-(U503-+VIN)
- added copper zone on F.Cu, net Net-(U505-~{SHDN})
- added copper zone on F.Cu, net Net-(U506-~{SHDN})
- added copper zone on B.Cu, net VCCQ
- added copper zone on F.Cu, net VCCQ

Commit message: PCB layout
Parts:
- moved H101 26.5 mm to (110.0, 63.5)
- moved J401 21.2 mm to (177.9, 95.9)
- moved J402 20.1 mm to (177.9, 116.5)
- moved R406 19.7 mm to (180.0, 116.2)
- moved R412 15.8 mm to (180.0, 117.5)
- moved R303 8.64 mm to (143.5, 111.0)
- moved H102 7.00 mm to (110.0, 126.5)
- moved R409 5.86 mm to (179.8, 94.5)
- moved C307 4.82 mm to (147.7, 107.4), turned to 180 degrees
- moved C308 4.58 mm to (147.7, 102.7), turned to 0 degrees
- moved R404 3.91 mm to (180.0, 121.3)
- moved R407 3.34 mm to (179.8, 99.6)
- moved R411 3.32 mm to (180.0, 120.0)
- moved R408 2.22 mm to (179.8, 97.0)
- moved R304 2.18 mm to (147.7, 104.5), turned to 0 degrees
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- renumbered R402 to R401, R403 to R402, R404 to R403, R405 to R404, R406 to R405, R401 to R406, R408 to R407, R409 to R408, R410 to R409, R411 to R410, R412 to R411, R407 to R412
Connections:
- C232 pad 1: +3.3V -> +5V
- J401 pad 2: /Isolation/CONN_SDO0 -> /Isolation/CONN_SDO3
- J401 pad 5: /Isolation/CONN_SDO3 -> /Isolation/CONN_SDO0
- J401 pad 7: /Isolation/CONN_~{CS} -> /Isolation/CONN_CNV
- J401 pad 8: /Isolation/CONN_SDI -> /Isolation/CONN_SCK
- J402 pad 1: /Isolation/CONN_SCK -> /Isolation/CONN_SDI
- J402 pad 2: /Isolation/CONN_CNV -> /Isolation/CONN_~{CS}
- J403 pad 11: Net-(J403-Pin_11) -> unconnected-(J403-Pin_11-Pad11)
- J403 pad 12: Net-(J403-Pin_12) -> unconnected-(J403-Pin_12-Pad12)
- J404 pad 11: Net-(J404-Pin_11) -> unconnected-(J404-Pin_11-Pad11)
- J404 pad 12: Net-(J404-Pin_12) -> unconnected-(J404-Pin_12-Pad12)
- J404 pad 5: unconnected-(J404-Pin_5-Pad5) -> Net-(J404-Pin_5)
- J404 pad 6: unconnected-(J404-Pin_6-Pad6) -> Net-(J404-Pin_6)
- J404 pad 7: unconnected-(J404-Pin_7-Pad7) -> Net-(J404-Pin_7)
- J404 pad 8: unconnected-(J404-Pin_8-Pad8) -> Net-(J404-Pin_8)
- R401 pad 1: /Isolation/CONN_SDO2 -> /Isolation/CONN_SDO0
- R402 pad 1: /Isolation/CONN_BUSY -> /Isolation/CONN_SDO1
- R403 pad 1: /Isolation/CONN_~{CS} -> /Isolation/CONN_100MHz
- R404 pad 1: /Isolation/CONN_SCK -> /Isolation/CONN_GAIN_x20
- R404 pad 2: Net-(J404-Pin_12) -> Net-(J404-Pin_10)
- R405 pad 1: /Isolation/CONN_CNV -> /Isolation/CONN_SDI
- R405 pad 2: Net-(J404-Pin_10) -> Net-(J404-Pin_8)
- R406 pad 1: /Isolation/CONN_SDO0 -> /Isolation/CONN_CNV
- R406 pad 2: Net-(J403-Pin_12) -> Net-(J404-Pin_6)
- R407 pad 2: /Isolation/CONN_SDO3 -> /Isolation/CONN_BUSY
- R408 pad 2: /Isolation/CONN_100MHz -> /Isolation/CONN_SDO2
- R409 pad 2: /Isolation/CONN_SDI -> /Isolation/CONN_SDO3
- R410 pad 1: Net-(J404-Pin_11) -> Net-(J404-Pin_9)
- R410 pad 2: /Isolation/CONN_GAIN_x20 -> /Isolation/CONN_GAIN_x10
- R411 pad 1: Net-(J404-Pin_9) -> Net-(J404-Pin_7)
- R411 pad 2: /Isolation/CONN_GAIN_x10 -> /Isolation/CONN_~{CS}
- R412 pad 1: Net-(J403-Pin_11) -> Net-(J404-Pin_5)
- R412 pad 2: /Isolation/CONN_SDO1 -> /Isolation/CONN_SCK
- U210 pad 6: +3.3V -> +5V
- U401 pad 11: /Isolation/CONN_SDO3 -> /Isolation/CONN_SDO0
- U401 pad 14: /Isolation/CONN_SDO0 -> /Isolation/CONN_SDO3
- U401 pad 3: /ADC/ADC_SDO0 -> /ADC/ADC_SDO3
- U401 pad 6: /ADC/ADC_SDO3 -> /ADC/ADC_SDO0
- U402 pad 10: /DIFF/Gain_x10 -> /ADC/ADC_CNV
- U402 pad 11: /DIFF/GAIN_x20 -> /ADC/ADC_SCK
- U402 pad 12: /ADC/ADC_CNV -> /ADC/ADC_SDI
- U402 pad 13: /ADC/ADC_SCK -> /ADC/ADC_~{CS}
- U402 pad 14: /ADC/ADC_SDI -> /DIFF/GAIN_x20
- U402 pad 15: /ADC/ADC_~{CS} -> /DIFF/Gain_x10
- U402 pad 2: /Isolation/CONN_~{CS} -> /Isolation/CONN_GAIN_x10
- U402 pad 3: /Isolation/CONN_SDI -> /Isolation/CONN_GAIN_x20
- U402 pad 4: /Isolation/CONN_SCK -> /Isolation/CONN_~{CS}
- U402 pad 5: /Isolation/CONN_CNV -> /Isolation/CONN_SDI
- U402 pad 6: /Isolation/CONN_GAIN_x20 -> /Isolation/CONN_SCK
- U402 pad 7: /Isolation/CONN_GAIN_x10 -> /Isolation/CONN_CNV
Routing:
- net /DIFF/Gain_x10: track 0.00 -> 33.9 mm
- net /ADC/ADC_CNV: track 0.00 -> 31.9 mm, vias 0 -> 2
- net /DIFF/GAIN_x20: track 15.6 -> 45.1 mm, vias 2 -> 3
- net /Isolation/CONN_CNV: track 0.00 -> 21.9 mm, vias 0 -> 1
- net /Isolation/CONN_SCK: track 0.00 -> 21.6 mm, vias 0 -> 1
- net /Isolation/CONN_~{CS}: track 0.00 -> 21.1 mm, vias 0 -> 1
- net /Isolation/CONN_GAIN_x10: track 0.00 -> 20.5 mm, vias 0 -> 1
- net /Isolation/CONN_SDI: track 0.00 -> 19.0 mm, vias 0 -> 1
- net /Isolation/CONN_GAIN_x20: track 0.00 -> 17.1 mm, vias 0 -> 1
- net /Isolation/CONN_100MHz: track 0.00 -> 17.0 mm, vias 0 -> 1
- net /Isolation/CONN_SDO3: track 0.00 -> 16.7 mm, vias 0 -> 1
- net /Isolation/CONN_SDO2: track 0.00 -> 16.5 mm, vias 0 -> 1
- net /ADC/CLK_100MHz: track 4.07 -> 20.0 mm
- net /Isolation/CONN_BUSY: track 0.00 -> 15.7 mm, vias 0 -> 1
- net /Isolation/CONN_SDO1: track 0.00 -> 15.6 mm, vias 0 -> 1
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- added copper zone on B.Cu, net +5VA
- added copper zone on F.Cu, net Net-(R308-Pad2)
- added copper zone on In2.Cu, net VCCQ
