File: AD4030/Hardware/AD4030-Voltage/AD4030-Voltage.kicad_sch (KiCad schematic)
At the start: 0 parts

Commit message: Hardware design
Other:
- sheet ADC ports: added V_OUT; removed none
- sheet DIFF ports: added GAIN_x3, Gain_x10-x100, V_OUT; removed GAIN_x10-100, V_OUTPUT
Changed lines of the file:
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@@
 	(sheet
 		(at 53.34 68.58)
-		(size 27.94 19.05)
+		(size 27.94 20.32)
 		(fields_autoplaced yes)
 		(stroke
@@
 		)
 		(property "Sheetfile" "DIFF.kicad_sch"
-			(at 53.34 88.2146 0)
+			(at 53.34 89.4846 0)
 			(effects
 				(font
@@
 			)
 		)
-		(pin "GAIN_x10-100" input
-			(at 81.28 73.66 0)
+		(pin "GAIN_x3" input
+			(at 81.28 85.09 0)
 			(effects
 				(font
@@
 			)
 		)
-		(pin "V_OUTPUT" output
-			(at 81.28 80.01 0)
+		(pin "Gain_x10-x100" input
+			(at 81.28 82.55 0)
+			(effects
+				(font
+					(size 1.27 1.27)
+				)
+				(justify right)
+			)
+		)
+		(pin "V_OUT" output
+			(at 81.28 71.12 0)
 			(effects
 				(font
@@
 	)
 	(sheet
-		(at 96.52 67.31)
-		(size 40.64 20.32)
+		(at 92.71 68.58)
+		(size 30.48 20.32)
 		(fields_autoplaced yes)
 		(stroke
@@
 		)
 		(property "Sheetname" "ADC"
-			(at 96.52 66.5984 0)
+			(at 92.71 67.8684 0)
 			(effects
 				(font
@@
 		)
 		(property "Sheetfile" "ADC.kicad_sch"
-			(at 96.52 88.2146 0)
+			(at 92.71 89.4846 0)
 			(effects
 				(font
@@
 			)
 		)
+		(pin "V_OUT" input
+			(at 92.71 71.12 180)
+			(effects
+				(font
+					(size 1.27 1.27)
+				)
+				(justify left)
+			)
+		)

Commit message: Hardware
Other:
- added sheet Isolation (Isolation.kicad_sch)
- added sheet Power (Power.kicad_sch)
- note added: "Power DIFF 63 mW ADC 40 mW"
Changed lines of the file:
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@@
 	(generator_version "8.0")
 	(paper "A4")
+	(text "Power \nDIFF 63 mW \nADC 40 mW"
+		(exclude_from_sim no)
+		(at 70.358 31.75 0)
+		(effects
+			(font
+				(size 1.27 1.27)
+			)
+		)
+	)
 	(sheet
 		(at 53.34 68.58)
@@
 	)
 	(sheet
+		(at 135.89 68.58)
+		(size 52.07 31.75)
+		(fields_autoplaced yes)
+		(stroke
+			(width 0.1524)
+			(type solid)
+		)
+		(fill
+			(color 0 0 0 0.0000)
+		)
+		(property "Sheetname" "Isolation"
+			(at 135.89 67.8684 0)
+			(effects
+				(font
+					(size 1.27 1.27)
+				)
+				(justify left bottom)
+			)
+		)
+		(property "Sheetfile" "Isolation.kicad_sch"
+			(at 135.89 100.9146 0)
+			(effects
+				(font
+					(size 1.27 1.27)
+				)
+				(justify left top)
+			)
+		)
+		(instances
+			(project "AD4030-Voltage"
+				(path "/af28bfe6-a5ae-47dd-9259-97a6edcec559"
+					(page "4")
+				)
+			)
+		)
+	)
+	(sheet
 		(at 92.71 68.58)
 		(size 30.48 20.32)
@@
 				)
 			)
+		)
+	)
+	(sheet
+		(at 139.7 114.3)
+		(size 46.99 31.75)
+		(fields_autoplaced yes)
+		(stroke
+			(width 0.1524)
+			(type solid)
+		)
+		(fill
+			(color 0 0 0 0.0000)
+		)
+		(property "Sheetname" "Power"
+			(at 139.7 113.5884 0)
+			(effects
+				(font
+					(size 1.27 1.27)
+				)
+				(justify left bottom)
+			)
+		)
+		(property "Sheetfile" "Power.kicad_sch"
+			(at 139.7 146.6346 0)
+			(effects
+				(font
+					(size 1.27 1.27)
+				)
+				(justify left top)
+			)
+		)
+		(instances
+			(project "AD4030-Voltage"
+				(path "/af28bfe6-a5ae-47dd-9259-97a6edcec559"
+					(page "5")
+				)
+			)

Commit message: Hardware
Parts:
- added H101, H102: MountingHole, symbol Mechanical:MountingHole
Other:
- sheet ADC ports: added ADC_BUSY, ADC_CNV, ADC_SCK, ADC_SDI, ADC_SDO0, ADC_SDO1, ADC_SDO2, ADC_SDO3, ADC_~{CS}; removed none
- sheet Isolation ports: added ADC_BUSY, ADC_CNV, ADC_SCK, ADC_SDI, ADC_SDO0, ADC_SDO1, ADC_SDO2, ADC_SDO3, ADC_~{CS}, GAIN_x3, Gain_x10-x100; removed none
- note removed: "Power DIFF 63 mW ADC 40 mW"

Commit message: Hardware
Parts:
- H101, H102: footprint (none) -> MountingHole:MountingHole_3.2mm_M3_DIN965
Changed lines of the file:
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@@
 			)
 		)
-		(property "Footprint" ""
+		(property "Footprint" "MountingHole:MountingHole_3.2mm_M3_DIN965"
 			(at 20.32 190.5 0)
 			(effects
@@
 			)
 		)
-		(property "Footprint" ""
+		(property "Footprint" "MountingHole:MountingHole_3.2mm_M3_DIN965"
 			(at 41.91 190.5 0)
 			(effects

Commit message: Hardware and started to create simulation.
Other:
- sheet ADC ports: added CLK_100MHz; removed none
- sheet Isolation ports: added CLK_100MHz; removed none
Changed lines of the file:
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@@
+	(wire
+		(pts
+			(xy 154.94 71.12) (xy 167.64 71.12)
+		)
+		(stroke
+			(width 0)
+			(type default)
+		)
+	)
 	(wire
 		(pts
@@
 			)
 		)
+		(pin "CLK_100MHz" input
+			(at 167.64 71.12 180)
+			(effects
+				(font
+					(size 1.27 1.27)
+				)
+				(justify left)
+			)
+		)
 		(instances
 			(project "AD4030-Voltage"
@@
 			(effects
 				(font
+					(size 1.27 1.27)
+				)
+				(justify right)
+			)
+		)
+		(pin "CLK_100MHz" output
+			(at 154.94 71.12 0)
+			(effects
+				(font

Commit message: Hardware design and simulation
Other:
- sheet DIFF ports: added GAIN_x20, Gain_x10; removed GAIN_x3, Gain_x10-x100
- sheet Isolation ports: added GAIN_x20, Gain_x10; removed GAIN_x3, Gain_x10-x100
Changed lines of the file:
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@@
 			)
 		)
-		(pin "GAIN_x3" input
+		(pin "GAIN_x20" input
 			(at 109.22 76.2 0)
 			(effects
@@
 			)
 		)
-		(pin "Gain_x10-x100" input
+		(pin "Gain_x10" input
 			(at 109.22 73.66 0)
 			(effects
@@
 			)
 		)
-		(pin "Gain_x10-x100" output
+		(pin "Gain_x10" output
 			(at 167.64 82.55 180)
 			(effects
@@
 			)
 		)
-		(pin "GAIN_x3" output
+		(pin "GAIN_x20" output
 			(at 167.64 85.09 180)
 			(effects
