File: AD4030/Hardware/AD4030-Current/ADC.kicad_sch (KiCad schematic)
At the start: 33 parts, among them U301 AD8475ACPZ, U302 SN74AUC1G79DBVR, U303 AD4030-24, U304 LTC6655BHMS8-5, X301 ECS-2520MV-1000-BN-TR

Commit message: Hardware
Connections:
- net +5VA: now also C301.1; no longer C306.1, C309.1
- net +5V4: now reaches U303.A3 (VDD_5V), U303.B3 (VDD_5V)
- net +5V4: now also C306.1, C309.1
Changed lines of the file:
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@@
 	)
 	(symbol
-		(lib_id "Device:C")
-		(at 137.16 49.53 90)
+		(lib_id "AD4030:+5V4")
+		(at 160.02 50.8 0)
 		(unit 1)
 		(exclude_from_sim no)
@@
 		(dnp no)
 		(fields_autoplaced yes)
-		(property "Reference" "C311"
-			(at 137.16 41.91 90)
+		(property "Reference" "#PWR0203"
+			(at 160.02 54.61 0)
 			(effects
 				(font
 					(size 1.27 1.27)
 				)
+				(hide yes)
 			)
 		)
-		(property "Value" "1u"
-			(at 137.16 44.45 90)
+		(property "Value" "+5V4"
+			(at 160.02 45.72 0)
 			(effects
 				(font
@@
 			)
 		)
-		(property "Footprint" "Capacitor_SMD:C_0603_1608Metric_Pad1.08x0.95mm_HandSolder"
-			(at 140.97 48.5648 0)
+		(property "Footprint" ""
+			(at 160.02 50.8 0)
 			(effects
 				(font
@@
 			)
 		)
-		(property "Datasheet" "~"
-			(at 137.16 49.53 0)
+		(property "Datasheet" ""
+			(at 160.02 50.8 0)
 			(effects
 				(font
@@
 			)
 		)
-		(property "Description" "Unpolarized capacitor"
-			(at 137.16 49.53 0)
+		(property "Description" ""
+			(at 160.02 50.8 0)
 			(effects
 				(font
@@
 		(pin "1"
 		)
-		(pin "2"
-		)
 		(instances
-			(project ""
+			(project "AD4030-Current"
 				(path "/8c00fb7d-8cfe-468b-9ed3-32d6000462dd/0fe1e8e6-94f3-423b-8365-cd8c8da34f38"
-					(reference "C311")
-					(unit 1)
-				)
-			)
-			(project ""
-				(path "/af28bfe6-a5ae-47dd-9259-97a6edcec559/cfc38c8d-3c9b-4f41-9734-05b81b218479"
-					(reference "C311")
+					(reference "#PWR0203")
 					(unit 1)
 				)
@@
 	)
 	(symbol
-		(lib_id "power:GND")
-		(at 133.35 49.53 270)
+		(lib_id "Device:C")
+		(at 137.16 49.53 90)
 		(unit 1)
 		(exclude_from_sim no)
@@
 		(dnp no)
 		(fields_autoplaced yes)
-		(property "Reference" "#PWR0320"
-			(at 127 49.53 0)
+		(property "Reference" "C311"
+			(at 137.16 41.91 90)
 			(effects
 				(font
 					(size 1.27 1.27)
 				)
-				(hide yes)
 			)
 		)
-		(property "Value" "GND"
-			(at 129.54 49.5299 90)
+		(property "Value" "1u"
+			(at 137.16 44.45 90)
 			(effects
 				(font
 					(size 1.27 1.27)
 				)
-				(justify right)
 			)
 		)
-		(property "Footprint" ""
-			(at 133.35 49.53 0)
+		(property "Footprint" "Capacitor_SMD:C_0603_1608Metric_Pad1.08x0.95mm_HandSolder"
+			(at 140.97 48.5648 0)
 			(effects
 				(font
@@
 			)
 		)
-		(property "Datasheet" ""
-			(at 133.35 49.53 0)
+		(property "Datasheet" "~"
+			(at 137.16 49.53 0)
 			(effects
 				(font
@@
 			)
 		)
-		(property "Description" "Power symbol creates a global label with name \"GND\" , ground"
-			(at 133.35 49.53 0)
+		(property "Description" "Unpolarized capacitor"
+			(at 137.16 49.53 0)
 			(effects
 				(font
@@
 		(pin "1"
 		)
+		(pin "2"
+		)
 		(instances
-			(project "AD4030-Voltage"
+			(project ""
 				(path "/8c00fb7d-8cfe-468b-9ed3-32d6000462dd/0fe1e8e6-94f3-423b-8365-cd8c8da34f38"
-					(reference "#PWR0320")
+					(reference "C311")
 					(unit 1)
 				)
 			)
-			(project "AD4030-Voltage"
+			(project ""
 				(path "/af28bfe6-a5ae-47dd-9259-97a6edcec559/cfc38c8d-3c9b-4f41-9734-05b81b218479"
-					(reference "#PWR0320")
+					(reference "C311")
 					(unit 1)
 				)
@@
 	)
 	(symbol
-		(lib_id "power:+5VA")
-		(at 102.87 176.53 0)
+		(lib_id "power:GND")
+		(at 133.35 49.53 270)
 		(unit 1)
 		(exclude_from_sim no)
@@
 		(dnp no)
 		(fields_autoplaced yes)
-		(property "Reference" "#PWR0318"
-			(at 102.87 180.34 0)
+		(property "Reference" "#PWR0320"
+			(at 127 49.53 0)
 			(effects
 				(font
@@
 			)
 		)
-		(property "Value" "+5VA"
-			(at 102.87 171.45 0)
+		(property "Value" "GND"
+			(at 129.54 49.5299 90)
 			(effects
 				(font
 					(size 1.27 1.27)
 				)
+				(justify right)
 			)
 		)
 		(property "Footprint" ""
-			(at 102.87 176.53 0)
+			(at 133.35 49.53 0)
 			(effects
 				(font
@@
 		)
 		(property "Datasheet" ""
-			(at 102.87 176.53 0)
+			(at 133.35 49.53 0)
 			(effects
 				(font
@@
 			)
 		)
-		(property "Description" "Power symbol creates a global label with name \"+5VA\""
-			(at 102.87 176.53 0)
+		(property "Description" "Power symbol creates a global label with name \"GND\" , ground"
+			(at 133.35 49.53 0)
 			(effects
 				(font
@@
 			(project "AD4030-Voltage"
 				(path "/8c00fb7d-8cfe-468b-9ed3-32d6000462dd/0fe1e8e6-94f3-423b-8365-cd8c8da34f38"
-					(reference "#PWR0318")
+					(reference "#PWR0320")
 					(unit 1)
 				)
@@
 			(project "AD4030-Voltage"
 				(path "/af28bfe6-a5ae-47dd-9259-97a6edcec559/cfc38c8d-3c9b-4f41-9734-05b81b218479"
-					(reference "#PWR0318")
+					(reference "#PWR0320")
 					(unit 1)
 				)
@@
 	)
 	(symbol
+		(lib_id "power:+5VA")
+		(at 16.51 177.8 0)
+		(unit 1)
+		(exclude_from_sim no)
+		(in_bom yes)
+		(on_board yes)
+		(dnp no)
+		(fields_autoplaced yes)
+		(property "Reference" "#PWR0201"
+			(at 16.51 181.61 0)
+			(effects
+				(font
+					(size 1.27 1.27)
+				)
+				(hide yes)
+			)
+		)
+		(property "Value" "+5VA"
+			(at 16.51 172.72 0)
+			(effects
+				(font
+					(size 1.27 1.27)
+				)
+			)
+		)
+		(property "Footprint" ""
+			(at 16.51 177.8 0)
+			(effects
+				(font
+					(size 1.27 1.27)
+				)
+				(hide yes)
+			)
+		)
+		(property "Datasheet" ""
+			(at 16.51 177.8 0)
+			(effects
+				(font
+					(size 1.27 1.27)
+				)
+				(hide yes)
+			)
+		)
+		(property "Description" "Power symbol creates a global label with name \"+5VA\""
+			(at 16.51 177.8 0)
+			(effects
+				(font
+					(size 1.27 1.27)
+				)
+				(hide yes)
+			)
+		)
+		(pin "1"
+		)
+		(instances
+			(project "AD4030-Current"
+				(path "/8c00fb7d-8cfe-468b-9ed3-32d6000462dd/0fe1e8e6-94f3-423b-8365-cd8c8da34f38"
+					(reference "#PWR0201")
+					(unit 1)
+				)
+			)
+		)
+	)
+	(symbol
 		(lib_id "power:GND")
 		(at 162.56 187.96 0)
@@
 					(unit 1)
 				)
+			)
+		)
+	)
+	(symbol
+		(lib_id "AD4030:+5V4")
+		(at 102.87 176.53 0)
+		(unit 1)
+		(exclude_from_sim no)
+		(in_bom yes)
+		(on_board yes)
+		(dnp no)
+		(fields_autoplaced yes)
+		(property "Reference" "#PWR0202"
+			(at 102.87 180.34 0)
+			(effects
+				(font
+					(size 1.27 1.27)
+				)
+				(hide yes)
+			)
+		)
+		(property "Value" "+5V4"
+			(at 102.87 171.45 0)
+			(effects
+				(font
+					(size 1.27 1.27)
+				)
+			)
+		)
+		(property "Footprint" ""
+			(at 102.87 176.53 0)
+			(effects
+				(font
+					(size 1.27 1.27)
+				)
+				(hide yes)
+			)
+		)
+		(property "Datasheet" ""
+			(at 102.87 176.53 0)
+			(effects
+				(font
+					(size 1.27 1.27)
+				)
+				(hide yes)
+			)
+		)
+		(property "Description" ""
+			(at 102.87 176.53 0)
+			(effects
+				(font
+					(size 1.27 1.27)
+				)
+				(hide yes)
+			)
+		)
+		(pin "1"
+		)
+		(instances
+			(project ""
+				(path "/8c00fb7d-8cfe-468b-9ed3-32d6000462dd/0fe1e8e6-94f3-423b-8365-cd8c8da34f38"
+					(reference "#PWR0202")
+					(unit 1)
+				)

Commit message: Hardware
Connections:
- net +5VA is gone; now on net +5V4: C301.1, U301.6 (+Vs), U301.7 (+Vs), U301.8 (+Vs)
Changed lines of the file:
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@@
+	)
+	(symbol
+		(lib_id "AD4030:+5V4")
+		(at 81.28 60.96 0)
+		(unit 1)
+		(exclude_from_sim no)
+		(in_bom yes)
+		(on_board yes)
+		(dnp no)
+		(fields_autoplaced yes)
+		(property "Reference" "#PWR0204"
+			(at 81.28 64.77 0)
+			(effects
+				(font
+					(size 1.27 1.27)
+				)
+				(hide yes)
+			)
+		)
+		(property "Value" "+5V4"
+			(at 81.28 55.88 0)
+			(effects
+				(font
+					(size 1.27 1.27)
+				)
+			)
+		)
+		(property "Footprint" ""
+			(at 81.28 60.96 0)
+			(effects
+				(font
+					(size 1.27 1.27)
+				)
+				(hide yes)
+			)
+		)
+		(property "Datasheet" ""
+			(at 81.28 60.96 0)
+			(effects
+				(font
+					(size 1.27 1.27)
+				)
+				(hide yes)
+			)
+		)
+		(property "Description" ""
+			(at 81.28 60.96 0)
+			(effects
+				(font
+					(size 1.27 1.27)
+				)
+				(hide yes)
+			)
+		)
+		(pin "1"
+		)
+		(instances
+			(project "AD4030-Current"
+				(path "/8c00fb7d-8cfe-468b-9ed3-32d6000462dd/0fe1e8e6-94f3-423b-8365-cd8c8da34f38"
+					(reference "#PWR0204")
+					(unit 1)
+				)
+			)
+		)
 	)
 	(symbol
@@
 	)
 	(symbol
-		(lib_id "power:+5VA")
-		(at 16.51 177.8 0)
-		(unit 1)
-		(exclude_from_sim no)
-		(in_bom yes)
-		(on_board yes)
-		(dnp no)
-		(fields_autoplaced yes)
-		(property "Reference" "#PWR0201"
-			(at 16.51 181.61 0)
-			(effects
-				(font
-					(size 1.27 1.27)
-				)
-				(hide yes)
-			)
-		)
-		(property "Value" "+5VA"
-			(at 16.51 172.72 0)
-			(effects
-				(font
-					(size 1.27 1.27)
-				)
-			)
-		)
-		(property "Footprint" ""
-			(at 16.51 177.8 0)
-			(effects
-				(font
-					(size 1.27 1.27)
-				)
-				(hide yes)
-			)
-		)
-		(property "Datasheet" ""
-			(at 16.51 177.8 0)
-			(effects
-				(font
-					(size 1.27 1.27)
-				)
-				(hide yes)
-			)
-		)
-		(property "Description" "Power symbol creates a global label with name \"+5VA\""
-			(at 16.51 177.8 0)
-			(effects
-				(font
-					(size 1.27 1.27)
-				)
-				(hide yes)
-			)
-		)
-		(pin "1"
-		)
-		(instances
-			(project "AD4030-Current"
-				(path "/8c00fb7d-8cfe-468b-9ed3-32d6000462dd/0fe1e8e6-94f3-423b-8365-cd8c8da34f38"
-					(reference "#PWR0201")
-					(unit 1)
-				)
-			)
-		)
-	)
-	(symbol
 		(lib_id "power:GND")
 		(at 162.56 187.96 0)
@@
 				(path "/af28bfe6-a5ae-47dd-9259-97a6edcec559/cfc38c8d-3c9b-4f41-9734-05b81b218479"
 					(reference "C314")
-					(unit 1)
-				)
-			)
-		)
-	)
-	(symbol
-		(lib_id "power:+5VA")
-		(at 81.28 60.96 0)
-		(unit 1)
-		(exclude_from_sim no)
-		(in_bom yes)
-		(on_board yes)
-		(dnp no)
-		(fields_autoplaced yes)
-		(property "Reference" "#PWR0309"
-			(at 81.28 64.77 0)
-			(effects
-				(font
-					(size 1.27 1.27)
-				)
-				(hide yes)
-			)
-		)
-		(property "Value" "+5VA"
-			(at 81.28 55.88 0)
-			(effects
-				(font
-					(size 1.27 1.27)
-				)
-			)
-		)
-		(property "Footprint" ""
-			(at 81.28 60.96 0)
-			(effects
-				(font
-					(size 1.27 1.27)
-				)
-				(hide yes)
-			)
-		)
-		(property "Datasheet" ""
-			(at 81.28 60.96 0)
-			(effects
-				(font
-					(size 1.27 1.27)
-				)
-				(hide yes)
-			)
-		)
-		(property "Description" "Power symbol creates a global label with name \"+5VA\""
-			(at 81.28 60.96 0)
-			(effects
-				(font
-					(size 1.27 1.27)
-				)
-				(hide yes)
-			)
-		)
-		(pin "1"
-		)
-		(instances
-			(project ""
-				(path "/8c00fb7d-8cfe-468b-9ed3-32d6000462dd/0fe1e8e6-94f3-423b-8365-cd8c8da34f38"
-					(reference "#PWR0309")
-					(unit 1)
-				)
-			)
-			(project ""
-				(path "/af28bfe6-a5ae-47dd-9259-97a6edcec559/cfc38c8d-3c9b-4f41-9734-05b81b218479"
-					(reference "#PWR0309")
 					(unit 1)
 				)
@@
 					(unit 1)
 				)
+			)
+		)
+	)
+	(symbol
+		(lib_id "AD4030:+5V4")
+		(at 16.51 177.8 0)
+		(unit 1)
+		(exclude_from_sim no)
+		(in_bom yes)
+		(on_board yes)
+		(dnp no)
+		(fields_autoplaced yes)
+		(property "Reference" "#PWR0205"
+			(at 16.51 181.61 0)
+			(effects
+				(font
+					(size 1.27 1.27)
+				)
+				(hide yes)
+			)
+		)
+		(property "Value" "+5V4"
+			(at 16.51 172.72 0)
+			(effects
+				(font
+					(size 1.27 1.27)
+				)
+			)
+		)
+		(property "Footprint" ""
+			(at 16.51 177.8 0)
+			(effects
+				(font
+					(size 1.27 1.27)
+				)
+				(hide yes)
+			)
+		)
+		(property "Datasheet" ""
+			(at 16.51 177.8 0)
+			(effects
+				(font
+					(size 1.27 1.27)
+				)
+				(hide yes)
+			)
+		)
+		(property "Description" ""
+			(at 16.51 177.8 0)
+			(effects
+				(font
+					(size 1.27 1.27)
+				)
+				(hide yes)
+			)
+		)
+		(pin "1"
+		)
+		(instances
+			(project "AD4030-Current"
+				(path "/8c00fb7d-8cfe-468b-9ed3-32d6000462dd/0fe1e8e6-94f3-423b-8365-cd8c8da34f38"
+					(reference "#PWR0205")
+					(unit 1)
+				)

Commit message: PCB layout
Parts:
- renumbered C301 to C201, C302 to C202, C303 to C203, C304 to C204, C305 to C205, C306 to C206, C309 to C207, C307 to C208, C308 to C209, C310 to C210, C311 to C211, C312 to C212, C313 to C213, C314 to C214, C315 to C215, C316 to C216, C317 to C217, C318 to C218, C319 to C219, FB301 to FB201, R301 to R201, R302 to R202, R305 to R203, R306 to R204, R307 to R205, R308 to R206, R309 to R207, RN301 to RN201, U301 to U201, U302 to U202, U303 to U203, U304 to U204, X301 to X201
