File: AD4030/Hardware/AD4030-Current/Power.kicad_sch (KiCad schematic)
At the start: 30 parts, among them J501 1715721, Q501 SI5618A, Q502 MMBT3904, U501 ADP7142AUJZ, U502 TSR_1-2433, U503 TEC3-2419WI, U504 LT1763CDE-ADJ, U505 ADP7142AUJZ, U506 ADP5070AREZ, U507 ADP7182AUJZ, U508 ADP7142AUJZ, U509 LM1117LD-ADJ

Commit message: Hardware
Parts:
- removed U501, U505: ADP7142AUJZ, Package_TO_SOT_SMD:TSOT-23-5, symbol Regulator_Linear:ADP7142AUJZ
- added C501, C504, C505, C508, C512, C514, C516, C518: 2u2/35V, Capacitor_SMD:C_1206_3216Metric_Pad1.33x1.80mm_HandSolder, symbol Device:C
- added C509, C511, C519, C520: 10u/25V, Capacitor_SMD:C_1206_3216Metric_Pad1.33x1.80mm_HandSolder, symbol Device:C
- added R505, R507, R508, R509, R510, R511: R, Resistor_SMD:R_0603_1608Metric_Pad0.98x0.95mm_HandSolder, symbol Device:R
- added U501, U510: ADP7142AUJZ-1.8, Package_TO_SOT_SMD:TSOT-23-5, symbol Regulator_Linear:ADP7142AUJZ-1.8
- added U505: LM1117LD-3.3, Package_SON:WSON-8-1EP_4x4mm_P0.8mm_EP2.2x3mm, symbol Regulator_Linear:LM1117LD-3.3
Connections:
- net +15V: now also U508.5 (VOUT), C512.1, R508.1
- net +1V8: now also C508.1, U501.4 (SENSE/ADJ), U501.5 (VOUT)
- net +3.3V: now also C504.1, C505.1, C520.1, U501.1 (VIN), U501.3 (EN), U505.5 (VO), U505.6 (VO), U505.7 (VO), U505.9 (VO), U510.1 (VIN), U510.3 (EN)
- net +5V4: now also U509.5 (VO), U509.6 (VO), U509.7 (VO), U509.9 (VO), C509.1, C519.1, R505.1, U505.2 (VI), U505.3 (VI), U505.4 (VI)
- net +9V: now also U509.2 (VI), U509.3 (VI), U509.4 (VI), C511.1
- net -15V: now also U507.5 (VOUT), C514.2, R510.2
- net GND: now also U507.1 (GND), U508.2 (GND), C501.2, C504.2, C505.2, C508.2, C509.2, C511.2, C512.2, C514.1, C516.1, C518.2, C519.2, C520.2, R507.2, R509.2, R511.1, U501.2 (GND), U505.1 (GND), U510.2 (GND)
- net VIO: now also C501.1, U510.4 (SENSE/ADJ), U510.5 (VOUT)
- net at U509.1 (ADJ): now also R505.2, R507.1
- net +16V: now reaches U508.1 (VIN)
- net +16V: now also U508.3 (EN), C518.1
- net at U508.4 (SENSE/ADJ): now also R508.2, R509.1
- net -16V: now reaches U507.2 (VIN)
- net -16V: now also U507.3 (EN), C516.2
- net at U507.4 (ADJ): now also R510.1, R511.2
Other:
- note removed: "LT8686S LT8601 LT7200S * LTM4668A LT8692S"
- note removed: "https://www.analog.com/en/resources/technical-articles/bipolar-power-solutions-for-precision-test-and-measurement-systems.html https://xdevs.com/article/x732/"
- moved on the sheet: C503, C507, D501, D502, F501, J501, L504, Q501, Q502, R501, R502, U503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

Commit message: Hardware
Parts:
- removed U506: ADP5070AREZ, Package_SO:ETSSOP-20-1EP_4.4x6.5mm_P0.65mm_EP3x4.2mm, symbol AD4030:ADP5070AREZ
- added C521, C525, C528: 1u, Capacitor_SMD:C_0603_1608Metric_Pad1.08x0.95mm_HandSolder, symbol Device:C
- added C522: 0.1u, Capacitor_SMD:C_0603_1608Metric_Pad1.08x0.95mm_HandSolder, symbol Device:C
- added C523: 68n, Capacitor_SMD:C_0603_1608Metric_Pad1.08x0.95mm_HandSolder, symbol Device:C
- added C524: 47n, Capacitor_SMD:C_0603_1608Metric_Pad1.08x0.95mm_HandSolder, symbol Device:C
- added C526, C527, C529: 10u/35V, Capacitor_SMD:C_1206_3216Metric_Pad1.33x1.80mm_HandSolder, symbol Device:C
- added D503, D504: DFLS240-7, AD4030:POWERDI123_DIO, symbol Device:D
- added L501: XAL4030-682MEC, Inductor_SMD:L_Coilcraft_XAL4030-XXX, symbol Device:L
- added L502: XAL4040-153MEB, Inductor_SMD:L_Coilcraft_XAL4040-XXX, symbol Device:L
- added R512: 1k, Resistor_SMD:R_0603_1608Metric_Pad0.98x0.95mm_HandSolder, symbol Device:R
- added R513: 4k64, Resistor_SMD:R_0603_1608Metric_Pad0.98x0.95mm_HandSolder, symbol Device:R
- added R514: 15k, Resistor_SMD:R_0603_1608Metric_Pad0.98x0.95mm_HandSolder, symbol Device:R
- added R515: 12k, Resistor_SMD:R_0603_1608Metric_Pad0.98x0.95mm_HandSolder, symbol Device:R
- added R516: 2M15, Resistor_SMD:R_0603_1608Metric_Pad0.98x0.95mm_HandSolder, symbol Device:R
- added R517: 113k, Resistor_SMD:R_0603_1608Metric_Pad0.98x0.95mm_HandSolder, symbol Device:R
- added R518: 100k, Resistor_SMD:R_0603_1608Metric_Pad0.98x0.95mm_HandSolder, symbol Device:R
- added R519: 2M1, Resistor_SMD:R_0603_1608Metric_Pad0.98x0.95mm_HandSolder, symbol Device:R
- added R520, R521: 10k, Resistor_SMD:R_0603_1608Metric_Pad0.98x0.95mm_HandSolder, symbol Device:R
- added U506: ADP5070ACPZ, Package_DFN_QFN:QFN-20-1EP_4x4mm_P0.5mm_EP2.6x2.6mm_ThermalVias, symbol AD4030:ADP5070ACPZ
- R505: value R -> 3k32
- R507: value R -> 1k
- R508: value R -> 20k
- R509: value R -> 10k
- R510: value R -> 52k3
- R511: value R -> 4k64
Connections:
- net +15V: now also C521.1
- net +16V: now also C526.1, D503.1 (K), R516.2
- net +9V: now also C529.1, R520.1, U506.15 (PVIN1), U506.16 (PVINSYS), U506.17 (PVIN2)
- net -15V: now also C522.2
- net -16V: now also C527.2, D504.2 (A), R519.2
- net GND: now also C523.1, C524.1, C525.1, C526.2, C527.1, C528.2, C529.2, L502.2, R517.2, R521.2, U506.13 (AGND), U506.19 (PGND), U506.2 (SYNC/FREQ), U506.21 (AGND)
- net at R508.2, R509.1, U508.4 (SENSE/ADJ): now also R512.1
- net at R510.1, R511.2, U507.4 (ADJ): now also R513.1
- new net: D503.2 (A), L501.2, U506.20 (SW1)
- new net: C522.1, R513.2
- new net: R516.1, R517.1, U506.5 (FB1)
- new net: C523.2, R514.1
- new net: R514.2, U506.10 (COMP2)
- new net: D504.1 (K), L502.1, U506.18 (SW2)
- new net: C528.1, R518.1, U506.12 (VREF)
- new net: R518.2, R519.1, U506.11 (FB2)
- new net: L501.1, U506.1 (INBK)
- new net: R520.2, R521.1, U506.7 (EN1), U506.9 (EN2)
- new net: C521.2, R512.2
- new net: C525.2, U506.14 (VREG)
- new net: R515.2, U506.6 (COMP1)
- new net: C524.2, R515.1
- no-connect marks 1 -> 4
Other:
- moved on the sheet: C501, C504, C505, C508, C509, C511, C512, C514, C516, C518, C519, C520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

Commit message: PCB layout
Parts:
- renumbered C529 to C501, C524 to C502, C523 to C503, C525 to C504, C503 to C505, C502 to C506, C528 to C507, C507 to C508, C526 to C509, C527 to C510, C506 to C511, C518 to C512, C516 to C513, C510 to C514, C511 to C515, C521 to C516, C522 to C517, C513 to C518, C509 to C519, C512 to C520, C514 to C521, C515 to C522, C504 to C523, C505 to C524, C519 to C525, C517 to C526, C520 to C527, C501 to C528, C508 to C529, L504 to L503, L503 to L504, R520 to R501, R521 to R502, R515 to R503, R514 to R504, R501 to R505, R502 to R506, R517 to R507, R518 to R508, R516 to R509, R519 to R510, R506 to R511, R508 to R512, R509 to R513, R511 to R514, R510 to R515, R507 to R516, R512 to R517, R503 to R518, R504 to R519, R513 to R520, R505 to R521, U506 to U501, U503 to U502, U502 to U503, U508 to U504, U507 to U505, U504 to U506, U509 to U507, U505 to U508, U510 to U509, U501 to U510
