File: AD4030/Hardware/AD4030-Current/Shunt.kicad_sch (KiCad schematic)
At the start: 52 parts, among them U403 AD8479, U404 ADG5236BCPZ, U405 ADG5236BCPZ, U406 ADG5236BCPZ, U407 AD797ARZ, U408 AD797ARZ, U409 AD797ARZ, U410 TXB0101DBV, U411 TXB0101DBV, U412 TXB0101DBV, U413 ADA4077-1xRM, U414 ADG5236BCPZ, U415 TXB0101DBV

Commit message: Hardware
Parts:
- removed R417: WSBS85181L000JK34, symbol Device:R_Shunt
- added R413: WSBS85181L000JK35, AD4030:WSBS8518-35, symbol Device:R
Connections:
- net at R414.1: now also R413.2
- net at U403.3 (+IN): now also R413.1
- no-connect marks 2 -> 0
Changed lines of the file:
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@@
 		(color 0 0 0 0)
 	)
-	(no_connect
-		(at 31.75 83.82)
-	)
-	(no_connect
-		(at 31.75 73.66)
-	)
 	(wire
 		(pts
@@
 	(wire
 		(pts
-			(xy 55.88 83.82) (xy 35.56 83.82)
+			(xy 55.88 83.82) (xy 31.75 83.82)
 		)
 		(stroke
@@
 	(wire
 		(pts
-			(xy 35.56 73.66) (xy 55.88 73.66)
+			(xy 31.75 73.66) (xy 55.88 73.66)
 		)
 		(stroke
@@
 	(wire
 		(pts
-			(xy 35.56 81.28) (xy 35.56 83.82)
+			(xy 31.75 82.55) (xy 31.75 83.82)
 		)
 		(stroke
@@
 	(wire
 		(pts
-			(xy 35.56 73.66) (xy 35.56 76.2)
+			(xy 31.75 73.66) (xy 31.75 74.93)
 		)
 		(stroke
@@
 	)
 	(symbol
+		(lib_id "Device:R")
+		(at 31.75 78.74 0)
+		(unit 1)
+		(exclude_from_sim no)
+		(in_bom yes)
+		(on_board yes)
+		(dnp no)
+		(fields_autoplaced yes)
+		(property "Reference" "R413"
+			(at 34.29 77.4699 0)
+			(effects
+				(font
+					(size 1.27 1.27)
+				)
+				(justify left)
+			)
+		)
+		(property "Value" "WSBS85181L000JK35"
+			(at 34.29 80.0099 0)
+			(effects
+				(font
+					(size 1.27 1.27)
+				)
+				(justify left)
+			)
+		)
+		(property "Footprint" "AD4030:WSBS8518-35"
+			(at 29.972 78.74 90)
+			(effects
+				(font
+					(size 1.27 1.27)
+				)
+				(hide yes)
+			)
+		)
+		(property "Datasheet" "~"
+			(at 31.75 78.74 0)
+			(effects
+				(font
+					(size 1.27 1.27)
+				)
+				(hide yes)
+			)
+		)
+		(property "Description" "Resistor"
+			(at 31.75 78.74 0)
+			(effects
+				(font
+					(size 1.27 1.27)
+				)
+				(hide yes)
+			)
+		)
+		(pin "2"
+		)
+		(pin "1"
+		)
+		(instances
+			(project ""
+				(path "/8c00fb7d-8cfe-468b-9ed3-32d6000462dd/1a7316af-c697-438b-8e8c-11ca1df305e7"
+					(reference "R413")
+					(unit 1)
+				)
+			)
+		)
+	)
+	(symbol
 		(lib_id "power:+15V")
 		(at 242.57 76.2 0)
@@
 					(unit 1)
 				)
-			)
-		)
-	)
-	(symbol
-		(lib_id "Device:R_Shunt")
-		(at 31.75 78.74 0)
-		(unit 1)
-		(exclude_from_sim no)
-		(in_bom yes)
-		(on_board yes)
-		(dnp no)
-		(property "Reference" "R417"
-			(at 48.768 77.216 0)
-			(effects
-				(font
-					(size 1.27 1.27)
-				)
-				(justify right)
-			)
-		)
-		(property "Value" "WSBS85181L000JK34"
-			(at 55.88 79.502 0)
-			(effects
-				(font
-					(size 1.27 1.27)
-				)
-				(justify right)
-			)
-		)
-		(property "Footprint" ""
-			(at 29.972 78.74 90)
-			(effects
-				(font
-					(size 1.27 1.27)
-				)
-				(hide yes)
-			)
-		)
-		(property "Datasheet" "~"
-			(at 31.75 78.74 0)
-			(effects
-				(font
-					(size 1.27 1.27)
-				)
-				(hide yes)
-			)
-		)
-		(property "Description" "Shunt resistor"
-			(at 31.75 78.74 0)
-			(effects
-				(font
-					(size 1.27 1.27)
-				)
-				(hide yes)
-			)
-		)
-		(pin "2"
-		)
-		(pin "4"
-		)
-		(pin "3"
-		)
-		(pin "1"
-		)
-		(instances
-			(project ""
-				(path "/8c00fb7d-8cfe-468b-9ed3-32d6000462dd/1a7316af-c697-438b-8e8c-11ca1df305e7"
-					(reference "R417")
-					(unit 1)
-				)

Commit message: Hardware
Parts:
- U403: value AD8479 -> AD8479ARZ
Connections:
- net +5V renamed +5V4

Commit message: PCB layout
Parts:
- added C430, C431: 0.1u, Capacitor_SMD:C_0603_1608Metric_Pad1.08x0.95mm_HandSolder, symbol Device:C
- renumbered C426 to C401, C419 to C402, C427 to C403, C420 to C404, C428 to C405, C421 to C406, C437 to C407, C422 to C408, C423 to C409, C424 to C410, C425 to C411, C434 to C412, C412 to C413, C409 to C414, C413 to C415, C414 to C416, C415 to C417, C416 to C418, C417 to C419, C410 to C420, C418 to C421, C435 to C422, C429 to C423, C430 to C424, C431 to C425, C411 to C426, C436 to C427, C433 to C428, C432 to C429, R413 to R401, R414 to R402, R415 to R403, R416 to R404, U403 to U401, U404 to U402, U407 to U403, U410 to U404, U408 to U406, U411 to U407, U406 to U408, U412 to U410, U414 to U411, U415 to U412
Connections:
- net +15V: now also C430.1
- net -15V: now also C431.1
- net GND: now also C430.2, C431.2
- net LP_FILTER renamed LP_Filter
Other:
- moved on the sheet: C413, C415, C416, C417, C418, C419, C421, C422, C423, C424, C425, C427
