File: AD4030/Hardware/AD4030-Current/AD4030-Current.kicad_sch (KiCad schematic)
At the start: 0 parts

Commit message: Hardware
Other:
- sheet ADC ports: added ADC_BUSY, ADC_CNV, ADC_SCK, ADC_SDI, ADC_SDO0, ADC_SDO1, ADC_SDO2, ADC_SDO3, ADC_~{CS}, CLK_100MHz, CURRENT_OUT; removed none
- sheet Isolation ports: added ADC_BUSY, ADC_CNV, ADC_SCK, ADC_SDI, ADC_SDO0, ADC_SDO1, ADC_SDO2, ADC_SDO3, ADC_~{CS}, CLK_100MHz, GAIN_x10B, Gain_x10A; removed none
- sheet Shunt ports: added CURRENT_OUT, Gain_x10A, Gain_x10B, Gain_x10C, LP_FILTER; removed none

Commit message: Hardware
Other:
- sheet Isolation ports: added Gain_x10B; removed GAIN_x10B
Changed lines of the file:
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@@
 			)
 		)
-		(pin "GAIN_x10B" output
+		(pin "Gain_x10B" output
 			(at 173.99 74.93 180)
 			(effects

Commit message: PCB layout
Other:
- sheet Isolation ports: added Gain_x10C, LP_Filter; removed none
- sheet Shunt ports: added LP_Filter; removed LP_FILTER
Changed lines of the file:
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@@
+	(wire
+		(pts
+			(xy 127 80.01) (xy 173.99 80.01)
+		)
+		(stroke
+			(width 0)
+			(type default)
+		)
+	)
 	(wire
 		(pts
 			(xy 167.64 59.69) (xy 173.99 59.69)
+		)
+		(stroke
+			(width 0)
+			(type default)
+		)
+	)
+	(wire
+		(pts
+			(xy 127 77.47) (xy 173.99 77.47)
 		)
 		(stroke
@@
 			)
 		)
-		(pin "LP_FILTER" input
+		(pin "LP_Filter" input
 			(at 127 80.01 0)
 			(effects
@@
 			(effects
 				(font
+					(size 1.27 1.27)
+				)
+				(justify left)
+			)
+		)
+		(pin "LP_Filter" output
+			(at 173.99 80.01 180)
+			(effects
+				(font
+					(size 1.27 1.27)
+				)
+				(justify left)
+			)
+		)
+		(pin "Gain_x10C" output
+			(at 173.99 77.47 180)
+			(effects
+				(font

Commit message: PCB layout
Parts:
- added H101, H102: MountingHole, MountingHole:MountingHole_3.2mm_M3_DIN965_Pad, symbol Mechanical:MountingHole
Changed lines of the file:
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@@
+		)
+	)
+	(symbol
+		(lib_id "Mechanical:MountingHole")
+		(at 25.4 186.69 0)
+		(unit 1)
+		(exclude_from_sim yes)
+		(in_bom no)
+		(on_board yes)
+		(dnp no)
+		(fields_autoplaced yes)
+		(property "Reference" "H102"
+			(at 27.94 185.4199 0)
+			(effects
+				(font
+					(size 1.27 1.27)
+				)
+				(justify left)
+			)
+		)
+		(property "Value" "MountingHole"
+			(at 27.94 187.9599 0)
+			(effects
+				(font
+					(size 1.27 1.27)
+				)
+				(justify left)
+			)
+		)
+		(property "Footprint" "MountingHole:MountingHole_3.2mm_M3_DIN965_Pad"
+			(at 25.4 186.69 0)
+			(effects
+				(font
+					(size 1.27 1.27)
+				)
+				(hide yes)
+			)
+		)
+		(property "Datasheet" "~"
+			(at 25.4 186.69 0)
+			(effects
+				(font
+					(size 1.27 1.27)
+				)
+				(hide yes)
+			)
+		)
+		(property "Description" "Mounting Hole without connection"
+			(at 25.4 186.69 0)
+			(effects
+				(font
+					(size 1.27 1.27)
+				)
+				(hide yes)
+			)
+		)
+		(instances
+			(project "AD4030-Current"
+				(path "/8c00fb7d-8cfe-468b-9ed3-32d6000462dd"
+					(reference "H102")
+					(unit 1)
+				)
+			)
+		)
+	)
+	(symbol
+		(lib_id "Mechanical:MountingHole")
+		(at 25.4 177.8 0)
+		(unit 1)
+		(exclude_from_sim yes)
+		(in_bom no)
+		(on_board yes)
+		(dnp no)
+		(fields_autoplaced yes)
+		(property "Reference" "H101"
+			(at 27.94 176.5299 0)
+			(effects
+				(font
+					(size 1.27 1.27)
+				)
+				(justify left)
+			)
+		)
+		(property "Value" "MountingHole"
+			(at 27.94 179.0699 0)
+			(effects
+				(font
+					(size 1.27 1.27)
+				)
+				(justify left)
+			)
+		)
+		(property "Footprint" "MountingHole:MountingHole_3.2mm_M3_DIN965_Pad"
+			(at 25.4 177.8 0)
+			(effects
+				(font
+					(size 1.27 1.27)
+				)
+				(hide yes)
+			)
+		)
+		(property "Datasheet" "~"
+			(at 25.4 177.8 0)
+			(effects
+				(font
+					(size 1.27 1.27)
+				)
+				(hide yes)
+			)
+		)
+		(property "Description" "Mounting Hole without connection"
+			(at 25.4 177.8 0)
+			(effects
+				(font
+					(size 1.27 1.27)
+				)
+				(hide yes)
+			)
+		)
+		(instances
+			(project ""
+				(path "/8c00fb7d-8cfe-468b-9ed3-32d6000462dd"
+					(reference "H101")
+					(unit 1)
+				)
+			)
 		)
 	)
