File: AD4030/Hardware/AD4030-Current/Isolation.kicad_sch (KiCad schematic)
At the start: 31 parts, among them J401 Conn_01x08, J402 Conn_01x07, J403 PMOD, J404 PMOD, U305 ADuM260N, U401 ADuM260N, U402 ADuM260N

Commit message: Hardware
Connections:
- net CONN_GAIN_x10: no longer R410.2, U402.2 (VIA)
- net CONN_GAIN_x100 renamed CONN_GAIN_x10B
- net GAIN_x100 renamed GAIN_x10B
- net Gain_x10 renamed Gain_x10A
- new net CONN_GAIN_x10A: R410.2, U402.2 (VIA)
Changed lines of the file:
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@@
 		)
 	)
-	(label "CONN_GAIN_x100"
+	(label "CONN_GAIN_x10B"
 		(at 139.7 73.66 180)
 		(fields_autoplaced yes)
@@
 		)
 	)
-	(label "CONN_GAIN_x10"
+	(label "CONN_GAIN_x10A"
 		(at 139.7 71.12 180)
 		(fields_autoplaced yes)
@@
 		)
 	)
-	(label "CONN_GAIN_x10"
+	(label "CONN_GAIN_x10A"
 		(at 278.13 57.15 180)
 		(fields_autoplaced yes)
@@
 		)
 	)
-	(label "CONN_GAIN_x100"
+	(label "CONN_GAIN_x10B"
 		(at 196.85 57.15 0)
 		(fields_autoplaced yes)
@@
 		)
 	)
-	(hierarchical_label "GAIN_x100"
+	(hierarchical_label "GAIN_x10B"
 		(shape output)
 		(at 85.09 73.66 180)
@@
 		)
 	)
-	(hierarchical_label "Gain_x10"
+	(hierarchical_label "Gain_x10A"
 		(shape output)
 		(at 85.09 71.12 180)

Commit message: Hardware
Connections:
- net GAIN_x10B renamed Gain_x10B
Changed lines of the file:
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@@
 		)
 	)
-	(hierarchical_label "GAIN_x10B"
+	(hierarchical_label "Gain_x10B"
 		(shape output)
 		(at 85.09 73.66 180)

Commit message: PCB layout
Parts:
- added R304, R311: 51, Resistor_SMD:R_0402_1005Metric_Pad0.72x0.64mm_HandSolder, symbol Device:R
- renumbered C401 to C301, C320 to C302, C402 to C303, C321 to C304, C403 to C305, C404 to C306, C405 to C307, C322 to C308, C406 to C309, C323 to C310, C407 to C311, C408 to C312, J401 to J301, J402 to J302, J403 to J303, J404 to J304, R401 to R301, R402 to R302, R403 to R303, R404 to R305, R405 to R306, R406 to R307, R407 to R308, R408 to R309, R409 to R310, R410 to R312, R411 to R313, R412 to R314, U401 to U301, U402 to U302, U305 to U303
Connections:
- net CONN_GAIN_x10 is gone; now on net CONN_GAIN_x10B: J302.4 (Pin_4)
- net CONN_GAIN_x20 is gone; now on net CONN_GAIN_x10A: J302.3 (Pin_3)
- net CONN_GAIN_x10C: now reaches J302.5 (Pin_5)
- net CONN_GAIN_x10C: now also U303.2 (VIA), R304.1
- net CONN_LP_FILTER: now reaches J302.6 (Pin_6)
- net CONN_LP_FILTER: now also U303.3 (VIB), R311.2
- net at J304.11 (Pin_11): now also R311.1
- net at J304.12 (Pin_12): now also R304.2
- net LP_Filter: now reaches U303.14 (VOB)
- net Gain_x10C: now reaches U303.15 (VOA)
- no-connect marks 10 -> 14

Commit message: PCB layout
Connections:
- net CONN_GAIN_x10C: now also J302.6 (Pin_6), U303.7 (VIF); no longer J302.5 (Pin_5), U303.2 (VIA)
- net CONN_LP_FILTER: now also J302.5 (Pin_5), U303.6 (VIE); no longer J302.6 (Pin_6), U303.3 (VIB)
- net Gain_x10C: now also U303.10 (VOF); no longer U303.15 (VOA)
- net LP_Filter: now also U303.11 (VOE); no longer U303.14 (VOB)
Changed lines of the file:
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@@
-	)
-	(no_connect
-		(at 118.11 120.65)
 	)
 	(no_connect
@@
 	)
 	(no_connect
+		(at 118.11 107.95)
+	)
+	(no_connect
 		(at 87.63 113.03)
+	)
+	(no_connect
+		(at 118.11 110.49)
 	)
 	(no_connect
@@
 	)
 	(no_connect
+		(at 87.63 107.95)
+	)
+	(no_connect
 		(at 231.14 67.31)
-	)
-	(no_connect
-		(at 87.63 118.11)
-	)
-	(no_connect
-		(at 118.11 118.11)
 	)
 	(no_connect
@@
 	)
 	(no_connect
-		(at 87.63 120.65)
+		(at 87.63 110.49)
 	)
 	(no_connect
@@
 	(wire
 		(pts
-			(xy 118.11 107.95) (xy 139.7 107.95)
+			(xy 118.11 118.11) (xy 139.7 118.11)
 		)
 		(stroke
@@
 	(wire
 		(pts
-			(xy 85.09 110.49) (xy 87.63 110.49)
+			(xy 85.09 120.65) (xy 87.63 120.65)
 		)
 		(stroke
@@
 	(wire
 		(pts
-			(xy 118.11 110.49) (xy 139.7 110.49)
+			(xy 118.11 120.65) (xy 139.7 120.65)
 		)
 		(stroke
@@
 	(wire
 		(pts
-			(xy 85.09 107.95) (xy 87.63 107.95)
+			(xy 85.09 118.11) (xy 87.63 118.11)
 		)
 		(stroke
@@
 	)
 	(label "CONN_LP_FILTER"
-		(at 139.7 110.49 180)
+		(at 139.7 118.11 180)
 		(fields_autoplaced yes)
 		(effects
@@
 	)
 	(label "CONN_GAIN_x10C"
-		(at 149.86 86.36 0)
+		(at 149.86 88.9 0)
 		(fields_autoplaced yes)
 		(effects
@@
 	)
 	(label "CONN_GAIN_x10C"
-		(at 139.7 107.95 180)
+		(at 139.7 120.65 180)
 		(fields_autoplaced yes)
 		(effects
@@
 	)
 	(label "CONN_LP_FILTER"
-		(at 149.86 88.9 0)
+		(at 149.86 86.36 0)
 		(fields_autoplaced yes)
 		(effects
@@
 	(hierarchical_label "Gain_x10C"
 		(shape output)
-		(at 85.09 107.95 180)
+		(at 85.09 120.65 180)
 		(fields_autoplaced yes)
 		(effects
@@
 	(hierarchical_label "LP_Filter"
 		(shape output)
-		(at 85.09 110.49 180)
-		(fields_autoplaced yes)
-		(effects
+		(at 85.09 118.11 180)
+		(fields_autoplaced yes)
+		(effects
