File: AD4030/Hardware/AD4030-Current/AD4030-Current.kicad_pcb (KiCad board)
At the start: 4 copper layers, 125 x 70 mm, 192 parts, among them J301 Conn_01x08, J302 Conn_01x07, J303 PMOD, J304 PMOD, J501 1715721, Q501 SI5618A, Q502 MMBT3904, U201 AD8475ACPZ, U202 SN74AUC1G79DBVR, U203 AD4030-24, U204 LTC6655BHMS8-5, U301 ADuM260N, U302 ADuM260N, U303 ADuM260N, U401 AD8479ARZ, U402 ADG5236BCPZ, U403 AD797ARZ, U404 TXB0101DBV, U405 ADG5236BCPZ, U406 AD797ARZ, U407 TXB0101DBV, U408 ADG5236BCPZ, U409 AD797ARZ, U410 TXB0101DBV, U411 ADG5236BCPZ, U412 TXB0101DBV, U413 ADA4077-1xRM, U501 ADP5070ACPZ, U502 TEC3-2419WI, U503 TSR_1-2433, U504 ADP7142AUJZ, U505 ADP7182AUJZ, U506 LT1763CDE-ADJ, U507 LM1117LD-ADJ, U508 LM1117LD-3.3, U509 ADP7142AUJZ-1.8, U510 ADP7142AUJZ-1.8, X201 ECS-2520MV-1000-BN-TR

Commit message: PCB layout
Parts:
- added H101: MountingHole, MountingHole:MountingHole_3.2mm_M3_DIN965_Pad, F.Cu at (120.0, 65.0)
- added H102: MountingHole, MountingHole:MountingHole_3.2mm_M3_DIN965_Pad, F.Cu at (120.0, 125.0)
- moved J304 3.06 mm to (203.3, 108.0)
- moved R304 3.05 mm to (200.2, 119.4)
- moved R305 3.05 mm to (200.2, 116.8)
- moved R306 3.05 mm to (200.2, 114.3)
- moved R307 3.05 mm to (200.2, 111.8)
- moved R311 3.05 mm to (200.2, 120.7)
- moved R312 3.05 mm to (200.2, 118.1)
- moved R314 3.05 mm to (200.2, 113.0)
- moved R313 3.05 mm to (200.2, 115.6)
- moved R402 1.78 mm to (108.8, 102.5)
- moved J303 1.53 mm to (203.3, 85.0)
- moved R301 1.52 mm to (200.2, 93.9)
- moved R302 1.52 mm to (200.2, 91.3)
- moved R303 1.52 mm to (200.2, 88.8)
- moved R308 1.52 mm to (200.2, 95.1)
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Connections:
- J302 pad 5: /Isolation/CONN_GAIN_x10C -> /Isolation/CONN_LP_FILTER
- J302 pad 6: /Isolation/CONN_LP_FILTER -> /Isolation/CONN_GAIN_x10C
- U303 pad 10: unconnected-(U303-VOF-Pad10) -> /Isolation/Gain_x10C
- U303 pad 11: unconnected-(U303-VOE-Pad11) -> /Isolation/LP_Filter
- U303 pad 14: /Isolation/LP_Filter -> unconnected-(U303-VOB-Pad14)
- U303 pad 15: /Isolation/Gain_x10C -> unconnected-(U303-VOA-Pad15)
- U303 pad 2: /Isolation/CONN_GAIN_x10C -> unconnected-(U303-VIA-Pad2)
- U303 pad 3: /Isolation/CONN_LP_FILTER -> unconnected-(U303-VIB-Pad3)
- U303 pad 6: unconnected-(U303-VIE-Pad6) -> /Isolation/CONN_LP_FILTER
- U303 pad 7: unconnected-(U303-VIF-Pad7) -> /Isolation/CONN_GAIN_x10C
Routing:
- net /Isolation/CONN_GAIN_x10B: track 0.00 -> 24.1 mm, vias 0 -> 1
- net /Isolation/CONN_SDO3: track 0.00 -> 23.3 mm, vias 0 -> 1
- net Net-(U401-+IN): track 0.00 -> 22.9 mm
- net Net-(R401-Pad2): track 0.00 -> 22.7 mm
- net /Isolation/CONN_100MHz: track 0.00 -> 22.2 mm, vias 0 -> 1
- net /Isolation/CONN_SDO2: track 0.00 -> 21.0 mm, vias 0 -> 1
- net /Isolation/CONN_SCK: track 0.00 -> 20.8 mm, vias 0 -> 1
- net /Isolation/CONN_GAIN_x10C: track 0.00 -> 20.1 mm, vias 0 -> 1
- net /Isolation/CONN_BUSY: track 0.00 -> 19.7 mm, vias 0 -> 1
- net /Isolation/CONN_LP_FILTER: track 0.00 -> 19.3 mm, vias 0 -> 1
- net /Isolation/CONN_~{CS}: track 0.00 -> 19.2 mm, vias 0 -> 1
- net /Isolation/CONN_CNV: track 0.00 -> 18.9 mm, vias 0 -> 1
- net /Isolation/CONN_SDO1: track 0.00 -> 18.4 mm, vias 0 -> 1
- net /Isolation/CONN_GAIN_x10A: track 0.00 -> 18.0 mm, vias 0 -> 1
- net /Isolation/CONN_SDI: track 0.00 -> 18.0 mm, vias 0 -> 1
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Other:
- outline, holes or cut-outs redrawn
